File: MP_SamBaseBoard_V1/MP_SamBaseBoard_V1.kicad_pcb (KiCad board)
At the start: 2 copper layers, 196 x 60 mm, 63 parts

Commit message: Add new design
Parts:
- added G***: LOGO, GiraffeTech-Utility:basebaord_text3, F.Cu at (94.0, 51.0)
- added REF**: GTK_TFMS08TK-PP-02, GiraffeTech-Connector:GTK_TFMS08TK-PP-02, F.Cu at (146.0, 45.0)
- added REF**: Dinkle_ED350V_2Pins_Pitch3.5mm, GiraffeTech-Connector:TerminalBlock_Dinkle_ED350V_1x02_P3.50mm_Horizontal, F.Cu at (138.0, 24.5)
- added REF**: Sensirion_SHT3x, GiraffeTech-Sensiroin:Sensirion_SHT3x, F.Cu at (68.5, 64.0)
- added REF**: LED_WS2812B_PLCC4_5.0x5.0mm_P3.2mm, LED_SMD:LED_WS2812B_PLCC4_5.0x5.0mm_P3.2mm, F.Cu at (88.5, 35.5)
- added REF**: LED_WS2812B_PLCC4_5.0x5.0mm_P3.2mm, LED_SMD:LED_WS2812B_PLCC4_5.0x5.0mm_P3.2mm, F.Cu at (78.8, 35.5)
- added REF**: USB_Micro-B_Amphenol_10118193_Horizontal, GiraffeTech-Connector:USB_Micro-B_Amphenol_10118193_Horizontal, F.Cu at (149.5, 52.0)
- added REF**: JST_PH_B4B-PH-K_1x04_P2.00mm_Vertical, Connector_JST:JST_PH_B4B-PH-K_1x04_P2.00mm_Vertical, F.Cu at (120.2, 29.5)
- added REF**: SW_SPST_B3S-1000, Button_Switch_SMD:SW_SPST_B3S-1000, F.Cu at (78.8, 26.2)
- added REF**: PinHeader_2x05_P1.27mm_Vertical, Connector_PinHeader_1.27mm:PinHeader_2x05_P1.27mm_Vertical, F.Cu at (125.0, 51.5)
- added REF**: QFN-16-1EP_3x3mm_Pitch0.5mm, GiraffeTech-Maxim:QFN-16-1EP_3x3mm_Pitch0.5mm, F.Cu at (130.8, 41.5)
- added REF**: GTK_TFMS08TK-PP-02, GiraffeTech-Connector:GTK_TFMS08TK-PP-02, F.Cu at (87.5, 76.0)
- added REF**: Dinkle_ED350V_2Pins_Pitch3.5mm, GiraffeTech-Connector:TerminalBlock_Dinkle_ED350V_1x02_P3.50mm_Horizontal, F.Cu at (147.5, 61.0)
- added REF**: JST_PH_B4B-PH-K_1x04_P2.00mm_Vertical, Connector_JST:JST_PH_B4B-PH-K_1x04_P2.00mm_Vertical, F.Cu at (82.0, 78.5)
- added REF**: MountingHole_3.5mm, MountingHole:MountingHole_3.5mm, F.Cu at (69.0, 77.0)
- added REF**: QFN-16-1EP_3x3mm_Pitch0.5mm, GiraffeTech-Maxim:QFN-16-1EP_3x3mm_Pitch0.5mm, F.Cu at (113.0, 65.2)
- added REF**: MountingHole_3.5mm, MountingHole:MountingHole_3.5mm, F.Cu at (147.0, 25.0)
- added REF**: JST_PH_B4B-PH-K_1x04_P2.00mm_Vertical, Connector_JST:JST_PH_B4B-PH-K_1x04_P2.00mm_Vertical, F.Cu at (128.2, 29.5)
- added REF**: SOT-23-5, Package_TO_SOT_SMD:SOT-23-5, F.Cu at (147.0, 69.0)
- added REF**: JST_PH_B4B-PH-K_1x04_P2.00mm_Vertical, Connector_JST:JST_PH_B4B-PH-K_1x04_P2.00mm_Vertical, F.Cu at (112.2, 29.5)
- added REF**: ESP32-WROOM-32, RF_Module:ESP32-WROOM-32, F.Cu at (37.2, 74.2)
- added REF**: BarrelJack_Horizontal, Connector_BarrelJack:BarrelJack_Horizontal, F.Cu at (137.5, 67.0)
- added REF**: TerminalBlock_DEGSON_DG300-5-2pol, GiraffeTech-Connector:TerminalBlock_DEGSON_DG300-5-2pol, F.Cu at (106.8, 73.0)
- added REF**: Symbol_Barrel_Polarity, Symbol:Symbol_Barrel_Polarity, F.Cu at (131.2, 76.5)
- added REF**: TerminalBlock_DEGSON_DG300-5-2pol, GiraffeTech-Connector:TerminalBlock_DEGSON_DG300-5-2pol, F.Cu at (116.8, 73.0)
- added REF**: MountingHole_3.5mm, MountingHole:MountingHole_3.5mm, F.Cu at (69.0, 25.0)
- added REF**: SW_SPST_B3S-1000, Button_Switch_SMD:SW_SPST_B3S-1000, F.Cu at (88.5, 26.2)
- added REF**: MountingHole_3.5mm, MountingHole:MountingHole_3.5mm, F.Cu at (147.0, 77.0)
- added REF**: JST_PH_B4B-PH-K_1x04_P2.00mm_Vertical, Connector_JST:JST_PH_B4B-PH-K_1x04_P2.00mm_Vertical, F.Cu at (104.2, 29.5)
- added REF**: JST_PH_B4B-PH-K_1x04_P2.00mm_Vertical, Connector_JST:JST_PH_B4B-PH-K_1x04_P2.00mm_Vertical, F.Cu at (75.8, 78.5)
- added REF**: Dinkle_ED350V_2Pins_Pitch3.5mm, GiraffeTech-Connector:TerminalBlock_Dinkle_ED350V_1x02_P3.50mm_Horizontal, F.Cu at (253.0, 107.5)
- added REF**: PinHeader_1x03_P2.54mm_Vertical, Connector_PinHeader_2.54mm:PinHeader_1x03_P2.54mm_Vertical, F.Cu at (239.0, 137.5)
- added REF**: PinHeader_1x03_P2.54mm_Vertical, Connector_PinHeader_2.54mm:PinHeader_1x03_P2.54mm_Vertical, F.Cu at (239.0, 132.5)
- added REF**: PinHeader_2x03_P2.54mm_Vertical, Connector_PinHeader_2.54mm:PinHeader_2x03_P2.54mm_Vertical, F.Cu at (241.0, 128.0)
- added REF**: LED_0603_1608Metric, LED_SMD:LED_0603_1608Metric, F.Cu at (150.0, 69.0)
- added REF**: LGA-16_3x3mm_P0.5mm_LayoutBorder3x5y, Package_LGA:LGA-16_3x3mm_P0.5mm_LayoutBorder3x5y, F.Cu at (68.5, 69.0)
- added REF**: TQFP-64_10x10mm_P0.5mm, Package_QFP:TQFP-64_10x10mm_P0.5mm, F.Cu at (108.0, 51.0)
- added REF**: ESP32-WROOM-32_ButtLess, GiraffeTech-NodeMCU:ESP32-WROOM-32_ButtLess, F.Cu at (81.0, 51.0)
- added REF**: PinHeader_1x03_P2.54mm_Vertical, Connector_PinHeader_2.54mm:PinHeader_1x03_P2.54mm_Vertical, F.Cu at (67.0, 33.0)
- added REF**: JST_PH_B4B-PH-K_1x04_P2.00mm_Vertical, Connector_JST:JST_PH_B4B-PH-K_1x04_P2.00mm_Vertical, F.Cu at (96.2, 29.5)
- moved REF** 38.1 mm to (245.2, 144.5), turned to 180 degrees
Other:
- board size 196 x 60 mm -> 201 x 139 mm
- board text added: "+"
- board text added: "-"
- board text added: "1"
- board text added: "2"
- board text added: "< 30V"
- board text added: "ACCEL"
- board text added: "CHG"
- board text added: "D1 UART"
- board text added: "D3 A1"
- board text added: "D4 A2"
- board text added: "D5 A3"
- board text added: "DO"
- board text added: "SPK"
- board text added: "T&H"
- board text added: "WS2812 CHAIN"

Commit message: update
Parts:
- removed the REF** at (87.5, 76.0)
- removed the REF** at (106.8, 73.0)
- removed the REF** at (116.8, 73.0)
- added REF**: R_0603_1608Metric, Resistor_SMD:R_0603_1608Metric, F.Cu at (73.2, 68.0)
- added REF**: C_0603_1608Metric, Capacitor_SMD:C_0603_1608Metric, F.Cu at (126.0, 40.5)
- added REF**: C_0603_1608Metric, Capacitor_SMD:C_0603_1608Metric, F.Cu at (143.2, 55.8)
- added REF**: C_0603_1608Metric, Capacitor_SMD:C_0603_1608Metric, F.Cu at (144.8, 55.8)
- added REF**: C_0603_1608Metric, Capacitor_SMD:C_0603_1608Metric, F.Cu at (148.8, 65.8)
- added REF**: C_0603_1608Metric, Capacitor_SMD:C_0603_1608Metric, F.Cu at (147.0, 72.0)
- added REF**: C_0603_1608Metric, Capacitor_SMD:C_0603_1608Metric, F.Cu at (145.2, 65.8)
- added REF**: SOT-23-6, Package_TO_SOT_SMD:SOT-23-6, F.Cu at (93.8, 66.8)
- added REF**: SOT-23-6, Package_TO_SOT_SMD:SOT-23-6, F.Cu at (89.5, 66.8)
- added REF**: DINKLE_EK500V-2P, GiraffeTech-Connector:DINKLE_EK500V-2P, F.Cu at (91.5, 76.0)
- added REF**: DINKLE_EK500V-2P, GiraffeTech-Connector:DINKLE_EK500V-2P, F.Cu at (102.2, 76.0)
- added REF**: R_0603_1608Metric, Resistor_SMD:R_0603_1608Metric, F.Cu at (75.0, 68.0)
- added REF**: PinHeader_2x03_P2.54mm_Vertical, Connector_PinHeader_2.54mm:PinHeader_2x03_P2.54mm_Vertical, F.Cu at (123.0, 79.0)
- added REF**: DINKLE_EK500V-2P, GiraffeTech-Connector:DINKLE_EK500V-2P, F.Cu at (113.0, 76.0)
- added REF**: C_0603_1608Metric, Capacitor_SMD:C_0603_1608Metric, F.Cu at (74.0, 29.8)
- added REF**: C_0603_1608Metric, Capacitor_SMD:C_0603_1608Metric, F.Cu at (83.8, 29.8)
- added REF**: C_0603_1608Metric, Capacitor_SMD:C_0603_1608Metric, F.Cu at (100.5, 22.8)
- added REF**: C_0603_1608Metric, Capacitor_SMD:C_0603_1608Metric, F.Cu at (108.5, 22.8)
- added REF**: C_0603_1608Metric, Capacitor_SMD:C_0603_1608Metric, F.Cu at (116.5, 22.8)
- added REF**: C_0603_1608Metric, Capacitor_SMD:C_0603_1608Metric, F.Cu at (132.5, 22.7)
- added REF**: C_0603_1608Metric, Capacitor_SMD:C_0603_1608Metric, F.Cu at (124.5, 22.8)
- moved REF** 6.08 mm to (97.2, 23.5), turned to 270 degrees
- moved REF** 6.08 mm to (121.2, 23.5), turned to 270 degrees
- moved REF** 6.08 mm to (83.0, 72.5), turned to 270 degrees
- moved REF** 6.08 mm to (129.2, 23.5), turned to 270 degrees
- moved REF** 6.08 mm to (113.2, 23.5), turned to 270 degrees
- moved REF** 6.08 mm to (105.2, 23.5), turned to 270 degrees
- moved REF** 6.05 mm to (76.5, 72.5), turned to 270 degrees
- moved REF** 5.10 mm to (108.0, 66.2)
Other:
- board text added: "CH1"
- board text added: "CH2"
- board text added: "LOAD"
- board text added: "MOTOR 1"
- board text added: "MOTOR 2"
- board text added: "S"
- board text added: "SERVO"

Commit message: Update
Parts:
- added G***: LOGO, GiraffeTech-Utility:basebaord_text3, F.Cu at (288.4, 51.0)
- added G***: LOGO, GiraffeTech-Utility:basebaord_text3, F.Cu at (192.5, 51.0)
- added MS2: FEATHERWING_NODIM, GiraffeTech-Connector:Adafruit-Feather_WoMountPoint, F.Cu at (335.6, 39.6)
- added MS2: FEATHERWING_NODIM, GiraffeTech-Connector:Adafruit-Feather_WoMountPoint, F.Cu at (249.2, 39.6)
- added MS2: FEATHERWING_NODIM, GiraffeTech-Connector:Adafruit-Feather, F.Cu at (98.2, 5.25)
- added REF**: SW_SPST_B3S-1000, Button_Switch_SMD:SW_SPST_B3S-1000, F.Cu at (341.0, 40.8)
- added REF**: PinHeader_2x05_P1.27mm_Vertical, Connector_PinHeader_1.27mm:PinHeader_2x05_P1.27mm_Vertical, F.Cu at (278.9, 64.1)
- added REF**: C_0603_1608Metric, Capacitor_SMD:C_0603_1608Metric, F.Cu at (182.2, 29.8)
- added REF**: USB_Micro-B_Amphenol_10118193_Horizontal, GiraffeTech-Connector:USB_Micro-B_Amphenol_10118193_Horizontal, F.Cu at (248.0, 51.0)
- added REF**: SOT-23-6, Package_TO_SOT_SMD:SOT-23-6, F.Cu at (233.5, 35.5)
- added REF**: DINKLE_EK500V-2P, GiraffeTech-Connector:DINKLE_EK500V-2P, F.Cu at (214.5, 26.0)
- added REF**: QFN-16-1EP_3x3mm_Pitch0.5mm, GiraffeTech-Maxim:QFN-16-1EP_3x3mm_Pitch0.5mm, F.Cu at (197.0, 33.2)
- added REF**: MountingHole_3.5mm, MountingHole:MountingHole_3.5mm, F.Cu at (245.5, 77.0)
- added REF**: SW_SPST_B3S-1000, Button_Switch_SMD:SW_SPST_B3S-1000, F.Cu at (187.0, 26.2)
- added REF**: MountingHole_3.5mm, MountingHole:MountingHole_3.5mm, F.Cu at (167.5, 25.0)
- added REF**: GTK_TFMS08TK-PP-02, GiraffeTech-Connector:GTK_TFMS08TK-PP-02, F.Cu at (210.8, 76.0)
- added REF**: R_0603_1608Metric, Resistor_SMD:R_0603_1608Metric, F.Cu at (174.0, 64.2)
- added REF**: JST_PH_B4B-PH-K_1x04_P2.00mm_Vertical, Connector_JST:JST_PH_B4B-PH-K_1x04_P2.00mm_Vertical, F.Cu at (270.2, 72.5)
- added REF**: C_0603_1608Metric, Capacitor_SMD:C_0603_1608Metric, F.Cu at (172.5, 29.8)
- added REF**: PinHeader_1x10_P2.54mm_Vertical, Connector_PinHeader_2.54mm:PinHeader_1x10_P2.54mm_Vertical, F.Cu at (96.8, 38.5)
- added REF**: PinHeader_1x10_P2.54mm_Vertical, Connector_PinHeader_2.54mm:PinHeader_1x10_P2.54mm_Vertical, F.Cu at (96.8, 62.8)
- added REF**: BarrelJack_Horizontal, Connector_BarrelJack:BarrelJack_Horizontal, F.Cu at (324.8, 67.0)
- added REF**: JST_PH_B4B-PH-K_1x04_P2.00mm_Vertical, Connector_JST:JST_PH_B4B-PH-K_1x04_P2.00mm_Vertical, F.Cu at (295.2, 72.5)
- added REF**: LGA-16_3x3mm_P0.5mm_LayoutBorder3x5y, Package_LGA:LGA-16_3x3mm_P0.5mm_LayoutBorder3x5y, F.Cu at (262.2, 68.8)
- added REF**: LED_0603_1608Metric, LED_SMD:LED_0603_1608Metric, F.Cu at (333.2, 67.8)
- added REF**: LED_0603_1608Metric, LED_SMD:LED_0603_1608Metric, F.Cu at (341.8, 32.5)
- added REF**: C_0603_1608Metric, Capacitor_SMD:C_0603_1608Metric, F.Cu at (325.5, 35.5)
- added REF**: QFN-16-1EP_3x3mm_Pitch0.5mm, GiraffeTech-Maxim:QFN-16-1EP_3x3mm_Pitch0.5mm, F.Cu at (315.2, 36.0)
- added REF**: Dinkle_ED350V_2Pins_Pitch3.5mm, GiraffeTech-Connector:TerminalBlock_Dinkle_ED350V_1x02_P3.50mm_Horizontal, F.Cu at (333.2, 77.5)
- added REF**: Buzzer_12x9.5RM7.6, Buzzer_Beeper:Buzzer_12x9.5RM7.6, F.Cu at (322.6, 54.8)
- added REF**: C_0603_1608Metric, Capacitor_SMD:C_0603_1608Metric, F.Cu at (337.8, 70.8)
- added REF**: C_0603_1608Metric, Capacitor_SMD:C_0603_1608Metric, F.Cu at (340.8, 70.0)
- added REF**: R_0603_1608Metric, Resistor_SMD:R_0603_1608Metric, F.Cu at (328.8, 38.2)
- added REF**: MountingHole_3.5mm, MountingHole:MountingHole_3.5mm, F.Cu at (262.8, 77.0)
- added REF**: ESP32-WROOM-32_ButtLess, GiraffeTech-NodeMCU:ESP32-WROOM-32_ButtLess, F.Cu at (179.5, 51.0)
- added REF**: JST_PH_B4B-PH-K_1x04_P2.00mm_Vertical, Connector_JST:JST_PH_B4B-PH-K_1x04_P2.00mm_Vertical, F.Cu at (276.5, 72.5)
- added REF**: SW_SPST_B3S-1000, Button_Switch_SMD:SW_SPST_B3S-1000, F.Cu at (272.5, 26.2)
- added REF**: SOT-23-6, Package_TO_SOT_SMD:SOT-23-6, F.Cu at (328.8, 35.5)
- added REF**: MountingHole_3.5mm, MountingHole:MountingHole_3.5mm, F.Cu at (340.8, 77.0)
- added REF**: PinHeader_2x03_P2.54mm_Vertical, Connector_PinHeader_2.54mm:PinHeader_2x03_P2.54mm_Vertical, F.Cu at (301.2, 28.0)
- added REF**: DINKLE_EK500V-2P, GiraffeTech-Connector:DINKLE_EK500V-2P, F.Cu at (331.2, 26.0)
- added REF**: Buzzer_CUI_CPT-9019S-SMT, Buzzer_Beeper:Buzzer_CUI_CPT-9019S-SMT, F.Cu at (354.0, 61.0)
- added REF**: QFN-16-1EP_3x3mm_Pitch0.5mm, GiraffeTech-Maxim:QFN-16-1EP_3x3mm_Pitch0.5mm, F.Cu at (292.2, 33.2)
- added REF**: SW_SPST_B3S-1000, Button_Switch_SMD:SW_SPST_B3S-1000, F.Cu at (282.2, 26.2)
- added REF**: LED_WS2812B_PLCC4_5.0x5.0mm_P3.2mm, LED_SMD:LED_WS2812B_PLCC4_5.0x5.0mm_P3.2mm, F.Cu at (272.5, 35.5)
- added REF**: C_0603_1608Metric, Capacitor_SMD:C_0603_1608Metric, F.Cu at (277.5, 29.8)
- added REF**: MountingHole_3.5mm, MountingHole:MountingHole_3.5mm, F.Cu at (340.8, 25.0)
- added REF**: DINKLE_EK500V-2P, GiraffeTech-Connector:DINKLE_EK500V-2P, F.Cu at (320.5, 26.0)
- added REF**: TQFP-64_10x10mm_P0.5mm, Package_QFP:TQFP-64_10x10mm_P0.5mm, F.Cu at (301.8, 51.0)
- added REF**: Sensirion_SHT3x, GiraffeTech-Sensiroin:Sensirion_SHT3x, F.Cu at (262.2, 64.0)
- added REF**: MountingHole_3.5mm, MountingHole:MountingHole_3.5mm, F.Cu at (262.8, 25.0)
- added REF**: LED_WS2812B_PLCC4_5.0x5.0mm_P3.2mm, LED_SMD:LED_WS2812B_PLCC4_5.0x5.0mm_P3.2mm, F.Cu at (282.2, 35.5)
- added REF**: MagneticBuzzer_CUI_CMT-8504-100-SMT, Buzzer_Beeper:MagneticBuzzer_CUI_CMT-8504-100-SMT, F.Cu at (354.8, 48.4)
- added REF**: R_0603_1608Metric, Resistor_SMD:R_0603_1608Metric, F.Cu at (333.2, 38.2)
- added REF**: JST_PH_B4B-PH-K_1x04_P2.00mm_Vertical, Connector_JST:JST_PH_B4B-PH-K_1x04_P2.00mm_Vertical, F.Cu at (301.5, 72.5)
- added REF**: Symbol_Barrel_Polarity, Symbol:Symbol_Barrel_Polarity, F.Cu at (343.2, 67.5)
- added REF**: PinHeader_1x03_P2.54mm_Vertical, Connector_PinHeader_2.54mm:PinHeader_1x03_P2.54mm_Vertical, F.Cu at (260.8, 33.0)
- added REF**: ESP32-WROOM-32_ButtLess, GiraffeTech-NodeMCU:ESP32-WROOM-32_ButtLess, F.Cu at (274.8, 51.0)
- added REF**: C_0603_1608Metric, Capacitor_SMD:C_0603_1608Metric, F.Cu at (287.5, 32.2)
- added REF**: SOT-23-5, Package_TO_SOT_SMD:SOT-23-5, F.Cu at (337.8, 67.8)
- added REF**: USB_Micro-B_Amphenol_10118193_Horizontal, GiraffeTech-Connector:USB_Micro-B_Amphenol_10118193_Horizontal, F.Cu at (343.2, 51.0)
- added REF**: C_0603_1608Metric, Capacitor_SMD:C_0603_1608Metric, F.Cu at (324.0, 35.5)
- added REF**: C_0603_1608Metric, Capacitor_SMD:C_0603_1608Metric, F.Cu at (311.5, 36.0)
- added REF**: DINKLE_EK500V-2P, GiraffeTech-Connector:DINKLE_EK500V-2P, F.Cu at (309.8, 26.0)
- added REF**: C_0603_1608Metric, Capacitor_SMD:C_0603_1608Metric, F.Cu at (310.0, 36.0)
- added REF**: JST_PH_B4B-PH-K_1x04_P2.00mm_Vertical, Connector_JST:JST_PH_B4B-PH-K_1x04_P2.00mm_Vertical, F.Cu at (289.0, 72.5)
- added REF**: SOT-23-6, Package_TO_SOT_SMD:SOT-23-6, F.Cu at (333.2, 35.5)
- added REF**: JST_PH_B4B-PH-K_1x04_P2.00mm_Vertical, Connector_JST:JST_PH_B4B-PH-K_1x04_P2.00mm_Vertical, F.Cu at (282.8, 72.5)
- added REF**: Dinkle_ED350V_2Pins_Pitch3.5mm, GiraffeTech-Connector:TerminalBlock_Dinkle_ED350V_1x02_P3.50mm_Horizontal, F.Cu at (291.0, 24.5)
- added REF**: C_0603_1608Metric, Capacitor_SMD:C_0603_1608Metric, F.Cu at (340.8, 66.8)
- added REF**: C_0603_1608Metric, Capacitor_SMD:C_0603_1608Metric, F.Cu at (319.0, 36.0)
- added REF**: C_0603_1608Metric, Capacitor_SMD:C_0603_1608Metric, F.Cu at (320.5, 36.0)
- added REF**: R_0603_1608Metric, Resistor_SMD:R_0603_1608Metric, F.Cu at (233.5, 38.2)
- added REF**: R_0603_1608Metric, Resistor_SMD:R_0603_1608Metric, F.Cu at (238.0, 38.2)
- added REF**: C_0603_1608Metric, Capacitor_SMD:C_0603_1608Metric, F.Cu at (267.8, 29.8)
- added REF**: LED_0603_1608Metric, LED_SMD:LED_0603_1608Metric, F.Cu at (246.5, 32.5)
- added REF**: C_0603_1608Metric, Capacitor_SMD:C_0603_1608Metric, F.Cu at (245.5, 66.8)
- added REF**: C_0603_1608Metric, Capacitor_SMD:C_0603_1608Metric, F.Cu at (245.5, 70.0)
- added REF**: C_0603_1608Metric, Capacitor_SMD:C_0603_1608Metric, F.Cu at (242.8, 35.5)
- added REF**: C_0603_1608Metric, Capacitor_SMD:C_0603_1608Metric, F.Cu at (241.2, 35.5)
- added REF**: C_0603_1608Metric, Capacitor_SMD:C_0603_1608Metric, F.Cu at (228.8, 35.5)
- added REF**: C_0603_1608Metric, Capacitor_SMD:C_0603_1608Metric, F.Cu at (230.2, 35.5)
- added REF**: C_0603_1608Metric, Capacitor_SMD:C_0603_1608Metric, F.Cu at (225.2, 36.0)
- added REF**: C_0603_1608Metric, Capacitor_SMD:C_0603_1608Metric, F.Cu at (223.8, 36.0)
- added REF**: C_0603_1608Metric, Capacitor_SMD:C_0603_1608Metric, F.Cu at (214.8, 36.0)
- added REF**: GTK_TFMS08TK-PP-02, GiraffeTech-Connector:GTK_TFMS08TK-PP-02, F.Cu at (306.0, 76.0)
- added REF**: C_0603_1608Metric, Capacitor_SMD:C_0603_1608Metric, F.Cu at (216.2, 36.0)
- added REF**: JST_PH_B4B-PH-K_1x04_P2.00mm_Vertical, Connector_JST:JST_PH_B4B-PH-K_1x04_P2.00mm_Vertical, F.Cu at (206.2, 72.5)
- added REF**: Dinkle_ED350V_2Pins_Pitch3.5mm, GiraffeTech-Connector:TerminalBlock_Dinkle_ED350V_1x02_P3.50mm_Horizontal, F.Cu at (195.8, 24.5)
- added REF**: JST_PH_B4B-PH-K_1x04_P2.00mm_Vertical, Connector_JST:JST_PH_B4B-PH-K_1x04_P2.00mm_Vertical, F.Cu at (200.0, 72.5)
- added REF**: Dinkle_ED350V_2Pins_Pitch3.5mm, GiraffeTech-Connector:TerminalBlock_Dinkle_ED350V_1x02_P3.50mm_Horizontal, F.Cu at (238.0, 77.5)
- added REF**: JST_PH_B4B-PH-K_1x04_P2.00mm_Vertical, Connector_JST:JST_PH_B4B-PH-K_1x04_P2.00mm_Vertical, F.Cu at (193.8, 72.5)
- added REF**: PinHeader_2x03_P2.54mm_Vertical, Connector_PinHeader_2.54mm:PinHeader_2x03_P2.54mm_Vertical, F.Cu at (206.0, 28.0)
- added REF**: JST_PH_B4B-PH-K_1x04_P2.00mm_Vertical, Connector_JST:JST_PH_B4B-PH-K_1x04_P2.00mm_Vertical, F.Cu at (181.2, 72.5)
- added REF**: Symbol_Barrel_Polarity, Symbol:Symbol_Barrel_Polarity, F.Cu at (248.0, 67.5)
- added REF**: TQFP-64_10x10mm_P0.5mm, Package_QFP:TQFP-64_10x10mm_P0.5mm, F.Cu at (206.5, 51.0)
- added REF**: R_0603_1608Metric, Resistor_SMD:R_0603_1608Metric, F.Cu at (269.2, 64.2)
- added REF**: PinHeader_1x03_P2.54mm_Vertical, Connector_PinHeader_2.54mm:PinHeader_1x03_P2.54mm_Vertical, F.Cu at (165.5, 33.0)
- added REF**: JST_PH_B4B-PH-K_1x04_P2.00mm_Vertical, Connector_JST:JST_PH_B4B-PH-K_1x04_P2.00mm_Vertical, F.Cu at (175.0, 72.5)
- added REF**: Sensirion_SHT3x, GiraffeTech-Sensiroin:Sensirion_SHT3x, F.Cu at (167.0, 64.0)
- added REF**: BarrelJack_Horizontal, Connector_BarrelJack:BarrelJack_Horizontal, F.Cu at (229.5, 67.0)
- added REF**: DINKLE_EK500V-2P, GiraffeTech-Connector:DINKLE_EK500V-2P, F.Cu at (225.2, 26.0)
- added REF**: SOT-23-6, Package_TO_SOT_SMD:SOT-23-6, F.Cu at (238.0, 35.5)
- added REF**: SW_SPST_B3S-1000, Button_Switch_SMD:SW_SPST_B3S-1000, F.Cu at (177.2, 26.2)
- added REF**: LED_0603_1608Metric, LED_SMD:LED_0603_1608Metric, F.Cu at (238.0, 67.8)
- added REF**: PinHeader_2x05_P1.27mm_Vertical, Connector_PinHeader_1.27mm:PinHeader_2x05_P1.27mm_Vertical, F.Cu at (223.5, 51.5)
- added REF**: LGA-16_3x3mm_P0.5mm_LayoutBorder3x5y, Package_LGA:LGA-16_3x3mm_P0.5mm_LayoutBorder3x5y, F.Cu at (167.0, 68.8)
- added REF**: R_0603_1608Metric, Resistor_SMD:R_0603_1608Metric, F.Cu at (269.2, 62.8)
- added REF**: C_0603_1608Metric, Capacitor_SMD:C_0603_1608Metric, F.Cu at (192.2, 32.2)
- added REF**: LED_WS2812B_PLCC4_5.0x5.0mm_P3.2mm, LED_SMD:LED_WS2812B_PLCC4_5.0x5.0mm_P3.2mm, F.Cu at (187.0, 35.5)
- added REF**: R_0603_1608Metric, Resistor_SMD:R_0603_1608Metric, F.Cu at (174.0, 62.8)
- added REF**: SOT-23-5, Package_TO_SOT_SMD:SOT-23-5, F.Cu at (242.5, 67.8)
- added REF**: DINKLE_EK500V-2P, GiraffeTech-Connector:DINKLE_EK500V-2P, F.Cu at (236.0, 26.0)
- added REF**: C_0603_1608Metric, Capacitor_SMD:C_0603_1608Metric, F.Cu at (242.5, 70.8)
- added REF**: QFN-16-1EP_3x3mm_Pitch0.5mm, GiraffeTech-Maxim:QFN-16-1EP_3x3mm_Pitch0.5mm, F.Cu at (220.0, 36.0)
- added REF**: MountingHole_3.5mm, MountingHole:MountingHole_3.5mm, F.Cu at (167.5, 77.0)
- added REF**: MountingHole_3.5mm, MountingHole:MountingHole_3.5mm, F.Cu at (245.5, 25.0)
- added REF**: LED_WS2812B_PLCC4_5.0x5.0mm_P3.2mm, LED_SMD:LED_WS2812B_PLCC4_5.0x5.0mm_P3.2mm, F.Cu at (177.2, 35.5)
- moved REF** 76.1 mm to (187.5, 72.5)
- moved REF** 12.8 mm to (120.8, 67.0)
Other:
- board size 201 x 139 mm -> 279.8 x 139 mm
- board text added: "D2 A1"
- board text added: "D3 A2"
- board text added: "D4 A3"
- board text added: "PWR"
- board text added: "RESET"
