File: MP_SamBaseBoard_V1/MP_SamBaseBoard_V1.kicad_pcb (KiCad board)
At the start: 4 copper layers, 80 x 60 mm, 132 parts, among them J1 MA_CONN, J10 P1_CONN, J11 I2C_CONN, J12 I2C_CONN, J13 SAM_SWD, J14 WS2812_EXT, J15 PWR_JACK, J16 USB_B_Micro, J17 BATT_CONN, J2 MB_CONN, J3 Adafruit_Feather_CONN, J4 LOAD_CONN, J5 SPEAKER, J7 SERVO_CONN, J8 P3_CONN, J9 P2_CONN, Q1 DMP3098L, Q2 ALS-PT19-315C/L177/TR8, Q3 BSS138-7-F, SW1 RESET, SW2 3v3_PWR_SW, SW3 SW1, SW4 SW2, U1 ESP32-WROOM-32, U10 KXTJ3-1057, U11 IRFHM3911PbF, U12 IRFHM9331PbF, U13 SST25VF016B-50-4C-S2AF, U14 IRFHM9331PbF, U2 ATSAMD51J19A-A, U3 74LVC1G125, U4 TPS62135, U5 PAM8301, U6 BQ24075, U7 DRV8833RTY, U8 Sensirion_SHT3x, U9 LD39200PU33R, Y1 Crystal

Commit message: finalize 1
Parts:
- moved C31 25.9 mm to (189.8, 100.5), turned to 180 degrees
- moved U10 25.8 mm to (188.8, 97.8), turned to 270 degrees
- moved C30 21.8 mm to (192.8, 95.2)
- moved Q2 8.19 mm to (146.2, 90.2), turned to 270 degrees
- moved R20 4.51 mm to (149.8, 90.2), turned to 90 degrees
- moved MK1 3.78 mm to (153.5, 90.3), turned to 180 degrees
- moved C19 2.92 mm to (151.2, 90.2), turned to 90 degrees
- moved R1 1.60 mm to (144.5, 90.2), turned to 270 degrees
Connections:
- U10 pad 3: +3V3 -> (no net)
- U10 pad 7: +3V3 -> (no net)
Routing:
- net Adf_A4: track 14.9 -> 50.2 mm, vias 1 -> 2
- net D0_RxD0: track 66.4 -> 98.9 mm
- net D1_TxD0: track 69.0 -> 95.9 mm
- net Adf_A3: track 20.2 -> 44.6 mm
- net +3V3: track 424.5 -> 446.9 mm
- net Adf_A1_DAC1: track 26.5 -> 40.5 mm
- net Adf_A5: track 13.6 -> 26.3 mm
- net GND: track 58.2 -> 65.1 mm, vias 178 -> 188
- net ~RESET: track 69.0 -> 73.6 mm
- net ESP_CS-D8: track 40.9 -> 43.9 mm
- net I2C_SCL: track 97.1 -> 99.8 mm, vias 1 -> 2
- net I2C_SDA: track 104.3 -> 106.7 mm, vias 1 -> 2
- net Adf_A2: track 48.3 -> 46.4 mm
- net SAM_RxLED: track 33.7 -> 33.0 mm
- net USB_ID: track 44.0 -> 44.7 mm
Other:
- board text added: "LIGHT"
