File: MP_SamBaseBoard_V1/MP_SamBaseBoard_V1.sch (KiCad schematic (older format))
At the start: 128 parts, among them J1 MA_CONN, J10 P1_CONN, J11 I2C_CONN, J12 I2C_CONN, J13 SAM_SWD, J14 WS2812_EXT, J15 PWR_JACK, J16 USB_B_Micro, J17 BATT_CONN, J2 MB_CONN, J3 Adafruit_Feather_CONN, J4 LOAD_CONN, J5 SPEAKER, J7 SERVO_CONN, J8 P3_CONN, J9 P2_CONN, Q1 DMP3098L, Q2 ALS-PT19-315C/L177/TR8, SW1 RESET, SW2 3v3_PWR_SW, SW3 SW1, SW4 SW2, U1 ESP32-WROOM-32, U10 KXTJ3-1057, U11 IRFHM9331PbF, U13 SST25VF016B-50-4C-S2AF, U2 ATSAMD51J19A-A, U3 74LVC1G125, U4 TPS62135, U5 PAM8301, U6 BQ24075, U7 DRV8833RTY, U8 Sensirion_SHT3x, U9 LD39200PU33R, Y1 Crystal

Commit message: update
Parts:
- removed R33, R34: R_USB, Resistor_SMD:R_0603_1608Metric, symbol Device:R_Small
- added C32: 0.1uF, Capacitor_SMD:C_0603_1608Metric, symbol Device:C_Small
- J4: footprint GiraffeTech-Connector:TerminalBlock_DEGSON_DG300-5-3pol -> GiraffeTech-Connector:TerminalBlock_Dinkle_ED350V_1x03_P3.50mm_Horizontal
Connections:
- net ESP_CS is gone; now on net ESP_CS-D8: R1.2
- net +3V3: now also R23.1, C32.1; no longer D3.2 (A)
- net GND: now also D3.1 (K), J4.1 (Pin_1), C32.2; no longer J4.3 (Pin_3), R23.2
- net USB_DM: now also J16.2 (D-)
- net USB_DP: now also J16.3 (D+)
- net VIN: now also J4.3 (Pin_3); no longer J4.1 (Pin_1)
- net at C24.2, U7.16 (AOUT1): now also J1.1 (Pin_1); no longer J1.2 (Pin_2)
- net at C24.1, U7.2 (AOUT2): now also J1.2 (Pin_2); no longer J1.1 (Pin_1)
- net at C25.2, U7.3 (BOUT2): now also J2.1 (Pin_1); no longer J2.2 (Pin_2)
- net at C25.1, U7.5 (BOUT1): now also J2.2 (Pin_2); no longer J2.1 (Pin_1)
- new net: D3.2 (A), R23.2
Other:
- moved on the sheet: D3, J16, R23
Changed lines of the file:
@@
 Text GLabel 3200 3400 2    50   Input ~ 0
 BLUE_LED
-Text GLabel 900  1350 3    50   Input ~ 0
-ESP_CS
 $Comp
 L Device:R_Small R1
@@
 L Connector_Generic:Conn_01x02 J2
 U 1 1 5F0DEFB5
-P 3400 8650
-F 0 "J2" H 3480 8642 50  0000 L CNN
-F 1 "MB_CONN" H 3480 8551 50  0000 L CNN
-F 2 "GiraffeTech-Connector:TerminalBlock_Dinkle_ED350V_1x02_P3.50mm_Horizontal" H 3400 8650 50  0001 C CNN
-F 3 "~" H 3400 8650 50  0001 C CNN
-	1    3400 8650
-	1    0    0    -1
+P 3400 8750
+F 0 "J2" H 3480 8742 50  0000 L CNN
+F 1 "MB_CONN" H 3480 8651 50  0000 L CNN
+F 2 "GiraffeTech-Connector:TerminalBlock_Dinkle_ED350V_1x02_P3.50mm_Horizontal" H 3400 8750 50  0001 C CNN
+F 3 "~" H 3400 8750 50  0001 C CNN
+	1    3400 8750
+	1    0    0    1
 $EndComp
 $Comp
@@
 	11450 4700 11450 4800
 $Comp
-L Switch:SW_Push SW3
-U 1 1 5F59416F
-P 10350 8050
-F 0 "SW3" H 10350 8335 50  0000 C CNN
-F 1 "SW1" H 10350 8244 50  0000 C CNN
-F 2 "GiraffeTech-Electromechanical:SW_Push_TS-1145A-B-A" H 10350 8250 50  0001 C CNN
-F 3 "~" H 10350 8250 50  0001 C CNN
-	1    10350 8050
-	1    0    0    -1
-$EndComp
-$Comp
-L Switch:SW_Push SW4
-U 1 1 5F595E63
-P 10350 8500
-F 0 "SW4" H 10350 8785 50  0000 C CNN
-F 1 "SW2" H 10350 8694 50  0000 C CNN
-F 2 "GiraffeTech-Electromechanical:SW_Push_TS-1145A-B-A" H 10350 8700 50  0001 C CNN
-F 3 "~" H 10350 8700 50  0001 C CNN
-	1    10350 8500
-	1    0    0    -1
-$EndComp
-$Comp
-L power:GND #PWR0225
-U 1 1 5F5969E8
-P 10650 8600
-F 0 "#PWR0225" H 10650 8350 50  0001 C CNN
-F 1 "GND" H 10655 8427 50  0000 C CNN
-F 2 "" H 10650 8600 50  0001 C CNN
-F 3 "" H 10650 8600 50  0001 C CNN
-	1    10650 8600
-	1    0    0    -1
-$EndComp
-Wire Wire Line
-	10550 8050 10650 8050
-Wire Wire Line
-	10650 8050 10650 8500
-Wire Wire Line
-	10550 8500 10650 8500
-Connection ~ 10650 8500
-Wire Wire Line
-	10650 8500 10650 8600
-Wire Wire Line
-	10050 8500 10150 8500
-Wire Wire Line
-	10050 8050 10150 8050
-$Comp
 L LED:WS2812B D6
 U 1 1 5EC19F88
@@
 L Connector:USB_B_Micro J16
 U 1 1 5ED07E36
-P 4200 5500
-F 0 "J16" H 4257 5967 50  0000 C CNN
-F 1 "USB_B_Micro" H 4257 5876 50  0000 C CNN
-F 2 "GiraffeTech-Connector:USB_Micro-B_Amphenol_10118193_Horizontal" H 4350 5450 50  0001 C CNN
-F 3 "~" H 4350 5450 50  0001 C CNN
-	1    4200 5500
+P 4250 5350
+F 0 "J16" H 4307 5817 50  0000 C CNN
+F 1 "USB_B_Micro" H 4307 5726 50  0000 C CNN
+F 2 "GiraffeTech-Connector:USB_Micro-B_Amphenol_10118193_Horizontal" H 4400 5300 50  0001 C CNN
+F 3 "~" H 4400 5300 50  0001 C CNN
+	1    4250 5350
 	1    0    0    -1
 $EndComp
@@
 L power:GND #PWR0233
 U 1 1 5ED9F1BF
-P 4150 6000
-F 0 "#PWR0233" H 4150 5750 50  0001 C CNN
-F 1 "GND" H 4155 5827 50  0000 C CNN
-F 2 "" H 4150 6000 50  0001 C CNN
-F 3 "" H 4150 6000 50  0001 C CNN
-	1    4150 6000
+P 4200 5850
+F 0 "#PWR0233" H 4200 5600 50  0001 C CNN
+F 1 "GND" H 4205 5677 50  0000 C CNN
+F 2 "" H 4200 5850 50  0001 C CNN
+F 3 "" H 4200 5850 50  0001 C CNN
+	1    4200 5850
 	1    0    0    -1
 $EndComp
 Wire Wire Line
-	4100 5900 4100 5950
+	4150 5750 4150 5800
 Wire Wire Line
-	4100 5950 4150 5950
+	4150 5800 4200 5800
 Wire Wire Line
-	4200 5950 4200 5900
+	4250 5800 4250 5750
 Wire Wire Line
-	4150 6000 4150 5950
-Connection ~ 4150 5950
+	4200 5850 4200 5800
+Connection ~ 4200 5800
 Wire Wire Line
-	4150 5950 4200 5950
+	4200 5800 4250 5800
 $Comp
 L power:VBUS #PWR0234
 U 1 1 5EE6E443
-P 4600 5200
-F 0 "#PWR0234" H 4600 5050 50  0001 C CNN
-F 1 "VBUS" H 4615 5373 50  0000 C CNN
-F 2 "" H 4600 5200 50  0001 C CNN
-F 3 "" H 4600 5200 50  0001 C CNN
-	1    4600 5200
-	1    0    0    -1
+P 4650 5150
+F 0 "#PWR0234" H 4650 5000 50  0001 C CNN
+F 1 "VBUS" H 4665 5323 50  0000 C CNN
+F 2 "" H 4650 5150 50  0001 C CNN
+F 3 "" H 4650 5150 50  0001 C CNN
+	1    4650 5150
+	0    1    1    0
 $EndComp
 Wire Wire Line
-	4500 5300 4600 5300
-Wire Wire Line
-	4600 5300 4600 5200
+	4550 5150 4650 5150
 Text Notes 8250 7800 0    50   ~ 0
 PIEZO BUZZER
-$Comp
-L Device:R_Small R33
-U 1 1 5EF0CCE5
-P 4850 5400
-F 0 "R33" V 4654 5400 50  0000 C CNN
-F 1 "R_USB" V 4745 5400 50  0000 C CNN
-F 2 "Resistor_SMD:R_0603_1608Metric" H 4850 5400 50  0001 C CNN
-F 3 "~" H 4850 5400 50  0001 C CNN
-	1    4850 5400
-	0    1    1    0
-$EndComp
-$Comp
-L Device:R_Small R34
-U 1 1 5EF0D3FD
-P 4850 5700
-F 0 "R34" V 4654 5700 50  0000 C CNN
-F 1 "R_USB" V 4745 5700 50  0000 C CNN
-F 2 "Resistor_SMD:R_0603_1608Metric" H 4850 5700 50  0001 C CNN
-F 3 "~" H 4850 5700 50  0001 C CNN
-	1    4850 5700
-	0    1    1    0
-$EndComp
-Wire Wire Line
-	4500 5500 4650 5500
-Wire Wire Line
-	4650 5500 4650 5400
-Wire Wire Line
-	4650 5400 4750 5400
-Wire Wire Line
-	4500 5600 4650 5600
-Wire Wire Line
-	4650 5600 4650 5700
-Wire Wire Line
-	4650 5700 4750 5700
-Text GLabel 5050 5700 2    50   Input ~ 0
+Text GLabel 4650 5450 2    50   Input ~ 0
 USB_DM
-Text GLabel 5050 5400 2    50   Input ~ 0
+Text GLabel 4650 5350 2    50   Input ~ 0
 USB_DP
 Wire Wire Line
-	4950 5400 5050 5400
+	4550 5350 4650 5350
 Wire Wire Line
-	4950 5700 5050 5700
+	4550 5450 4650 5450
 $Comp
 L Device:R_Small R35
@@
 Wire Wire Line
 	14850 2550 15000 2550
-Text GLabel 4700 5900 2    50   Input ~ 0
+Text GLabel 4650 5550 2    50   Input ~ 0
 USB_ID
 Wire Wire Line
-	4500 5700 4600 5700
-Wire Wire Line
-	4600 5700 4600 5900
-Wire Wire Line
-	4600 5900 4700 5900
+	4550 5550 4650 5550
 $Comp
 L power:+BATT #PWR0235
@@
 L Connector_Generic:Conn_01x02 J1
 U 1 1 5F0DE9E4
-P 3400 7350
-F 0 "J1" H 3480 7342 50  0000 L CNN
-F 1 "MA_CONN" H 3480 7251 50  0000 L CNN
-F 2 "GiraffeTech-Connector:TerminalBlock_Dinkle_ED350V_1x02_P3.50mm_Horizontal" H 3400 7350 50  0001 C CNN
-F 3 "~" H 3400 7350 50  0001 C CNN
-	1    3400 7350
-	1    0    0    1
+P 3400 7250
+F 0 "J1" H 3480 7242 50  0000 L CNN
+F 1 "MA_CONN" H 3480 7151 50  0000 L CNN
+F 2 "GiraffeTech-Connector:TerminalBlock_Dinkle_ED350V_1x02_P3.50mm_Horizontal" H 3400 7250 50  0001 C CNN
+F 3 "~" H 3400 7250 50  0001 C CNN
+	1    3400 7250
+	1    0    0    -1
 $EndComp
 $Comp
@@
 F 0 "J4" H 9180 10642 50  0000 L CNN
 F 1 "LOAD_CONN" H 9180 10551 50  0000 L CNN
-F 2 "GiraffeTech-Connector:TerminalBlock_DEGSON_DG300-5-3pol" H 9100 10600 50  0001 C CNN
+F 2 "GiraffeTech-Connector:TerminalBlock_Dinkle_ED350V_1x03_P3.50mm_Horizontal" H 9100 10600 50  0001 C CNN
 F 3 "~" H 9100 10600 50  0001 C CNN
 	1    9100 10600
-	1    0    0    -1
+	1    0    0    1
 $EndComp
-Text GLabel 10050 8050 0    50   Input ~ 0
-D0_RxD0
-Text GLabel 10050 8500 0    50   Input ~ 0
-D1_TxD0
-Text Notes 9950 7600 0    50   ~ 0
-PUSH BUTTON
 Text GLabel 3200 3600 2    50   Input ~ 0
 ESP_BUSY-D13
@@
 	2100 10400 2100 10500
 Wire Wire Line
-	2100 9700 2100 9800
+	2100 9700 2100 9750
 Text GLabel 1300 10000 0    50   Input ~ 0
 Adf_A0_DAC0
@@
 L Device:LED D3
 U 1 1 5EE5D35E
-P 15500 4850
-F 0 "D3" V 15539 4732 50  0000 R CNN
-F 1 "PWR_LED" V 15448 4732 50  0000 R CNN
-F 2 "LED_SMD:LED_0603_1608Metric" H 15500 4850 50  0001 C CNN
-F 3 "~" H 15500 4850 50  0001 C CNN
-	1    15500 4850
+P 15500 5150
+F 0 "D3" V 15539 5032 50  0000 R CNN
+F 1 "PWR_LED" V 15448 5032 50  0000 R CNN
+F 2 "LED_SMD:LED_0603_1608Metric" H 15500 5150 50  0001 C CNN
+F 3 "~" H 15500 5150 50  0001 C CNN
+	1    15500 5150
 	0    -1   -1   0
 $EndComp
@@
 L Device:R_Small R23
 U 1 1 5EE5E86B
-P 15500 5200
-F 0 "R23" H 15559 5246 50  0000 L CNN
-F 1 "1K" H 15559 5155 50  0000 L CNN
-F 2 "Resistor_SMD:R_0603_1608Metric" H 15500 5200 50  0001 C CNN
-F 3 "~" H 15500 5200 50  0001 C CNN
-	1    15500 5200
+P 15500 4800
+F 0 "R23" H 15559 4846 50  0000 L CNN
+F 1 "1K" H 15559 4755 50  0000 L CNN
+F 2 "Resistor_SMD:R_0603_1608Metric" H 15500 4800 50  0001 C CNN
+F 3 "~" H 15500 4800 50  0001 C CNN
+	1    15500 4800
 	1    0    0    -1
 $EndComp
 Wire Wire Line
-	15500 5000 15500 5100
-Wire Wire Line
 	15500 5300 15500 5400
 Wire Wire Line
@@
 Wire Wire Line
 	15500 4600 15500 4700
+$Comp
+L Device:C_Small C32
+U 1 1 5EF28AEF
+P 2700 9750
+F 0 "C32" H 2792 9796 50  0000 L CNN
+F 1 "0.1uF" H 2792 9705 50  0000 L CNN
+F 2 "Capacitor_SMD:C_0603_1608Metric" H 2700 9750 50  0001 C CNN
+F 3 "~" H 2700 9750 50  0001 C CNN
+	1    2700 9750
+	0    -1   -1   0
+$EndComp
+Wire Wire Line
+	2100 9750 2600 9750
+Connection ~ 2100 9750
+Wire Wire Line
+	2100 9750 2100 9800
+$Comp
+L power:GND #PWR0198
+U 1 1 5EF92CE8
+P 2900 9750
+F 0 "#PWR0198" H 2900 9500 50  0001 C CNN
+F 1 "GND" V 2905 9622 50  0000 R CNN
+F 2 "" H 2900 9750 50  0001 C CNN
+F 3 "" H 2900 9750 50  0001 C CNN
+	1    2900 9750
+	0    -1   -1   0
+$EndComp
+Wire Wire Line
+	2800 9750 2900 9750
+Text Notes 9950 7650 0    50   ~ 0
+PUSH BUTTON
+Wire Wire Line
+	10550 8050 10650 8050
+$Comp
+L Switch:SW_Push SW3
+U 1 1 5F59416F
+P 10350 8050
+F 0 "SW3" H 10350 8335 50  0000 C CNN
+F 1 "SW1" H 10350 8244 50  0000 C CNN
+F 2 "GiraffeTech-Electromechanical:SW_Push_TS-1145A-B-A" H 10350 8250 50  0001 C CNN
+F 3 "~" H 10350 8250 50  0001 C CNN
+	1    10350 8050
+	1    0    0    -1
+$EndComp
+Wire Wire Line
+	10050 8050 10150 8050
+Text GLabel 10050 8050 0    50   Input ~ 0
+D0_RxD0
+Text GLabel 10050 8500 0    50   Input ~ 0
+D1_TxD0
+Wire Wire Line
+	10050 8500 10150 8500
+$Comp
+L Switch:SW_Push SW4
+U 1 1 5F595E63
+P 10350 8500
+F 0 "SW4" H 10350 8785 50  0000 C CNN
+F 1 "SW2" H 10350 8694 50  0000 C CNN
+F 2 "GiraffeTech-Electromechanical:SW_Push_TS-1145A-B-A" H 10350 8700 50  0001 C CNN
+F 3 "~" H 10350 8700 50  0001 C CNN
+	1    10350 8500
+	1    0    0    -1
+$EndComp
+$Comp
+L power:GND #PWR0225
+U 1 1 5F5969E8
+P 10650 8600
+F 0 "#PWR0225" H 10650 8350 50  0001 C CNN
+F 1 "GND" H 10655 8427 50  0000 C CNN
+F 2 "" H 10650 8600 50  0001 C CNN
+F 3 "" H 10650 8600 50  0001 C CNN
+	1    10650 8600
+	1    0    0    -1
+$EndComp
+Wire Wire Line
+	10650 8500 10650 8600
+Wire Wire Line
+	10550 8500 10650 8500
+Connection ~ 10650 8500
+Wire Wire Line
+	10650 8050 10650 8500
+Text GLabel 900  1350 3    50   Input ~ 0
+ESP_CS-D8
+Wire Wire Line
+	15500 4900 15500 5000
 $EndSCHEMATC

Commit message: update
Parts:
- removed R12: 10K, Resistor_SMD:R_0603_1608Metric, symbol Device:R_Small
Connections:
- net 3v3_EN: now also SW2.2 (B); no longer SW2.1 (A)
- net CHG_OUT: now also SW2.3 (C); no longer SW2.2 (B)
- net GND: now also SW2.1 (A)
- no-connect marks 43 -> 42
Changed lines of the file:
@@
 	1    0    0    -1
 $EndComp
+Text GLabel 15050 6150 2    50   Input ~ 0
+CHG_OUT
+Wire Wire Line
+	14450 6050 14550 6050
 Text GLabel 14450 6050 0    50   Input ~ 0
-CHG_OUT
-Wire Wire Line
-	14450 6050 14550 6050
-Text GLabel 15050 5950 2    50   Input ~ 0
 3v3_EN
 Wire Wire Line
@@
 Wire Wire Line
 	14950 6150 15050 6150
-NoConn ~ 15050 6150
 $Comp
 L Connector_Generic:Conn_01x02 J2
@@
 U 1 1 5F3DF7A7
 P 11750 9150
-F 0 "J17" H 11668 8825 50  0000 C CNN
-F 1 "BATT_CONN" H 11668 8916 50  0000 C CNN
+F 0 "J17" H 11700 8800 50  0000 C CNN
+F 1 "BATT_CONN" H 11700 8900 50  0000 C CNN
 F 2 "GiraffeTech-Connector:TerminalBlock_Dinkle_ED350V_1x02_P3.50mm_Horizontal" H 11750 9150 50  0001 C CNN
 F 3 "~" H 11750 9150 50  0001 C CNN
@@
 Wire Wire Line
 	13150 4600 13250 4600
-Wire Wire Line
-	13850 4950 13800 4950
 $Comp
 L power:GND #PWR0136
@@
 Text GLabel 13750 4950 0    50   Input ~ 0
 3v3_EN
-$Comp
-L Device:R_Small R12
-U 1 1 5F69E03F
-P 13600 5250
-F 0 "R12" H 13659 5296 50  0000 L CNN
-F 1 "10K" H 13659 5205 50  0000 L CNN
-F 2 "Resistor_SMD:R_0603_1608Metric" H 13600 5250 50  0001 C CNN
-F 3 "~" H 13600 5250 50  0001 C CNN
-	1    13600 5250
-	1    0    0    -1
-$EndComp
-Wire Wire Line
-	13600 5150 13600 5050
-Wire Wire Line
-	13600 5050 13800 5050
-Wire Wire Line
-	13800 5050 13800 4950
-Connection ~ 13800 4950
-Wire Wire Line
-	13800 4950 13750 4950
-$Comp
-L power:GND #PWR0139
-U 1 1 5F7F177D
-P 13600 5450
-F 0 "#PWR0139" H 13600 5200 50  0001 C CNN
-F 1 "GND" H 13605 5277 50  0000 C CNN
-F 2 "" H 13600 5450 50  0001 C CNN
-F 3 "" H 13600 5450 50  0001 C CNN
-	1    13600 5450
-	1    0    0    -1
-$EndComp
-Wire Wire Line
-	13600 5350 13600 5450
 $Comp
 L Battery_Management:BQ24075 U6
@@
 Wire Wire Line
 	15500 4900 15500 5000
+$Comp
+L power:GND #PWR0199
+U 1 1 5F3984C3
+P 15050 5950
+F 0 "#PWR0199" H 15050 5700 50  0001 C CNN
+F 1 "GND" H 15055 5777 50  0000 C CNN
+F 2 "" H 15050 5950 50  0001 C CNN
+F 3 "" H 15050 5950 50  0001 C CNN
+	1    15050 5950
+	0    -1   -1   0
+$EndComp
+Wire Wire Line
+	13750 4950 13850 4950
 $EndSCHEMATC

Commit message: update
Parts:
- removed R25: 10K, Resistor_SMD:R_0603_1608Metric, symbol Device:R_Small
- removed U11: IRFHM9331PbF, GiraffeTech-IR:PQFN_3x3mm, symbol InGarage_FETs:IRFHM9331PbF
- added F?: 6V Trip 2.5A, Fuse:Fuse_1812_4532Metric, symbol Device:Polyfuse_Small
- added F?: 6V Trip 4A, Fuse:Fuse_1206_3216Metric, symbol Device:Polyfuse_Small
- added F?: 16V Trip 4A, Fuse:Fuse_1812_4532Metric, symbol Device:Polyfuse_Small
- added U?: IRFHM9331PbF, GiraffeTech-IR:PQFN_3x3mm_IRFHM9331TRPbF, symbol InGarage_FETs:IRFHM9331PbF
- added U?: IRFHM3911PbF, GiraffeTech-IR:PQFN_3x3mm_IRFHM3911PbF, symbol InGarage_FETs:IRFHM3911PbF
- R24: value 1K -> 10K
Connections:
- net +5V: now also F?.1; no longer J14.2 (Pin_2)
- net Adf_D6: now also U?.4 (GATE)
- net GND: now also R24.1, U?.1 (SOURCE), U?.2 (SOURCE), U?.3 (SOURCE), U?.4 (GATE)
- net VBUS: now also F?.1; no longer J16.1 (VBUS)
- net VIN: now also U?.1 (SOURCE), U?.2 (SOURCE), U?.3 (SOURCE); no longer J15.1, J4.3 (Pin_3)
- net at J4.2 (Pin_2): now also U?.5 (DRAIN), U?.6 (DRAIN), U?.7 (DRAIN), U?.8 (DRAIN)
- new net: F?.2, J16.1 (VBUS)
- new net: F?.2, J14.2 (Pin_2)
- new net: F?.2, J4.3 (Pin_3)
- new net VIN_RAW: F?.1, J15.1, U?.5 (DRAIN), U?.6 (DRAIN), U?.7 (DRAIN), U?.8 (DRAIN)
Other:
- moved on the sheet: C17, C21, C26, D1, D2, J15, J17, J4, R11, R13, R14, R15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
