File: MP_SamBaseBoard_V1_DraftDesign/MP_SamBaseBoard_V1.sch (KiCad schematic (older format))
At the start: 9 parts, among them U1 ESP32-WROOM-32, U2 ATSAMD51J19A-A

Commit message: update
Parts:
- added L1: 10uH, symbol Device:L_Small
- added Q1: DMP3098L, Package_TO_SOT_SMD:SOT-23, symbol Device:Q_PMOS_GSD
- added R2, R3, R4, R5: 10k, Resistor_SMD:R_0603_1608Metric, symbol Device:R_Small
- added U3: 74LVC1G125, symbol 74xGxx:74LVC1G125
Connections:
- net labels added: +3V3_FTDI, +5V, USB_PWR_SEL, VBUS, VIN, VSW
- net labels removed: +VSW, PWR_SEL
- wire segments 139 -> 157
Changed lines of the file:
@@
 	8000 1850 8000 2050
-$Comp
-L power:+VSW #PWR0104
-U 1 1 5EA74FF2
-P 7750 1850
-F 0 "#PWR0104" H 7750 1700 50  0001 C CNN
-F 1 "+VSW" H 7765 2023 50  0000 C CNN
-F 2 "" H 7750 1850 50  0001 C CNN
-F 3 "" H 7750 1850 50  0001 C CNN
-	1    7750 1850
-	1    0    0    -1
-$EndComp
-Wire Wire Line
-	7750 1850 7750 1950
-Wire Wire Line
-	7750 1950 7900 1950
-Wire Wire Line
-	7900 1950 7900 2050
 $Comp
 L Device:C_Small C3
@@
 D1_TxD0
 Text GLabel 9100 3250 2    50   Input ~ 0
-PWR_SEL
+USB_PWR_SEL
 Text GLabel 7500 4850 0    50   Input ~ 0
 USB_DM
@@
 SWDIO
 NoConn ~ 7500 3950
+Text GLabel 7900 1850 1    50   Input ~ 0
+VSW
+Wire Wire Line
+	7900 1850 7900 2050
+Text GLabel 9250 1650 2    50   Input ~ 0
+VDD-CORE
+Text GLabel 8750 1650 0    50   Input ~ 0
+VSW
+$Comp
+L Device:L_Small L1
+U 1 1 5EA9BB1E
+P 9000 1650
+F 0 "L1" V 9185 1650 50  0000 C CNN
+F 1 "10uH" V 9094 1650 50  0000 C CNN
+F 2 "" H 9000 1650 50  0001 C CNN
+F 3 "~" H 9000 1650 50  0001 C CNN
+	1    9000 1650
+	0    -1   -1   0
+$EndComp
+Wire Wire Line
+	8750 1650 8900 1650
+Wire Wire Line
+	9100 1650 9250 1650
+$Comp
+L 74xGxx:74LVC1G125 U3
+U 1 1 5EAA1E21
+P 12500 1600
+F 0 "U3" H 12475 1333 50  0000 C CNN
+F 1 "74LVC1G125" H 12475 1424 50  0000 C CNN
+F 2 "" H 12500 1600 50  0001 C CNN
+F 3 "http://www.ti.com/lit/sg/scyt129e/scyt129e.pdf" H 12500 1600 50  0001 C CNN
+	1    12500 1600
+	-1   0    0    1
+$EndComp
+$Comp
+L Device:R_Small R3
+U 1 1 5EAA6919
+P 11500 1400
+F 0 "R3" H 11441 1354 50  0000 R CNN
+F 1 "10k" H 11441 1445 50  0000 R CNN
+F 2 "Resistor_SMD:R_0603_1608Metric" H 11500 1400 50  0001 C CNN
+F 3 "~" H 11500 1400 50  0001 C CNN
+	1    11500 1400
+	-1   0    0    1
+$EndComp
+$Comp
+L Device:R_Small R4
+U 1 1 5EAADDE8
+P 11500 1800
+F 0 "R4" H 11441 1754 50  0000 R CNN
+F 1 "10k" H 11441 1845 50  0000 R CNN
+F 2 "Resistor_SMD:R_0603_1608Metric" H 11500 1800 50  0001 C CNN
+F 3 "~" H 11500 1800 50  0001 C CNN
+	1    11500 1800
+	-1   0    0    1
+$EndComp
+$Comp
+L Device:R_Small R2
+U 1 1 5EAAE565
+P 10400 1450
+F 0 "R2" H 10341 1404 50  0000 R CNN
+F 1 "10k" H 10341 1495 50  0000 R CNN
+F 2 "Resistor_SMD:R_0603_1608Metric" H 10400 1450 50  0001 C CNN
+F 3 "~" H 10400 1450 50  0001 C CNN
+	1    10400 1450
+	-1   0    0    1
+$EndComp
+Text GLabel 13100 1600 2    50   Input ~ 0
+USB_PWR_SEL
+$Comp
+L Device:R_Small R5
+U 1 1 5EAC0BCE
+P 12950 1350
+F 0 "R5" H 12891 1304 50  0000 R CNN
+F 1 "10k" H 12891 1395 50  0000 R CNN
+F 2 "Resistor_SMD:R_0603_1608Metric" H 12950 1350 50  0001 C CNN
+F 3 "~" H 12950 1350 50  0001 C CNN
+	1    12950 1350
+	-1   0    0    1
+$EndComp
+Wire Wire Line
+	12800 1600 12950 1600
+Wire Wire Line
+	12950 1600 12950 1450
+Wire Wire Line
+	12950 1600 13100 1600
+Connection ~ 12950 1600
+$Comp
+L InGarage_Power:+3V3_FTDI #PWR0104
+U 1 1 5EACFBB5
+P 12950 1150
+F 0 "#PWR0104" H 12950 1000 50  0001 C CNN
+F 1 "+3V3_FTDI" H 12965 1323 50  0000 C CNN
+F 2 "" H 12950 1150 50  0001 C CNN
+F 3 "" H 12950 1150 50  0001 C CNN
+	1    12950 1150
+	1    0    0    -1
+$EndComp
+Wire Wire Line
+	12950 1150 12950 1250
+Wire Wire Line
+	12500 1800 12500 1900
+Wire Wire Line
+	12500 1900 12950 1900
+Wire Wire Line
+	12950 1900 12950 1600
+$Comp
+L Device:Q_PMOS_GSD Q1
+U 1 1 5EAEFB40
+P 12000 1250
+F 0 "Q1" V 12342 1250 50  0000 C CNN
+F 1 "DMP3098L" V 12251 1250 50  0000 C CNN
+F 2 "Package_TO_SOT_SMD:SOT-23" H 12200 1350 50  0001 C CNN
+F 3 "~" H 12000 1250 50  0001 C CNN
+	1    12000 1250
+	0    -1   -1   0
+$EndComp
+Wire Wire Line
+	11500 1500 11500 1600
+Wire Wire Line
+	11500 1600 12000 1600
+Connection ~ 11500 1600
+Wire Wire Line
+	11500 1600 11500 1700
+Wire Wire Line
+	12000 1450 12000 1600
+Connection ~ 12000 1600
+Wire Wire Line
+	12000 1600 12250 1600
+Text GLabel 11500 1200 1    50   Input ~ 0
+VIN
+Wire Wire Line
+	11500 1200 11500 1300
+$Comp
+L power:GND #PWR0112
+U 1 1 5EB30215
+P 11500 2000
+F 0 "#PWR0112" H 11500 1750 50  0001 C CNN
+F 1 "GND" H 11505 1827 50  0000 C CNN
+F 2 "" H 11500 2000 50  0001 C CNN
+F 3 "" H 11500 2000 50  0001 C CNN
+	1    11500 2000
+	1    0    0    -1
+$EndComp
+Wire Wire Line
+	11500 2000 11500 1900
+$Comp
+L power:+5V #PWR0113
+U 1 1 5EB3AEA4
+P 12300 1050
+F 0 "#PWR0113" H 12300 900 50  0001 C CNN
+F 1 "+5V" H 12315 1223 50  0000 C CNN
+F 2 "" H 12300 1050 50  0001 C CNN
+F 3 "" H 12300 1050 50  0001 C CNN
+	1    12300 1050
+	1    0    0    -1
+$EndComp
+Wire Wire Line
+	12200 1150 12300 1150
+Wire Wire Line
+	12300 1150 12300 1050
+$Comp
+L power:VBUS #PWR0114
+U 1 1 5EB43869
+P 11700 1050
+F 0 "#PWR0114" H 11700 900 50  0001 C CNN
+F 1 "VBUS" H 11715 1223 50  0000 C CNN
+F 2 "" H 11700 1050 50  0001 C CNN
+F 3 "" H 11700 1050 50  0001 C CNN
+	1    11700 1050
+	1    0    0    -1
+$EndComp
+Wire Wire Line
+	11700 1050 11700 1150
+Wire Wire Line
+	11700 1150 11800 1150
 $EndSCHEMATC

Commit message: update
Parts:
- added C? (x2): 22nF, symbol Device:C_Small
- added C? (x2): 4.7uF, symbol Device:C_Small
- added C? (x2): 0.1uF, symbol Device:C_Small
- added C? (x2): 1uF, symbol Device:C_Small
- added U?: TPS62132, Package_DFN_QFN:VQFN-16-1EP_3x3mm_P0.5mm_EP1.68x1.68mm_ThermalVias, symbol Regulator_Switching:TPS62132
- added U?: TPS62086, symbol InGarage_Regulator_Switching:TPS62086
- added Y?: Crystal, Crystal:Crystal_SMD_2012-2Pin_2.0x1.2mm, symbol Device:Crystal
Connections:
- net labels removed: +3V3_FTDI
- wire segments 157 -> 177
Other:
- note added: "POWER SUPPLY"
- moved on the sheet: Q1, R3, R4, R5, U3

Commit message: update
Parts:
- removed U?: TPS62132, Package_DFN_QFN:VQFN-16-1EP_3x3mm_P0.5mm_EP1.68x1.68mm_ThermalVias, symbol Regulator_Switching:TPS62132
- added C11, C14, C17, C18: 10uF, Capacitor_Tantalum_SMD:CP_EIA-3216-12_Kemet-S, symbol Device:C_Small
- added L2: 0.47uH, GiraffeTech-Inductor:L_0806_2016Metric, symbol Device:L_Small
- added L3: 1uH, GiraffeTech-Inductor:L_1616_2020Metric, symbol Device:L_Small
- added R6: 619K, Resistor_SMD:R_0603_1608Metric, symbol Device:R_Small
- added R7, R8: 100K, Resistor_SMD:R_0603_1608Metric, symbol Device:R_Small
- added U4: TPS62135, GiraffeTech-Texas:VQFN-HR-11, symbol InGarage_Regulator_Switching:TPS62135
- C10, C12, C13, C15, C16, C9: renamed from C?; footprint (none) -> Capacitor_SMD:C_0603_1608Metric
- C7, C8: renamed from C?; footprint (none) -> Capacitor_SMD:C_0603_1608Metric; Mfg. Part (none) -> 06036C223KAT2A
- L1: footprint (none) -> Inductor_SMD:L_0805_2012Metric; Mfg. Part (none) -> LQM21DH100M70L
- R1, R3, R4, R5: value 10k -> 10K
- R2: value 10k -> 1M
- U3: footprint (none) -> Package_TO_SOT_SMD:SOT-23-5
- gave numbers to parts that had none: 2
Connections:
- net labels added: PG_5V
- wire segments 177 -> 235
- no-connect marks 29 -> 30
Other:
- moved on the sheet: C10, C12, C13, C15, C16, C9, Q1, R3, R4, R5, U3, U5

Commit message: update
Parts:
- added J?: Adafruit_Feather_Conn, GiraffeTech-Connector:Adafruit-Feather_WoMountPoint, symbol Connector_Generic:Conn_01x28
Connections:
- net +3V3: now also J?.2 (Pin_2)
- net AREF: now also J?.3 (Pin_3)
- net Adf_A0_DAC0: now also J?.5 (Pin_5)
- net Adf_A1_DAC1: now also J?.6 (Pin_6)
- net Adf_A2: now also J?.7 (Pin_7)
- net Adf_A3: now also J?.8 (Pin_8)
- net Adf_A4: now also J?.9 (Pin_9)
- net Adf_A5: now also J?.10 (Pin_10)
- net Adf_D10: now also J?.22 (Pin_22)
- net Adf_D11: now also J?.23 (Pin_23)
- net Adf_D12: now also J?.24 (Pin_24)
- net Adf_D13: now also J?.25 (Pin_25)
- net Adf_D4: now also J?.16 (Pin_16)
- net Adf_D5: now also J?.19 (Pin_19)
- net Adf_D6: now also J?.20 (Pin_20)
- net Adf_D9: now also J?.21 (Pin_21)
- net D0_RxD0: now also J?.14 (Pin_14)
- net D1_TxD0: now also J?.15 (Pin_15)
- net GND: now also J?.4 (Pin_4)
- net I2C_SCL: now also J?.18 (Pin_18)
- net I2C_SDA: now also J?.17 (Pin_17)
- net SPI_MISO: now also J?.13 (Pin_13)
- net SPI_MOSI: now also J?.12 (Pin_12)
- net SPI_SCK: now also J?.11 (Pin_11)
- net ~RESET: now also J?.1 (Pin_1)
- new net BAT: J?.28 (Pin_28)
- new net EN: J?.27 (Pin_27)
- new net USB: J?.26 (Pin_26)
Changed lines of the file:
@@
 Wire Wire Line
 	12700 5300 12700 5400
+$Comp
+L Connector_Generic:Conn_01x28 J?
+U 1 1 5EB09696
+P 4800 2800
+F 0 "J?" H 4718 1175 50  0000 C CNN
+F 1 "Adafruit_Feather_Conn" H 4718 1266 50  0000 C CNN
+F 2 "GiraffeTech-Connector:Adafruit-Feather_WoMountPoint" H 4800 2800 50  0001 C CNN
+F 3 "~" H 4800 2800 50  0001 C CNN
+	1    4800 2800
+	-1   0    0    1
+$EndComp
+Wire Wire Line
+	5100 1400 5000 1400
+Wire Wire Line
+	5100 1500 5000 1500
+Wire Wire Line
+	5100 1600 5000 1600
+Wire Wire Line
+	5100 1700 5000 1700
+Wire Wire Line
+	5100 1800 5000 1800
+Wire Wire Line
+	5100 1900 5000 1900
+Wire Wire Line
+	5100 2000 5000 2000
+Wire Wire Line
+	5100 2100 5000 2100
+Wire Wire Line
+	5100 2200 5000 2200
+Wire Wire Line
+	5100 2300 5000 2300
+Wire Wire Line
+	5100 2400 5000 2400
+Wire Wire Line
+	5100 2500 5000 2500
+Wire Wire Line
+	5100 2600 5000 2600
+Wire Wire Line
+	5100 2700 5000 2700
+Wire Wire Line
+	5100 2800 5000 2800
+Wire Wire Line
+	5100 2900 5000 2900
+Wire Wire Line
+	5100 3000 5000 3000
+Wire Wire Line
+	5100 3100 5000 3100
+Wire Wire Line
+	5100 3200 5000 3200
+Wire Wire Line
+	5100 3300 5000 3300
+Wire Wire Line
+	5100 3400 5000 3400
+Wire Wire Line
+	5100 3500 5000 3500
+Wire Wire Line
+	5100 3600 5000 3600
+Wire Wire Line
+	5100 3700 5000 3700
+Wire Wire Line
+	5100 3800 5000 3800
+Wire Wire Line
+	5100 3900 5000 3900
+Wire Wire Line
+	5300 4000 5000 4000
+Wire Wire Line
+	5100 4100 5000 4100
+Text GLabel 5100 1400 2    50   Input ~ 0
+BAT
+Text GLabel 5100 1500 2    50   Input ~ 0
+EN
+Text GLabel 5100 1600 2    50   Input ~ 0
+USB
+Text GLabel 5100 2800 2    50   Input ~ 0
+D0_RxD0
+Text GLabel 5100 2700 2    50   Input ~ 0
+D1_TxD0
+Text GLabel 5100 2100 2    50   Input ~ 0
+Adf_D9
+Text GLabel 5100 2000 2    50   Input ~ 0
+Adf_D10
+Text GLabel 5100 1900 2    50   Input ~ 0
+Adf_D11
+Text GLabel 5100 1800 2    50   Input ~ 0
+Adf_D12
+Text GLabel 5100 1700 2    50   Input ~ 0
+Adf_D13
+Text GLabel 5100 2300 2    50   Input ~ 0
+Adf_D5
+Text GLabel 5100 2200 2    50   Input ~ 0
+Adf_D6
+Text GLabel 5100 2500 2    50   Input ~ 0
+I2C_SDA
+Text GLabel 5100 2400 2    50   Input ~ 0
+I2C_SCL
+Text GLabel 5100 2600 2    50   Input ~ 0
+Adf_D4
+Text GLabel 5100 2900 2    50   Input ~ 0
+SPI_MISO
+Text GLabel 5100 3000 2    50   Input ~ 0
+SPI_MOSI
+Text GLabel 5100 3100 2    50   Input ~ 0
+SPI_SCK
+Text GLabel 5100 3300 2    50   Input ~ 0
+Adf_A4
+Text GLabel 5100 3200 2    50   Input ~ 0
+Adf_A5
+Text GLabel 5100 3700 2    50   Input ~ 0
+Adf_A0_DAC0
+Text GLabel 5100 3600 2    50   Input ~ 0
+Adf_A1_DAC1
+Text GLabel 5100 3500 2    50   Input ~ 0
+Adf_A2
+Text GLabel 5100 3400 2    50   Input ~ 0
+Adf_A3
+$Comp
+L power:GND #PWR?
+U 1 1 5EDE7447
+P 5100 3800
+F 0 "#PWR?" H 5100 3550 50  0001 C CNN
+F 1 "GND" V 5105 3672 50  0000 R CNN
+F 2 "" H 5100 3800 50  0001 C CNN
+F 3 "" H 5100 3800 50  0001 C CNN
+	1    5100 3800
+	0    -1   -1   0
+$EndComp
+Text GLabel 5100 3900 2    50   Input ~ 0
+AREF
+$Comp
+L power:+3V3 #PWR?
+U 1 1 5EDEC800
+P 5300 4000
+F 0 "#PWR?" H 5300 3850 50  0001 C CNN
+F 1 "+3V3" H 5315 4173 50  0000 C CNN
+F 2 "" H 5300 4000 50  0001 C CNN
+F 3 "" H 5300 4000 50  0001 C CNN
+	1    5300 4000
+	0    1    1    0
+$EndComp
+Text GLabel 5100 4100 2    50   Input ~ 0
+~RESET
 $EndSCHEMATC

Commit message: update
Parts:
- added U?: MCP73871-1CC, Package_DFN_QFN:QFN-20-1EP_4x4mm_P0.5mm_EP2.5x2.5mm, symbol Battery_Management:MCP73871-1CC
Connections:
- net +5V: now also U?.18 (IN), U?.19 (IN)
- net GND: now also U?.10 (VSS), U?.11 (VSS), U?.21 (VSS)
- new net: U?.1 (OUT), U?.20 (OUT)
- new net: U?.14 (VBAT), U?.15 (VBAT)
Changed lines of the file:
@@
 Text GLabel 5100 4100 2    50   Input ~ 0
 ~RESET
+$Comp
+L Battery_Management:MCP73871-1CC U?
+U 1 1 5EB4EC78
+P 13500 8100
+F 0 "U?" H 12950 8950 50  0000 C CNN
+F 1 "MCP73871-1CC" H 13900 8950 50  0000 C CNN
+F 2 "Package_DFN_QFN:QFN-20-1EP_4x4mm_P0.5mm_EP2.5x2.5mm" H 13700 7200 50  0001 L CIN
+F 3 "http://www.mouser.com/ds/2/268/22090a-52174.pdf" H 13350 8650 50  0001 C CNN
+	1    13500 8100
+	1    0    0    -1
+$EndComp
+$Comp
+L power:GND #PWR?
+U 1 1 5EB512E7
+P 13500 9100
+F 0 "#PWR?" H 13500 8850 50  0001 C CNN
+F 1 "GND" H 13505 8927 50  0000 C CNN
+F 2 "" H 13500 9100 50  0001 C CNN
+F 3 "" H 13500 9100 50  0001 C CNN
+	1    13500 9100
+	1    0    0    -1
+$EndComp
+Wire Wire Line
+	13500 9000 13500 9100
+$Comp
+L power:+5V #PWR?
+U 1 1 5EB66286
+P 13500 7100
+F 0 "#PWR?" H 13500 6950 50  0001 C CNN
+F 1 "+5V" H 13515 7273 50  0000 C CNN
+F 2 "" H 13500 7100 50  0001 C CNN
+F 3 "" H 13500 7100 50  0001 C CNN
+	1    13500 7100
+	1    0    0    -1
+$EndComp
+Wire Wire Line
+	13500 7100 13500 7200
 $EndSCHEMATC

Commit message: update
Parts:
- added C?: 10uF, symbol Device:C_Small
- added D? (x3): LED, symbol Device:LED
- added R? (x3): 330, symbol Device:R_Small
- added R?: R_Small, symbol Device:R_Small
- added R?: 2K, symbol Device:R_Small
- added R? (x5): 10K, symbol Device:R_Small
Connections:
- net +5V: now also U?.2 (VPCC), R?.1, R?.1, R?.1, R?.1, R?.1, R?.1
- net GND: now also C?.2, R?.2, R?.2, R?.2
- net CHG_OUT: now reaches U?.1 (OUT), U?.20 (OUT)
- net PROG3: now reaches U?.12 (PROG3)
- net PROG3: now also R?.1
- net PROG1: now reaches U?.13 (PROG1)
- net PROG1: now also R?.1
- net +BATT: now reaches U?.14 (VBAT), U?.15 (VBAT)
- net +BATT: now also U?.16 (Vbat_SENSE), C?.1
- net REG_SEL: now reaches U?.3 (SEL)
- net REG_SEL: now also R?.2
- net PROG2: now reaches U?.4 (PROG2)
- net PROG2: now also R?.2
- net THERMAL: now reaches U?.5 (THERM)
- net THERMAL: now also R?.1
- net ~PG: now reaches U?.6 (~PG~)
- net ~PG: now also D?.1 (K)
- net STAT2: now reaches U?.7 (STAT2)
- net STAT2: now also D?.1 (K)
- net STAT1: now reaches U?.8 (STAT1/~LBO~)
- net STAT1: now also D?.1 (K)
- net ~TE: now reaches U?.9 (~TE)
- net ~TE: now also R?.2
- new net: D?.2 (A), R?.2 (x3)
Other:
- moved on the sheet: U?

Commit message: update
Parts:
- removed R?: R_Small, symbol Device:R_Small
- added R?: 10K, symbol Device:R_Small
Connections:
- net +5V: now also R?.1; no longer C14.1, U5.1 (EN), U5.7 (VIN)
- net CE: now also U?.17 (CE), R?.2
- net CHG_OUT: now also C14.1, U5.7 (VIN)
- new net 3v3_EN: U5.1 (EN)
Other:
- moved on the sheet: C14, C?, D?, R?, U?

Commit message: update
Parts:
- added J?: Micro_SD_Card, symbol Connector:Micro_SD_Card
- added R?: 10K, symbol Device:R_Small
- added R?: R_Small, symbol Device:R_Small
- added SW?: RESET, symbol Switch:SW_Push
Connections:
- net ESP_CS is gone; now on net Adf_D8: R1.1, U1.29 (IO5)
- net ESP_IO0 is gone; now on net Adf_D3: U1.25 (IO0)
- net ESP_MISO is gone; now on net SPI_MISO: U1.37 (IO23)
- net ESP_MOSI is gone; now on net SPI_MOSI: U1.13 (IO14)
- net ESP_RESET is gone; now on net Adf_D2: U1.3 (EN)
- net ESP_RxD is gone; now on net D0_RxD0: U1.34 (RXD0/IO3)
- net ESP_SCK is gone; now on net SPI_SCK: U1.30 (IO18)
- net ESP_TxD is gone; now on net D1_TxD0: U1.35 (TXD0/IO1)
- net +3V3: now also J?.4 (VDD), R?.1, R?.2
- net GND: now also J?.6 (VSS), J?.9 (SHIELD), SW?.2
- net QSPI_CS: now also R?.2
- net SPI_MISO: now also J?.3 (CMD)
- net SPI_MOSI: now also J?.7 (DAT0)
- net SPI_SCK: now also J?.5 (CLK)
- net ~RESET: now also R?.1, SW?.1
Changed lines of the file:
@@
 Wire Wire Line
 	1800 1500 1900 1500
-Text GLabel 3200 1600 2    50   Input ~ 0
-ESP_TxD
-Text GLabel 3200 1800 2    50   Input ~ 0
-ESP_RxD
 Wire Wire Line
 	3100 1500 3200 1500
@@
 	9100 3550 9000 3550
 Wire Wire Line
-	9100 3650 9000 3650
+	9650 3650 9550 3650
 Wire Wire Line
 	9100 3750 9000 3750
@@
 	9100 4050 9000 4050
 Wire Wire Line
-	9100 4150 9000 4150
-Wire Wire Line
-	9100 4250 9000 4250
+	9650 4150 9600 4150
+Wire Wire Line
+	9650 4250 9550 4250
 Wire Wire Line
 	9100 4350 9000 4350
@@
 	7500 3550 7600 3550
 Wire Wire Line
-	7500 3650 7600 3650
-Wire Wire Line
-	7500 3750 7600 3750
-Wire Wire Line
-	7500 3850 7600 3850
-Wire Wire Line
 	7500 3950 7600 3950
 Wire Wire Line
@@
 	7500 4450 7600 4450
 Wire Wire Line
-	7500 4550 7600 4550
-Wire Wire Line
-	7500 4650 7600 4650
-Wire Wire Line
-	7500 4750 7600 4750
+	7000 4550 7050 4550
 Wire Wire Line
 	7500 4850 7600 4850
@@
 NoConn ~ 3200 2200
 NoConn ~ 3200 2400
-Text GLabel 3200 3100 2    50   Input ~ 0
-ESP_MISO
-Text GLabel 3200 2700 2    50   Input ~ 0
-ESP_SCK
 Text GLabel 3200 2000 2    50   Input ~ 0
 ESP_CS
-Text GLabel 3200 2300 2    50   Input ~ 0
-ESP_MOSI
 Text GLabel 3200 3600 2    50   Input ~ 0
 ESP_ACK
@@
 Text GLabel 9100 3750 2    50   Input ~ 0
 Adf_D7
-Text GLabel 7500 4550 0    50   Input ~ 0
+Text GLabel 7000 4550 0    50   Input ~ 0
 Adf_D8
 Text GLabel 7500 4450 0    50   Input ~ 0
@@
 Text GLabel 9100 4350 2    50   Input ~ 0
 WS2812_INT
-Text GLabel 9100 4250 2    50   Input ~ 0
+Text GLabel 9650 4250 2    50   Input ~ 0
 Adf_D2
-Text GLabel 9100 4150 2    50   Input ~ 0
+Text GLabel 9650 4150 2    50   Input ~ 0
 Adf_D3
 Text GLabel 9100 3850 2    50   Input ~ 0
@@
 Text GLabel 9100 3550 2    50   Input ~ 0
 QSPI_SCK
-Text GLabel 9100 3650 2    50   Input ~ 0
+Text GLabel 9650 3650 2    50   Input ~ 0
 QSPI_CS
 Text GLabel 7500 3850 0    50   Input ~ 0
@@
 Wire Wire Line
 	12900 5050 13000 5050
+$Comp
+L Switch:SW_Push SW?
+U 1 1 5EB63614
+P 10650 1150
+F 0 "SW?" H 10650 1435 50  0000 C CNN
+F 1 "RESET" H 10650 1344 50  0000 C CNN
+F 2 "" H 10650 1350 50  0001 C CNN
+F 3 "~" H 10650 1350 50  0001 C CNN
+	1    10650 1150
+	1    0    0    -1
+$EndComp
+Text GLabel 10250 1150 0    50   Input ~ 0
+~RESET
+Wire Wire Line
+	10250 1150 10350 1150
+$Comp
+L power:GND #PWR?
+U 1 1 5EB8BCDD
+P 10950 1250
+F 0 "#PWR?" H 10950 1000 50  0001 C CNN
+F 1 "GND" H 10955 1077 50  0000 C CNN
+F 2 "" H 10950 1250 50  0001 C CNN
+F 3 "" H 10950 1250 50  0001 C CNN
+	1    10950 1250
+	1    0    0    -1
+$EndComp
+Wire Wire Line
+	10850 1150 10950 1150
+Wire Wire Line
+	10950 1150 10950 1250
+$Comp
+L Device:R_Small R?
+U 1 1 5EBA53E3
+P 10100 950
+F 0 "R?" V 9904 950 50  0000 C CNN
+F 1 "10K" V 9995 950 50  0000 C CNN
+F 2 "" H 10100 950 50  0001 C CNN
+F 3 "~" H 10100 950 50  0001 C CNN
+	1    10100 950
+	0    1    1    0
+$EndComp
+Wire Wire Line
+	10200 950  10350 950
+Wire Wire Line
+	10350 950  10350 1150
+Connection ~ 10350 1150
+Wire Wire Line
+	10350 1150 10450 1150
+$Comp
+L power:+3V3 #PWR?
+U 1 1 5EBBF903
+P 9900 850
+F 0 "#PWR?" H 9900 700 50  0001 C CNN
+F 1 "+3V3" H 9915 1023 50  0000 C CNN
+F 2 "" H 9900 850 50  0001 C CNN
+F 3 "" H 9900 850 50  0001 C CNN
+	1    9900 850
+	1    0    0    -1
+$EndComp
+Wire Wire Line
+	9900 850  9900 950
+Wire Wire Line
+	9900 950  10000 950
+Text GLabel 7000 4400 0    50   Input ~ 0
+ESP_CS
+Text GLabel 9650 4000 2    50   Input ~ 0
+ESP_IO0
+Text GLabel 9650 3900 2    50   Input ~ 0
+ESP_RESET
+$Comp
+L Device:R_Small R?
+U 1 1 5ECB68ED
+P 9900 3350
+F 0 "R?" H 9959 3396 50  0000 L CNN
+F 1 "R_Small" H 9959 3305 50  0000 L CNN
+F 2 "" H 9900 3350 50  0001 C CNN
+F 3 "~" H 9900 3350 50  0001 C CNN
+	1    9900 3350
+	1    0    0    -1
+$EndComp
+$Comp
+L power:+3V3 #PWR?
+U 1 1 5ECB73F8
+P 9900 3150
+F 0 "#PWR?" H 9900 3000 50  0001 C CNN
+F 1 "+3V3" H 9915 3323 50  0000 C CNN
+F 2 "" H 9900 3150 50  0001 C CNN
+F 3 "" H 9900 3150 50  0001 C CNN
+	1    9900 3150
+	1    0    0    -1
+$EndComp
+Wire Wire Line
+	9900 3150 9900 3250
+Wire Wire Line
+	9550 3650 9550 3550
+Wire Wire Line
+	9550 3550 9900 3550
+Wire Wire Line
+	9900 3550 9900 3450
+Connection ~ 9550 3650
+Wire Wire Line
+	9550 3650 9000 3650
+Wire Wire Line
+	7000 4400 7050 4400
+Wire Wire Line
+	7050 4400 7050 4550
+Wire Wire Line
+	9650 4000 9600 4000
+Wire Wire Line
+	9600 4000 9600 4150
+Connection ~ 9600 4150
+Wire Wire Line
+	9600 4150 9000 4150
+Wire Wire Line
+	9650 3900 9550 3900
+Wire Wire Line
+	9550 3900 9550 4250
+Connection ~ 9550 4250
+Wire Wire Line
+	9550 4250 9000 4250
+$Comp
+L Connector:Micro_SD_Card J?
+U 1 1 5F197AED
+P 8300 7050
+F 0 "J?" H 8250 7767 50  0000 C CNN
+F 1 "Micro_SD_Card" H 8250 7676 50  0000 C CNN
+F 2 "" H 9450 7350 50  0001 C CNN
+F 3 "http://katalog.we-online.de/em/datasheet/693072010801.pdf" H 8300 7050 50  0001 C CNN
+	1    8300 7050
+	1    0    0    -1
+$EndComp
+$Comp
+L power:GND #PWR?
+U 1 1 5F19B5B8
+P 9200 7750
+F 0 "#PWR?" H 9200 7500 50  0001 C CNN
+F 1 "GND" H 9205 7577 50  0000 C CNN
+F 2 "" H 9200 7750 50  0001 C CNN
+F 3 "" H 9200 7750 50  0001 C CNN
+	1    9200 7750
+	1    0    0    -1
+$EndComp
+Wire Wire Line
+	9100 7650 9200 7650
+Wire Wire Line
+	9200 7650 9200 7750
+$Comp
+L power:GND #PWR?
+U 1 1 5F1BC880
+P 6850 7250
+F 0 "#PWR?" H 6850 7000 50  0001 C CNN
+F 1 "GND" V 6855 7122 50  0000 R CNN
+F 2 "" H 6850 7250 50  0001 C CNN
+F 3 "" H 6850 7250 50  0001 C CNN
+	1    6850 7250
+	0    1    1    0
+$EndComp
+Wire Wire Line
+	7300 6750 7400 6750
+Wire Wire Line
+	7300 6850 7400 6850
+Wire Wire Line
+	7300 6950 7400 6950
+Wire Wire Line
+	6850 7050 7400 7050
+Wire Wire Line
+	7300 7150 7400 7150
+Wire Wire Line
+	6850 7250 7400 7250
+Wire Wire Line
+	7300 7350 7400 7350
+Wire Wire Line
+	7300 7450 7400 7450
+$Comp
+L power:+3V3 #PWR?
+U 1 1 5F2C89F7
+P 6850 7050
+F 0 "#PWR?" H 6850 6900 50  0001 C CNN
+F 1 "+3V3" H 6865 7223 50  0000 C CNN
+F 2 "" H 6850 7050 50  0001 C CNN
+F 3 "" H 6850 7050 50  0001 C CNN
+	1    6850 7050
+	0    -1   -1   0
+$EndComp
+Text GLabel 3200 3100 2    50   Input ~ 0
+SPI_MISO
+Text GLabel 3200 2300 2    50   Input ~ 0
+SPI_MOSI
+Text GLabel 3200 2700 2    50   Input ~ 0
+SPI_SCK
+Text GLabel 3200 1800 2    50   Input ~ 0
+D0_RxD0
+Text GLabel 3200 1600 2    50   Input ~ 0
+D1_TxD0
+Wire Wire Line
+	7500 4650 7600 4650
+Wire Wire Line
+	7500 4750 7600 4750
+Wire Wire Line
+	7500 3650 7600 3650
+Wire Wire Line
+	7500 3750 7600 3750
+Wire Wire Line
+	7500 3850 7600 3850
+Wire Wire Line
+	7050 4550 7600 4550
+Connection ~ 7050 4550
+Text GLabel 7300 6950 0    50   Input ~ 0
+SPI_MISO
+Text GLabel 7300 7350 0    50   Input ~ 0
+SPI_MOSI
+Text GLabel 7300 7150 0    50   Input ~ 0
+SPI_SCK
 $EndSCHEMATC
