File: MP_SamBaseBoard_V1_DraftDesign/MP_SamBaseBoard_V1.sch (KiCad schematic (older format))
At the start: 56 parts, among them Q1 DMP3098L, U1 ESP32-WROOM-32, U2 ATSAMD51J19A-A, U3 74LVC1G125, U4 TPS62135, U5 TPS62086, Y1 Crystal

Commit message: update
Parts:
- added C? (x2): 0.1uF, symbol Device:C_Small
- added C? (x3): 0.1uF 16V, symbol Device:C_Small
- added C?: 10uF 16V, symbol Device:C_Small
- added C?: CF, symbol Device:C_Small
- added J?: MOTOR A, symbol Connector_Generic:Conn_01x02
- added J?: MOTOR B, symbol Connector_Generic:Conn_01x02
- added MK?: Knowles_SPW2430HR5H-B, symbol InGarage_Sensor_Audio:Knowles_SPW2430HR5H-B
- added R?: 10K, symbol Device:R_Small
- added SW?: 3v3_PWR_SW, GiraffeTech-Electromechanical:SW_SPDT_CK-JS102011JCQN, symbol Switch:SW_SPDT
- added U?: HDC1080DMBR, Package_SON:WSON-6-1EP_3x3mm_P0.95mm, symbol InGarage_Sensor_Environment:HDC1080DMBR
- added U?: MAX98357AETE, Package_DFN_QFN:TQFN-16-1EP_3x3mm_P0.5mm_EP1.23x1.23mm, symbol InGarage_Audio_Amplifier:MAX98357AETE
- added U?: DRV8833RTY, Package_DFN_QFN:Texas_S-PWQFN-N16_EP2.1x2.1mm_ThermalVias, symbol Driver_Motor:DRV8833RTY
Connections:
- wire segments 338 -> 404
- no-connect marks 30 -> 35
Other:
- note added: "SENSORS & DRIVER"
- moved on the sheet: C14, J?

Commit message: update
Parts:
- removed U?: HDC1080DMBR, Package_SON:WSON-6-1EP_3x3mm_P0.95mm, symbol InGarage_Sensor_Environment:HDC1080DMBR
- added C27: 2.2uF 6.3V, Capacitor_SMD:C_0603_1608Metric, symbol Device:C_Small
- added C28, C29: 0.1uF, Capacitor_SMD:C_0603_1608Metric, symbol Device:C_Small
- added C30: 2.2nF, Capacitor_SMD:C_0603_1608Metric, symbol Device:C_Small
- added J?: P3, symbol Connector_Generic:Conn_01x04
- added J?: P2, symbol Connector_Generic:Conn_01x04
- added J?: P1, symbol Connector_Generic:Conn_01x04
- added J? (x2): I2C, symbol Connector_Generic:Conn_01x04
- added J?: WS2812_EXT, symbol Connector_Generic:Conn_01x03
- added R22: 10K, Resistor_SMD:R_0603_1608Metric, symbol Device:R_Small
- added U10: MPU-6050, Sensor_Motion:InvenSense_QFN-24_4x4mm_P0.5mm, symbol Sensor_Motion:MPU-6050
- added U8: HDC1080, Package_SON:Texas_PWSON-N6, symbol Sensor_Humidity:HDC1080
- C19, C20, C21, C22, C24, C25: renamed from C?; footprint (none) -> Capacitor_SMD:C_0603_1608Metric
- C23, C26: renamed from C?; footprint (none) -> Capacitor_Tantalum_SMD:CP_EIA-3216-12_Kemet-S
- D1, D2, D3: renamed from D?; footprint (none) -> LED_SMD:LED_0603_1608Metric
- J1: renamed from J?; value MOTOR A -> MOTOR-A_CONN; footprint (none) -> GiraffeTech-Connector:DINKLE_EK500V-2P
- J2: renamed from J?; value MOTOR B -> MOTOR-B_CONN; footprint (none) -> GiraffeTech-Connector:DINKLE_EK500V-2P
- MK1: renamed from MK?; footprint (none) -> GiraffeTech-Knowles:SPW2430HR5H-B
- R10, R11, R12, R13, R14, R15, R16, R17, R18, R19, R20, R21: renamed from R?; footprint (none) -> Resistor_SMD:R_0603_1608Metric
- R9: renamed from R?; value R_Small -> 10K; footprint (none) -> Resistor_SMD:R_0603_1608Metric
- SW1: renamed from SW?; footprint (none) -> Button_Switch_SMD:SW_SPST_B3S-1000
- U1: footprint RF_Module:ESP32-WROOM-32 -> GiraffeTech-NodeMCU:ESP32-WROOM-32_WifiNinaPin
- U5: footprint (none) -> GiraffeTech-Texas:Texas_VSON7
- gave numbers to parts that had none: 6
Connections:
- net labels added: WS2812_EXT
- wire segments 404 -> 452
- no-connect marks 35 -> 38
Other:
- moved on the sheet: C10, C11, C12, C13, C14, C15, C16, C17, C18, C19, C21, C22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

Commit message: update
Parts:
- added J?: SERVO_CONN, symbol Connector_Generic:Conn_02x03_Odd_Even
- added J?: PWR_JACK, symbol Connector:Barrel_Jack_Switch
- J3: value Adafruit_Feather_Conn -> Adafruit_Feather_CONN
- J4: value Micro_SD_Card -> uSD_Card
- J?: value P3 -> P3_CONN
- J?: value P2 -> P2_CONN
- J?: value P1 -> P1_CONN
- J? (x2): value I2C -> I2C_CONN
Connections:
- net +5V: now also J?.3 (Pin_3), J?.4 (Pin_4)
- net Adf_A0_DAC0: now also J?.4 (Pin_4)
- net Adf_A1_DAC1: now also J?.3 (Pin_3)
- net Adf_A2: now also J?.4 (Pin_4)
- net Adf_A3: now also J?.3 (Pin_3)
- net Adf_A4: now also J?.4 (Pin_4)
- net Adf_D13: now also J4.2 (DAT3/CD)
- net Adf_D4: now also J?.3 (Pin_3), J?.1 (Pin_1)
- net Adf_D7: now also J?.2 (Pin_2)
- net GND: now also J?.2, J?.3, J?.5 (Pin_5), J?.6 (Pin_6)
- net I2C_SCL: now also J?.4 (Pin_4), J?.4 (Pin_4)
- net I2C_SDA: now also J?.3 (Pin_3), J?.3 (Pin_3)
- net VIN: now also J?.1
- no-connect marks 38 -> 37
Other:
- moved on the sheet: C11, C14, C17, C18, D1, D2, D3, J?, L2, L3, R11, R16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

Commit message: update
Parts:
- added J?: Conn_01x02, GiraffeTech-Connector:DINKLE_EK500V-2P, symbol Connector_Generic:Conn_01x02
- added R?: 10K, symbol Device:R_Small
Connections:
- net +3V3: now also U6.7 (VDD), U6.8 (VDD), R?.1
- net GND: now also U6.11 (GND), U6.15 (GND), U6.16 (PAD), U6.2 (GAIN_SLOT), U6.3 (GND)
- net at U6.10 (OUTN): now also J?.2 (Pin_2)
- net at U6.4 (~SD_MODE): now also R?.2
- net at U6.9 (OUTP): now also J?.1 (Pin_1)
Changed lines of the file:
@@
 Wire Wire Line
 	9050 5200 9050 5300
+$Comp
+L power:GND #PWR?
+U 1 1 5EBCE8B3
+P 2050 10750
+F 0 "#PWR?" H 2050 10500 50  0001 C CNN
+F 1 "GND" H 2055 10577 50  0000 C CNN
+F 2 "" H 2050 10750 50  0001 C CNN
+F 3 "" H 2050 10750 50  0001 C CNN
+	1    2050 10750
+	1    0    0    -1
+$EndComp
+Wire Wire Line
+	2000 10650 2000 10700
+Wire Wire Line
+	2000 10700 2050 10700
+Wire Wire Line
+	2100 10700 2100 10650
+Wire Wire Line
+	2050 10700 2050 10750
+Connection ~ 2050 10700
+Wire Wire Line
+	2050 10700 2100 10700
+$Comp
+L power:+3V3 #PWR?
+U 1 1 5EC93765
+P 2000 9550
+F 0 "#PWR?" H 2000 9400 50  0001 C CNN
+F 1 "+3V3" H 2015 9723 50  0000 C CNN
+F 2 "" H 2000 9550 50  0001 C CNN
+F 3 "" H 2000 9550 50  0001 C CNN
+	1    2000 9550
+	1    0    0    -1
+$EndComp
+Wire Wire Line
+	2000 9550 2000 9650
+$Comp
+L Connector_Generic:Conn_01x02 J?
+U 1 1 5ECD71B7
+P 2800 10100
+F 0 "J?" H 2880 10092 50  0000 L CNN
+F 1 "Conn_01x02" H 2880 10001 50  0000 L CNN
+F 2 "GiraffeTech-Connector:DINKLE_EK500V-2P" H 2800 10100 50  0001 C CNN
+F 3 "~" H 2800 10100 50  0001 C CNN
+	1    2800 10100
+	1    0    0    -1
+$EndComp
+$Comp
+L power:GND #PWR?
+U 1 1 5ECD7DED
+P 2200 9550
+F 0 "#PWR?" H 2200 9300 50  0001 C CNN
+F 1 "GND" V 2205 9422 50  0000 R CNN
+F 2 "" H 2200 9550 50  0001 C CNN
+F 3 "" H 2200 9550 50  0001 C CNN
+	1    2200 9550
+	0    -1   -1   0
+$EndComp
+Wire Wire Line
+	2100 9650 2100 9550
+Wire Wire Line
+	2100 9550 2200 9550
+Wire Wire Line
+	2500 10050 2550 10050
+Wire Wire Line
+	2550 10050 2550 10100
+Wire Wire Line
+	2550 10100 2600 10100
+Wire Wire Line
+	2500 10250 2550 10250
+Wire Wire Line
+	2550 10250 2550 10200
+Wire Wire Line
+	2550 10200 2600 10200
+$Comp
+L power:+3V3 #PWR?
+U 1 1 5EDA8D80
+P 1250 9550
+F 0 "#PWR?" H 1250 9400 50  0001 C CNN
+F 1 "+3V3" H 1265 9723 50  0000 C CNN
+F 2 "" H 1250 9550 50  0001 C CNN
+F 3 "" H 1250 9550 50  0001 C CNN
+	1    1250 9550
+	1    0    0    -1
+$EndComp
+$Comp
+L Device:R_Small R?
+U 1 1 5EDA94F1
+P 1250 9750
+F 0 "R?" H 1309 9796 50  0000 L CNN
+F 1 "10K" H 1309 9705 50  0000 L CNN
+F 2 "" H 1250 9750 50  0001 C CNN
+F 3 "~" H 1250 9750 50  0001 C CNN
+	1    1250 9750
+	1    0    0    -1
+$EndComp
+Wire Wire Line
+	1250 9550 1250 9650
+Wire Wire Line
+	1250 9850 1250 10250
+Wire Wire Line
+	1250 10250 1500 10250
+Wire Wire Line
+	1100 9950 1500 9950
+Wire Wire Line
+	1100 10050 1500 10050
+Wire Wire Line
+	1100 10150 1500 10150
 $EndSCHEMATC

Commit message: update
Parts:
- added C?: 0.1uF, Capacitor_SMD:C_0603_1608Metric, symbol Device:C_Small
- added C?: 1uF, Capacitor_SMD:C_0603_1608Metric, symbol Device:C_Small
Connections:
- net +3V3: now also C?.1, C?.1
- net Adf_D10: now also U6.14 (LRCLK)
- net Adf_D11: now also U6.1 (DIN), U7.13 (AIN2)
- net Adf_D12: now also U7.8 (BIN2)
- net Adf_D5: no longer U7.8 (BIN2)
- net Adf_D6: no longer U7.7 (BIN1)
- net Adf_D9: now also U7.7 (BIN1); no longer U7.13 (AIN2)
- net D1_TxD0: now also U6.16 (PAD)
- net GND: now also C?.2, C?.2
Other:
- note added: "ACCELERO METER"
- note added: "I2S AMPLIFIER"
- note added: "TEMPERATURE & HUMIDITY"
- moved on the sheet: C20, C22, C23, C24, C25, C27, J1, J2, J?, R?, U6, U7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

Commit message: update
Parts:
- added R?: R_Small, symbol Device:R_Small
- added U?: IRFHM9331PbF, symbol InGarage_FETs:IRFHM9331PbF
Other:
- note added: "LOAD DRIVER"
Changed lines of the file:
@@
 Text Notes 1800 9100 0    50   ~ 0
 I2S AMPLIFIER
+$Comp
+L InGarage_FETs:IRFHM9331PbF U?
+U 1 1 5EC3E014
+P 8550 7800
+F 0 "U?" H 8930 7846 50  0000 L CNN
+F 1 "IRFHM9331PbF" H 8930 7755 50  0000 L CNN
+F 2 "" H 8050 8350 50  0001 C CNN
+F 3 "" H 8050 8350 50  0001 C CNN
+	1    8550 7800
+	1    0    0    -1
+$EndComp
+Text Notes 8300 6850 0    50   ~ 0
+LOAD DRIVER
+$Comp
+L Device:R_Small R?
+U 1 1 5EC581FE
+P 7750 7600
+F 0 "R?" H 7809 7646 50  0000 L CNN
+F 1 "R_Small" H 7809 7555 50  0000 L CNN
+F 2 "" H 7750 7600 50  0001 C CNN
+F 3 "~" H 7750 7600 50  0001 C CNN
+	1    7750 7600
+	1    0    0    -1
+$EndComp
+Text GLabel 7600 7800 0    50   Input ~ 0
+Adf_D6
 $EndSCHEMATC

Commit message: update
Parts:
- removed C21: CF, Capacitor_SMD:C_0603_1608Metric, symbol Device:C_Small
- added C32, C33: 4.7uF, Capacitor_SMD:C_0603_1608Metric, symbol Device:C_Small
- added C34, C35, C36, C37: 0.1uF, Capacitor_SMD:C_0603_1608Metric, symbol Device:C_Small
- added C38, C39, C40, C41: 1uF, Capacitor_SMD:C_0603_1608Metric, symbol Device:C_Small
- added J13: SAM_SWD, Connector_PinHeader_1.27mm:PinHeader_2x05_P1.27mm_Vertical, symbol Connector_Generic:Conn_02x05_Odd_Even
- added J6: Conn_01x02, GiraffeTech-Connector:DINKLE_EK500V-2P, symbol Connector_Generic:Conn_01x02
- added R25, R26, R27, R28: 10K, Resistor_SMD:R_0603_1608Metric, symbol Device:R_Small
- added R29: 820K, Resistor_SMD:R_0603_1608Metric, symbol Device:R_Small
- added SW3: SW1, Button_Switch_SMD:SW_SPST_B3S-1000, symbol Switch:SW_Push
- added SW4: SW2, Button_Switch_SMD:SW_SPST_B3S-1000, symbol Switch:SW_Push
- added U12: BD5291FVE-GTR, Package_TO_SOT_SMD:SOT-353_SC-70-5, symbol pspice:OPAMP
- J10, J11, J12, J8, J9: renamed from J?; footprint (none) -> Connector_JST:JST_PH_B4B-PH-K_1x04_P2.00mm_Vertical
- J14: renamed from J?; footprint (none) -> Connector_PinHeader_2.54mm:PinHeader_1x03_P2.54mm_Vertical
- J15: renamed from J?; footprint (none) -> Connector_BarrelJack:BarrelJack_Horizontal; ES No. (none) -> 0171-0140-3; Mfg. Part (none) -> DS-012-B-PBT-ROHS
- J7: renamed from J?; footprint (none) -> Connector_PinHeader_2.54mm:PinHeader_2x03_P2.54mm_Vertical
- R23: renamed from R?; footprint (none) -> Resistor_SMD:R_0603_1608Metric
- R24: renamed from R?; value R_Small -> RG; footprint (none) -> Resistor_SMD:R_0603_1608Metric
- U11: renamed from U?; footprint (none) -> GiraffeTech-IR:PQFN_3x3mm
- gave numbers to parts that had none: 3
Connections:
- net +3V3: now also J13.1 (Pin_1), R25.1, R26.1, U12.4 (V+)
- net +5V: now also C34.1, C35.1, C36.1, C37.1, C38.1, C39.1, C40.1, C41.1
- net Adf_A1_DAC1: now also SW3.1
- net Adf_A3: now also SW4.1
- net Adf_A5: now also R29.1, U12.3
- net Adf_D6: now also R24.2
- net GND: now also U11.5 (DRAIN), U11.6 (DRAIN), U11.7 (DRAIN), U11.8 (DRAIN), C33.1, C34.2, C35.2, C36.2, C37.2, C38.2, C39.2, C40.2, C41.2, J13.3 (Pin_3), J13.5 (Pin_5), J13.9 (Pin_9), J6.2 (Pin_2), R27.2, SW3.2, SW4.2, U12.5 (V-)
- net SWCLK: now also J13.4 (Pin_4)
- net SWDIO: now also J13.2 (Pin_2)
- net SWO: now also J13.6 (Pin_6)
- net ~RESET: now also J13.10 (Pin_10)
- net at MK1.1 (OUT): now also C32.2
- net at U11.1 (SOURCE): now also U11.2 (SOURCE), U11.3 (SOURCE), J6.1 (Pin_1)
- net at U11.4 (GATE): now also R24.1, R25.2
- new net: C33.2, R26.2, R27.1, U12.1 (+)
- new net: R28.1, R29.2, U12.2 (-)
- new net: C32.1, R28.2
- no-connect marks 37 -> 39
Other:
- note added: "MICROPHONE"
- moved on the sheet: C11, C14, C17, C18, C19, J15, J4, J7, L2, L3, MK1, R11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

Commit message: update
Parts:
- added D4, D5: LED, LED_SMD:LED_0603_1608Metric, symbol Device:LED
- added D6, D7: WS2812B, LED_SMD:LED_WS2812B_PLCC4_5.0x5.0mm_P3.2mm, symbol LED:WS2812B
- added R30, R31: 1K, Resistor_SMD:R_0603_1608Metric, symbol Device:R_Small
- J4: footprint (none) -> GiraffeTech-Connector:GTK_TFMS08TK-PP-02
- R16, R18, R20: value 330 -> 1K
Connections:
- net +3V3: now also D4.2 (A), D5.2 (A), D6.1 (VDD), D7.1 (VDD)
- net GND: now also D6.3 (VSS), D7.3 (VSS)
- net SAM_RxLED: now also R31.2
- net SAM_TxLED: now also R30.2
- net WS2812_EXT: now also D7.2 (DOUT)
- net WS2812_INT: now also D6.4 (DIN)
- new net: D6.2 (DOUT), D7.4 (DIN)
- new net: D4.1 (K), R30.1
- new net: D5.1 (K), R31.1
Other:
- moved on the sheet: J4
