File: MP_SamBaseBoard_V1_DraftDesign/MP_SamBaseBoard_V1.sch (KiCad schematic (older format))
At the start: 127 parts, among them J1 MOTOR-A_CONN, J10 P1_CONN, J11 I2C_CONN, J12 I2C_CONN, J13 SAM_SWD, J14 WS2812_EXT, J15 PWR_JACK, J16 USB_B_Micro, J17 BATT_CONN, J2 MOTOR-B_CONN, J3 Adafruit_Feather_CONN, J4 uSD_Card, J5 Conn_01x02, J6 Conn_01x02, J7 SERVO_CONN, J8 P3_CONN, J9 P2_CONN, Q1 DMP3098L, SW1 RESET, SW2 3v3_PWR_SW, SW3 SW1, SW4 SW2, U1 ESP32-WROOM-32, U10 MPU-6050, U11 IRFHM9331PbF, U12 BD5291FVE-GTR, U2 ATSAMD51J19A-A, U3 74LVC1G125, U4 TPS62135, U5 TPS62086, U6 MAX98357AETE, U7 DRV8833RTY, U8 HDC1080, U9 MCP73871-1CC, Y1 Crystal

Commit message: update
Parts:
- J3: footprint GiraffeTech-Connector:Adafruit-Feather_WoMountPoint_TypeA -> GiraffeTech-Connector:Adafruit-Feather_WoMountPoint_TypeB
- U13: renamed from U?; value SST25VF080B-50-4x-S2Ax -> SST25VF016B-50-4C-S2AF
Connections:
- net +3V3_FTDI is gone; now on net +3V3: U13.8 (VDD)
- net VCC is gone; now on net +3V3: U3.5 (VCC)
- net Adf_D13: no longer J3.25 (Pin_25)
- net QSPI_CS: now also U13.1 (~CE)
- net QSPI_IO0: now also U13.5 (SI)
- net QSPI_IO1: now also U13.2 (SO)
- net QSPI_IO2: now also U13.3 (~WP~)
- net QSPI_IO3: now also U13.7 (~HOLD~)
- net QSPI_SCK: now also U13.6 (SCK)
- no-connect marks 42 -> 43
Other:
- note added: "MEMORY"
Changed lines of the file:
@@
 Connection ~ 15300 1900
 Wire Wire Line
-	15300 1450 15300 1550
+	15300 1450 15300 1500
 Wire Wire Line
 	14850 2100 14850 2200
@@
 F 0 "J3" H 4118 1175 50  0000 C CNN
 F 1 "Adafruit_Feather_CONN" H 4118 1266 50  0000 C CNN
-F 2 "GiraffeTech-Connector:Adafruit-Feather_WoMountPoint_TypeA" H 4200 2800 50  0001 C CNN
+F 2 "GiraffeTech-Connector:Adafruit-Feather_WoMountPoint_TypeB" H 4200 2800 50  0001 C CNN
 F 3 "~" H 4200 2800 50  0001 C CNN
 	1    4200 2800
@@
 Text GLabel 4500 1800 2    50   Input ~ 0
 Adf_D12
-Text GLabel 4500 1700 2    50   Input ~ 0
-Adf_D13
 Text GLabel 4500 2300 2    50   Input ~ 0
 Adf_D5
@@
 	1    0    0    -1
 $EndComp
-Text Notes 2950 4700 0    100  ~ 0
+Text Notes 3400 6750 0    100  ~ 0
 SENSORS & DRIVER
 $Comp
@@
 NoConn ~ 4500 1600
 $Comp
-L Memory_Flash:SST25VF080B-50-4x-S2Ax U?
+L Memory_Flash:SST25VF080B-50-4x-S2Ax U13
 U 1 1 5F89670D
 P 4650 5550
-F 0 "U?" H 4400 5900 50  0000 L CNN
-F 1 "SST25VF080B-50-4x-S2Ax" H 5000 5300 50  0000 L CNN
+F 0 "U13" H 4400 5900 50  0000 L CNN
+F 1 "SST25VF016B-50-4C-S2AF" H 5000 5300 50  0000 L CNN
 F 2 "Package_SO:SOIC-8_5.275x5.275mm_P1.27mm" H 4650 4850 50  0001 C CNN
 F 3 "http://ww1.microchip.com/downloads/en/DeviceDoc/20005045C.pdf" H 4600 6100 50  0001 C CNN
@@
 $EndComp
 $Comp
-L power:GND #PWR?
+L power:GND #PWR0243
 U 1 1 5FA539E1
 P 4650 6050
-F 0 "#PWR?" H 4650 5800 50  0001 C CNN
+F 0 "#PWR0243" H 4650 5800 50  0001 C CNN
 F 1 "GND" H 4655 5877 50  0000 C CNN
 F 2 "" H 4650 6050 50  0001 C CNN
@@
 Wire Wire Line
 	4650 5950 4650 6050
+Wire Wire Line
+	4650 5050 4650 5150
 $Comp
-L InGarage_Power:+3V3_FTDI #PWR?
-U 1 1 5FAC282B
+L power:+3V3 #PWR0244
+U 1 1 5EC5AB49
 P 4650 5050
-F 0 "#PWR?" H 4650 4900 50  0001 C CNN
-F 1 "+3V3_FTDI" H 4665 5223 50  0000 C CNN
+F 0 "#PWR0244" H 4650 4900 50  0001 C CNN
+F 1 "+3V3" H 4665 5223 50  0000 C CNN
 F 2 "" H 4650 5050 50  0001 C CNN
 F 3 "" H 4650 5050 50  0001 C CNN
@@
 	1    0    0    -1
 $EndComp
+Text GLabel 4150 5350 0    50   Input ~ 0
+QSPI_IO0
+Text GLabel 5150 5350 2    50   Input ~ 0
+QSPI_IO1
+Text GLabel 4150 5650 0    50   Input ~ 0
+QSPI_IO2
+Text GLabel 4150 5750 0    50   Input ~ 0
+QSPI_IO3
 Wire Wire Line
-	4650 5050 4650 5150
+	4250 5350 4150 5350
+Wire Wire Line
+	4250 5450 4150 5450
+Wire Wire Line
+	4250 5550 4150 5550
+Wire Wire Line
+	4250 5650 4150 5650
+Wire Wire Line
+	4250 5750 4150 5750
+Wire Wire Line
+	5050 5350 5150 5350
+Text GLabel 4150 5450 0    50   Input ~ 0
+QSPI_SCK
+Text GLabel 4150 5550 0    50   Input ~ 0
+QSPI_CS
+Text Notes 3250 4750 0    100  ~ 0
+MEMORY
+$Comp
+L power:VCC #PWR0245
+U 1 1 5F256590
+P 15100 1450
+F 0 "#PWR0245" H 15100 1300 50  0001 C CNN
+F 1 "VCC" H 15115 1623 50  0000 C CNN
+F 2 "" H 15100 1450 50  0001 C CNN
+F 3 "" H 15100 1450 50  0001 C CNN
+	1    15100 1450
+	1    0    0    -1
+$EndComp
+Wire Wire Line
+	15100 1450 15100 1500
+Wire Wire Line
+	15100 1500 15300 1500
+Connection ~ 15300 1500
+Wire Wire Line
+	15300 1500 15300 1550
+NoConn ~ 4500 1700
 $EndSCHEMATC

Commit message: update
Connections:
- net at C24.2, U7.16 (AOUT1): now also J1.2 (Pin_2); no longer J1.1 (Pin_1)
- net at C24.1, U7.2 (AOUT2): now also J1.1 (Pin_1); no longer J1.2 (Pin_2)
Changed lines of the file:
@@
 NoConn ~ 15050 5800
-$Comp
-L Connector_Generic:Conn_01x02 J1
-U 1 1 5F0DE9E4
-P 3400 7250
-F 0 "J1" H 3480 7242 50  0000 L CNN
-F 1 "MOTOR-A_CONN" H 3480 7151 50  0000 L CNN
-F 2 "GiraffeTech-Connector:DINKLE_EK500V-2P" H 3400 7250 50  0001 C CNN
-F 3 "~" H 3400 7250 50  0001 C CNN
-	1    3400 7250
-	1    0    0    -1
-$EndComp
 $Comp
 L Connector_Generic:Conn_01x02 J2
@@
 	2350 7200 2350 7100
 NoConn ~ 2650 7800
-Wire Wire Line
-	2700 7250 3200 7250
 $Comp
 L Device:C_Small C24
@@
 	15300 1500 15300 1550
 NoConn ~ 4500 1700
+Wire Wire Line
+	2700 7250 3200 7250
+$Comp
+L Connector_Generic:Conn_01x02 J1
+U 1 1 5F0DE9E4
+P 3400 7350
+F 0 "J1" H 3480 7342 50  0000 L CNN
+F 1 "MOTOR-A_CONN" H 3480 7251 50  0000 L CNN
+F 2 "GiraffeTech-Connector:DINKLE_EK500V-2P" H 3400 7350 50  0001 C CNN
+F 3 "~" H 3400 7350 50  0001 C CNN
+	1    3400 7350
+	1    0    0    1
+$EndComp
 $EndSCHEMATC

Commit message: update to 4-layer
Connections:
- net +3V3: now also C34.1, C35.1, C36.1, C37.1, C38.1, C39.1, C40.1, C41.1
- net +5V: no longer C34.1, C35.1, C36.1, C37.1, C38.1, C39.1, C40.1, C41.1
Changed lines of the file:
@@
-$EndComp
-$Comp
-L power:+5V #PWR0209
-U 1 1 5F37A0C0
-P 11000 2000
-F 0 "#PWR0209" H 11000 1850 50  0001 C CNN
-F 1 "+5V" H 11015 2173 50  0000 C CNN
-F 2 "" H 11000 2000 50  0001 C CNN
-F 3 "" H 11000 2000 50  0001 C CNN
-	1    11000 2000
-	1    0    0    -1
 $EndComp
 $Comp
@@
 $EndComp
 $Comp
-L power:+5V #PWR0211
-U 1 1 5F37A0E0
-P 11450 2000
-F 0 "#PWR0211" H 11450 1850 50  0001 C CNN
-F 1 "+5V" H 11465 2173 50  0000 C CNN
-F 2 "" H 11450 2000 50  0001 C CNN
-F 3 "" H 11450 2000 50  0001 C CNN
-	1    11450 2000
-	1    0    0    -1
-$EndComp
-$Comp
 L power:GND #PWR0212
 U 1 1 5F37A0EA
@@
 $EndComp
 $Comp
-L power:+5V #PWR0213
-U 1 1 5F3DA9A9
-P 11000 2900
-F 0 "#PWR0213" H 11000 2750 50  0001 C CNN
-F 1 "+5V" H 11015 3073 50  0000 C CNN
-F 2 "" H 11000 2900 50  0001 C CNN
-F 3 "" H 11000 2900 50  0001 C CNN
-	1    11000 2900
-	1    0    0    -1
-$EndComp
-$Comp
 L power:GND #PWR0214
 U 1 1 5F3DA9B3
@@
 $EndComp
 $Comp
-L power:+5V #PWR0215
-U 1 1 5F3DA9C9
-P 11450 2900
-F 0 "#PWR0215" H 11450 2750 50  0001 C CNN
-F 1 "+5V" H 11465 3073 50  0000 C CNN
-F 2 "" H 11450 2900 50  0001 C CNN
-F 3 "" H 11450 2900 50  0001 C CNN
-	1    11450 2900
-	1    0    0    -1
-$EndComp
-$Comp
 L power:GND #PWR0216
 U 1 1 5F3DA9D3
@@
 $EndComp
 $Comp
-L power:+5V #PWR0217
-U 1 1 5F5204D9
-P 11000 3800
-F 0 "#PWR0217" H 11000 3650 50  0001 C CNN
-F 1 "+5V" H 11015 3973 50  0000 C CNN
-F 2 "" H 11000 3800 50  0001 C CNN
-F 3 "" H 11000 3800 50  0001 C CNN
-	1    11000 3800
-	1    0    0    -1
-$EndComp
-$Comp
 L power:GND #PWR0218
 U 1 1 5F5204E3
@@
 $EndComp
 $Comp
-L power:+5V #PWR0219
-U 1 1 5F5204F9
-P 11450 3800
-F 0 "#PWR0219" H 11450 3650 50  0001 C CNN
-F 1 "+5V" H 11465 3973 50  0000 C CNN
-F 2 "" H 11450 3800 50  0001 C CNN
-F 3 "" H 11450 3800 50  0001 C CNN
-	1    11450 3800
-	1    0    0    -1
-$EndComp
-$Comp
 L power:GND #PWR0220
 U 1 1 5F520503
@@
 $EndComp
 $Comp
-L power:+5V #PWR0221
-U 1 1 5F520519
-P 11000 4700
-F 0 "#PWR0221" H 11000 4550 50  0001 C CNN
-F 1 "+5V" H 11015 4873 50  0000 C CNN
-F 2 "" H 11000 4700 50  0001 C CNN
-F 3 "" H 11000 4700 50  0001 C CNN
-	1    11000 4700
-	1    0    0    -1
-$EndComp
-$Comp
 L power:GND #PWR0222
 U 1 1 5F520523
@@
 F 3 "~" H 11450 4900 50  0001 C CNN
 	1    11450 4900
-	1    0    0    -1
-$EndComp
-$Comp
-L power:+5V #PWR0223
-U 1 1 5F520539
-P 11450 4700
-F 0 "#PWR0223" H 11450 4550 50  0001 C CNN
-F 1 "+5V" H 11465 4873 50  0000 C CNN
-F 2 "" H 11450 4700 50  0001 C CNN
-F 3 "" H 11450 4700 50  0001 C CNN
-	1    11450 4700
 	1    0    0    -1
 $EndComp
@@
 	1    0    0    1
 $EndComp
+$Comp
+L power:+3V3 #PWR?
+U 1 1 5EF19B50
+P 11000 2000
+F 0 "#PWR?" H 11000 1850 50  0001 C CNN
+F 1 "+3V3" H 11015 2173 50  0000 C CNN
+F 2 "" H 11000 2000 50  0001 C CNN
+F 3 "" H 11000 2000 50  0001 C CNN
+	1    11000 2000
+	1    0    0    -1
+$EndComp
+$Comp
+L power:+3V3 #PWR?
+U 1 1 5EF1A50D
+P 11450 2000
+F 0 "#PWR?" H 11450 1850 50  0001 C CNN
+F 1 "+3V3" H 11465 2173 50  0000 C CNN
+F 2 "" H 11450 2000 50  0001 C CNN
+F 3 "" H 11450 2000 50  0001 C CNN
+	1    11450 2000
+	1    0    0    -1
+$EndComp
+$Comp
+L power:+3V3 #PWR?
+U 1 1 5EF1E310
+P 11000 2900
+F 0 "#PWR?" H 11000 2750 50  0001 C CNN
+F 1 "+3V3" H 11015 3073 50  0000 C CNN
+F 2 "" H 11000 2900 50  0001 C CNN
+F 3 "" H 11000 2900 50  0001 C CNN
+	1    11000 2900
+	1    0    0    -1
+$EndComp
+$Comp
+L power:+3V3 #PWR?
+U 1 1 5EF1E31A
+P 11450 2900
+F 0 "#PWR?" H 11450 2750 50  0001 C CNN
+F 1 "+3V3" H 11465 3073 50  0000 C CNN
+F 2 "" H 11450 2900 50  0001 C CNN
+F 3 "" H 11450 2900 50  0001 C CNN
+	1    11450 2900
+	1    0    0    -1
+$EndComp
+$Comp
+L power:+3V3 #PWR?
+U 1 1 5EF9C617
+P 11000 3800
+F 0 "#PWR?" H 11000 3650 50  0001 C CNN
+F 1 "+3V3" H 11015 3973 50  0000 C CNN
+F 2 "" H 11000 3800 50  0001 C CNN
+F 3 "" H 11000 3800 50  0001 C CNN
+	1    11000 3800
+	1    0    0    -1
+$EndComp
+$Comp
+L power:+3V3 #PWR?
+U 1 1 5EF9C621
+P 11450 3800
+F 0 "#PWR?" H 11450 3650 50  0001 C CNN
+F 1 "+3V3" H 11465 3973 50  0000 C CNN
+F 2 "" H 11450 3800 50  0001 C CNN
+F 3 "" H 11450 3800 50  0001 C CNN
+	1    11450 3800
+	1    0    0    -1
+$EndComp
+$Comp
+L power:+3V3 #PWR?
+U 1 1 5F0185B8
+P 11000 4700
+F 0 "#PWR?" H 11000 4550 50  0001 C CNN
+F 1 "+3V3" H 11015 4873 50  0000 C CNN
+F 2 "" H 11000 4700 50  0001 C CNN
+F 3 "" H 11000 4700 50  0001 C CNN
+	1    11000 4700
+	1    0    0    -1
+$EndComp
+$Comp
+L power:+3V3 #PWR?
+U 1 1 5F0185C2
+P 11450 4700
+F 0 "#PWR?" H 11450 4550 50  0001 C CNN
+F 1 "+3V3" H 11465 4873 50  0000 C CNN
+F 2 "" H 11450 4700 50  0001 C CNN
+F 3 "" H 11450 4700 50  0001 C CNN
+	1    11450 4700
+	1    0    0    -1
+$EndComp
 $EndSCHEMATC
