File: MP_SamBaseBoard_V1_DraftDesign/MP_SamBaseBoard_V1.kicad_pcb (KiCad board)
At the start: 2 copper layers, 86 x 60 mm, 60 parts

Commit message: update
Parts:
- added G***: LOGO, GiraffeTech-Utility:basebaord_text3, F.Cu at (288.4, 122.5)
- added MS2: FEATHERWING_NODIM, GiraffeTech-Connector:Adafruit-Feather_WoMountPoint, F.Cu at (335.6, 111.1)
- added REF**: C_0603_1608Metric, Capacitor_SMD:C_0603_1608Metric, F.Cu at (292.8, 110.0)
- added REF**: C_0603_1608Metric, Capacitor_SMD:C_0603_1608Metric, F.Cu at (315.2, 94.5)
- added REF**: C_0603_1608Metric, Capacitor_SMD:C_0603_1608Metric, F.Cu at (315.2, 97.5)
- added REF**: C_0603_1608Metric, Capacitor_SMD:C_0603_1608Metric, F.Cu at (322.8, 94.5)
- added REF**: C_0603_1608Metric, Capacitor_SMD:C_0603_1608Metric, F.Cu at (322.8, 97.5)
- added REF**: C_0603_1608Metric, Capacitor_SMD:C_0603_1608Metric, F.Cu at (330.2, 97.5)
- added REF**: C_0603_1608Metric, Capacitor_SMD:C_0603_1608Metric, F.Cu at (343.2, 110.8)
- added REF**: C_0603_1608Metric, Capacitor_SMD:C_0603_1608Metric, F.Cu at (341.8, 110.8)
- added REF**: C_0603_1608Metric, Capacitor_SMD:C_0603_1608Metric, F.Cu at (330.2, 94.5)
- added REF**: C_0603_1608Metric, Capacitor_SMD:C_0603_1608Metric, F.Cu at (340.2, 110.8)
- added REF**: PinHeader_1x03_P2.54mm_Vertical, Connector_PinHeader_2.54mm:PinHeader_1x03_P2.54mm_Vertical, F.Cu at (260.8, 104.5)
- added REF**: C_0603_1608Metric, Capacitor_SMD:C_0603_1608Metric, F.Cu at (289.8, 110.0)
- added REF**: Symbol_Barrel_Polarity, Symbol:Symbol_Barrel_Polarity, F.Cu at (343.2, 139.0)
- added REF**: QFN-16-1EP_3x3mm_Pitch0.5mm, GiraffeTech-Maxim:QFN-16-1EP_3x3mm_Pitch0.5mm, F.Cu at (272.8, 140.0)
- added REF**: PinHeader_2x03_P2.54mm_Vertical, Connector_PinHeader_2.54mm:PinHeader_2x03_P2.54mm_Vertical, F.Cu at (281.2, 145.2)
- added REF**: C_0603_1608Metric, Capacitor_SMD:C_0603_1608Metric, F.Cu at (276.8, 101.2)
- added REF**: QFN-16-1EP_3x3mm_Pitch0.5mm, GiraffeTech-Maxim:QFN-16-1EP_3x3mm_Pitch0.5mm, F.Cu at (298.2, 137.5)
- added REF**: BarrelJack_Horizontal, Connector_BarrelJack:BarrelJack_Horizontal, F.Cu at (324.8, 138.5)
- added REF**: C_0603_1608Metric, Capacitor_SMD:C_0603_1608Metric, F.Cu at (340.8, 141.5)
- added REF**: JST_PH_B4B-PH-K_1x04_P2.00mm_Vertical, Connector_JST:JST_PH_B4B-PH-K_1x04_P2.00mm_Vertical, F.Cu at (312.0, 95.2)
- added REF**: SW_SPST_B3S-1000, Button_Switch_SMD:SW_SPST_B3S-1000, F.Cu at (272.0, 97.8)
- added REF**: SW_SPST_B3S-1000, Button_Switch_SMD:SW_SPST_B3S-1000, F.Cu at (323.8, 122.5)
- added REF**: C_0603_1608Metric, Capacitor_SMD:C_0603_1608Metric, F.Cu at (278.2, 140.0)
- added REF**: R_0603_1608Metric, Resistor_SMD:R_0603_1608Metric, F.Cu at (287.0, 131.0)
- added REF**: C_0603_1608Metric, Capacitor_SMD:C_0603_1608Metric, F.Cu at (288.0, 138.0)
- added REF**: Sensirion_SHT3x, GiraffeTech-Sensiroin:Sensirion_SHT3x, F.Cu at (341.0, 102.2)
- added REF**: LED_WS2812B_PLCC4_5.0x5.0mm_P3.2mm, LED_SMD:LED_WS2812B_PLCC4_5.0x5.0mm_P3.2mm, F.Cu at (272.0, 107.0)
- added REF**: C_0603_1608Metric, Capacitor_SMD:C_0603_1608Metric, F.Cu at (289.5, 138.0)
- added REF**: Dinkle_ED350V_2Pins_Pitch3.5mm, GiraffeTech-Connector:TerminalBlock_Dinkle_ED350V_1x02_P3.50mm_Horizontal, F.Cu at (333.2, 149.0)
- added REF**: DINKLE_EK500V-2P, GiraffeTech-Connector:DINKLE_EK500V-2P, F.Cu at (292.8, 147.5)
- added REF**: LED_0603_1608Metric, LED_SMD:LED_0603_1608Metric, F.Cu at (342.0, 133.0)
- added REF**: MountingHole_3.5mm, MountingHole:MountingHole_3.5mm, F.Cu at (340.8, 148.5)
- added REF**: SOT-23-6, Package_TO_SOT_SMD:SOT-23-6, F.Cu at (317.0, 138.0)
- added REF**: C_0603_1608Metric, Capacitor_SMD:C_0603_1608Metric, F.Cu at (276.8, 140.0)
- added REF**: C_0603_1608Metric, Capacitor_SMD:C_0603_1608Metric, F.Cu at (303.5, 137.5)
- added REF**: C_0603_1608Metric, Capacitor_SMD:C_0603_1608Metric, F.Cu at (302.0, 137.5)
- added REF**: SOT-23-5, Package_TO_SOT_SMD:SOT-23-5, F.Cu at (337.8, 139.2)
- added REF**: SOT-23-6, Package_TO_SOT_SMD:SOT-23-6, F.Cu at (312.5, 138.0)
- added REF**: Dinkle_ED350V_2Pins_Pitch3.5mm, GiraffeTech-Connector:TerminalBlock_Dinkle_ED350V_1x02_P3.50mm_Horizontal, F.Cu at (274.0, 148.8)
- added REF**: DINKLE_EK500V-2P, GiraffeTech-Connector:DINKLE_EK500V-2P, F.Cu at (303.5, 147.5)
- added REF**: GTK_TFMS08TK-PP-02, GiraffeTech-Connector:GTK_TFMS08TK-PP-02, F.Cu at (299.5, 97.8)
- added REF**: JST_PH_B4B-PH-K_1x04_P2.00mm_Vertical, Connector_JST:JST_PH_B4B-PH-K_1x04_P2.00mm_Vertical, F.Cu at (334.5, 95.2)
- added REF**: MountingHole_3.5mm, MountingHole:MountingHole_3.5mm, F.Cu at (262.8, 148.5)
- added REF**: JST_PH_B4B-PH-K_1x04_P2.00mm_Vertical, Connector_JST:JST_PH_B4B-PH-K_1x04_P2.00mm_Vertical, F.Cu at (327.0, 95.2)
- added REF**: C_0603_1608Metric, Capacitor_SMD:C_0603_1608Metric, F.Cu at (269.2, 147.5)
- added REF**: USB_Micro-B_Amphenol_10118193_Horizontal, GiraffeTech-Connector:USB_Micro-B_Amphenol_10118193_Horizontal, F.Cu at (343.2, 122.5)
- added REF**: C_0603_1608Metric, Capacitor_SMD:C_0603_1608Metric, F.Cu at (293.0, 137.5)
- added REF**: C_0603_1608Metric, Capacitor_SMD:C_0603_1608Metric, F.Cu at (294.5, 137.5)
- added REF**: C_0603_1608Metric, Capacitor_SMD:C_0603_1608Metric, F.Cu at (340.8, 138.2)
- added REF**: LGA-16_3x3mm_P0.5mm_LayoutBorder3x5y, Package_LGA:LGA-16_3x3mm_P0.5mm_LayoutBorder3x5y, F.Cu at (341.0, 106.5)
- added REF**: JST_PH_B4B-PH-K_1x04_P2.00mm_Vertical, Connector_JST:JST_PH_B4B-PH-K_1x04_P2.00mm_Vertical, F.Cu at (319.5, 95.2)
- added REF**: R_0603_1608Metric, Resistor_SMD:R_0603_1608Metric, F.Cu at (288.5, 131.0)
- added REF**: C_0603_1608Metric, Capacitor_SMD:C_0603_1608Metric, F.Cu at (337.8, 142.2)
- added REF**: LED_0603_1608Metric, LED_SMD:LED_0603_1608Metric, F.Cu at (333.2, 139.2)
- added REF**: SW_SPST_B3S-1000, Button_Switch_SMD:SW_SPST_B3S-1000, F.Cu at (281.5, 97.8)
- added REF**: C_0603_1608Metric, Capacitor_SMD:C_0603_1608Metric, F.Cu at (269.2, 150.5)
- added REF**: PinHeader_2x05_P1.27mm_Vertical, Connector_PinHeader_1.27mm:PinHeader_2x05_P1.27mm_Vertical, F.Cu at (278.9, 135.6)
- added REF**: JST_PH_B4B-PH-K_1x04_P2.00mm_Vertical, Connector_JST:JST_PH_B4B-PH-K_1x04_P2.00mm_Vertical, F.Cu at (304.5, 95.2)
- added REF**: LED_WS2812B_PLCC4_5.0x5.0mm_P3.2mm, LED_SMD:LED_WS2812B_PLCC4_5.0x5.0mm_P3.2mm, F.Cu at (281.8, 107.0)
- added REF**: MountingHole_3.5mm, MountingHole:MountingHole_3.5mm, F.Cu at (262.8, 96.5)
- added REF**: ESP32-WROOM-32_ButtLess, GiraffeTech-NodeMCU:ESP32-WROOM-32_ButtLess, F.Cu at (274.8, 122.5)
- added REF**: R_0603_1608Metric, Resistor_SMD:R_0603_1608Metric, F.Cu at (312.5, 135.2)
- added REF**: TQFP-64_10x10mm_P0.5mm, Package_QFP:TQFP-64_10x10mm_P0.5mm, F.Cu at (301.8, 122.5)
- added REF**: DINKLE_EK500V-2P, GiraffeTech-Connector:DINKLE_EK500V-2P, F.Cu at (314.2, 147.5)
- added REF**: MountingHole_3.5mm, MountingHole:MountingHole_3.5mm, F.Cu at (340.8, 96.5)
- added REF**: R_0603_1608Metric, Resistor_SMD:R_0603_1608Metric, F.Cu at (317.0, 135.2)
- added REF**: C_0603_1608Metric, Capacitor_SMD:C_0603_1608Metric, F.Cu at (338.8, 110.8)
- added REF**: C_0603_1608Metric, Capacitor_SMD:C_0603_1608Metric, F.Cu at (267.2, 101.2)
- added REF**: C_0603_1608Metric, Capacitor_SMD:C_0603_1608Metric, F.Cu at (307.8, 97.5)
- added REF**: C_0603_1608Metric, Capacitor_SMD:C_0603_1608Metric, F.Cu at (307.8, 94.5)
- moved REF** 127.4 mm to (264.5, 138.2), turned to 90 degrees
Other:
- board size 86 x 60 mm -> 86 x 131.5 mm
- board text added: "P1"
- board text added: "P2"
- board text added: "P3"
- board text added: "PIEZO BUZZER"

Commit message: update
Parts:
- added G***: LOGO, GiraffeTech-Utility:basebaord_text3, F.Cu at (198.2, 122.5)
- added G***: LOGO, GiraffeTech-Utility:basebaord_text3, F.Cu at (313.2, 191.8)
- added MS2: FEATHERWING_NODIM, GiraffeTech-Connector:Adafruit-Feather_WoMountPoint, F.Cu at (248.2, 111.1)
- added MS2: FEATHERWING_NODIM, GiraffeTech-Connector:Adafruit-Feather_WoMountPoint, F.Cu at (344.8, 180.3)
- added REF**: SW_SPDT_CK-JS102011JCQN, GiraffeTech-Electromechanical:SW_SPDT_CK-JS102011JCQN, F.Cu at (240.0, 133.0)
- added REF**: QFN-16-1EP_3x3mm_Pitch0.5mm, GiraffeTech-Maxim:QFN-16-1EP_3x3mm_Pitch0.5mm, F.Cu at (203.2, 137.5)
- added REF**: Sensirion_SHT3x, GiraffeTech-Sensiroin:Sensirion_SHT3x, F.Cu at (341.0, 173.5)
- added REF**: LED_0603_1608Metric, LED_SMD:LED_0603_1608Metric, F.Cu at (333.2, 208.5)
- added REF**: C_0603_1608Metric, Capacitor_SMD:C_0603_1608Metric, F.Cu at (337.8, 211.5)
- added REF**: C_0603_1608Metric, Capacitor_SMD:C_0603_1608Metric, F.Cu at (340.8, 207.5)
- added REF**: JST_PH_B4B-PH-K_1x04_P2.00mm_Vertical, Connector_JST:JST_PH_B4B-PH-K_1x04_P2.00mm_Vertical, F.Cu at (327.0, 166.2)
- added REF**: C_0603_1608Metric, Capacitor_SMD:C_0603_1608Metric, F.Cu at (289.5, 207.2)
- added REF**: JST_PH_B4B-PH-K_1x04_P2.00mm_Vertical, Connector_JST:JST_PH_B4B-PH-K_1x04_P2.00mm_Vertical, F.Cu at (304.5, 166.2)
- added REF**: C_0603_1608Metric, Capacitor_SMD:C_0603_1608Metric, F.Cu at (322.8, 168.5)
- added REF**: C_0603_1608Metric, Capacitor_SMD:C_0603_1608Metric, F.Cu at (322.8, 165.5)
- added REF**: JST_PH_B4B-PH-K_1x04_P2.00mm_Vertical, Connector_JST:JST_PH_B4B-PH-K_1x04_P2.00mm_Vertical, F.Cu at (312.0, 166.2)
- added REF**: MagneticBuzzer_CUI_CMT-8504-100-SMT, Buzzer_Beeper:MagneticBuzzer_CUI_CMT-8504-100-SMT, F.Cu at (174.8, 138.0)
- added REF**: R_0603_1608Metric, Resistor_SMD:R_0603_1608Metric, F.Cu at (288.5, 200.2)
- added REF**: LED_0603_1608Metric, LED_SMD:LED_0603_1608Metric, F.Cu at (342.0, 202.2)
- added REF**: SOT-23-5, Package_TO_SOT_SMD:SOT-23-5, F.Cu at (337.8, 208.5)
- added REF**: C_0603_1608Metric, Capacitor_SMD:C_0603_1608Metric, F.Cu at (302.0, 206.8)
- added REF**: C_0603_1608Metric, Capacitor_SMD:C_0603_1608Metric, F.Cu at (307.8, 168.5)
- added REF**: SOT-23-6, Package_TO_SOT_SMD:SOT-23-6, F.Cu at (312.5, 207.2)
- added REF**: ESP32-WROOM-32_ButtLess, GiraffeTech-NodeMCU:ESP32-WROOM-32_ButtLess, F.Cu at (280.8, 191.8)
- added REF**: MountingHole_3.5mm, MountingHole:MountingHole_3.5mm, F.Cu at (268.8, 167.8)
- added REF**: DINKLE_EK500V-2P, GiraffeTech-Connector:DINKLE_EK500V-2P, F.Cu at (304.0, 216.8)
- added REF**: PinHeader_1x03_P2.54mm_Vertical, Connector_PinHeader_2.54mm:PinHeader_1x03_P2.54mm_Vertical, F.Cu at (266.5, 175.0)
- added REF**: DINKLE_EK500V-2P, GiraffeTech-Connector:DINKLE_EK500V-2P, F.Cu at (198.5, 147.5)
- added REF**: C_0603_1608Metric, Capacitor_SMD:C_0603_1608Metric, F.Cu at (193.0, 138.0)
- added REF**: Dinkle_ED350V_2Pins_Pitch3.5mm, GiraffeTech-Connector:TerminalBlock_Dinkle_ED350V_1x02_P3.50mm_Horizontal, F.Cu at (238.2, 149.0)
- added REF**: C_0603_1608Metric, Capacitor_SMD:C_0603_1608Metric, F.Cu at (208.5, 137.5)
- added REF**: QFN-16-1EP_3x3mm_Pitch0.5mm, GiraffeTech-Maxim:QFN-16-1EP_3x3mm_Pitch0.5mm, F.Cu at (182.8, 140.0)
- added REF**: MountingHole_3.5mm, MountingHole:MountingHole_3.5mm, F.Cu at (173.8, 148.5)
- added REF**: MountingHole_3.5mm, MountingHole:MountingHole_3.5mm, F.Cu at (245.8, 148.5)
- added REF**: SOT-23-6, Package_TO_SOT_SMD:SOT-23-6, F.Cu at (222.0, 138.0)
- added REF**: SW_SPST_B3S-1000, Button_Switch_SMD:SW_SPST_B3S-1000, F.Cu at (184.8, 96.2)
- added REF**: PinHeader_2x05_P1.27mm_Vertical, Connector_PinHeader_1.27mm:PinHeader_2x05_P1.27mm_Vertical, F.Cu at (199.5, 134.0)
- added REF**: LGA-16_3x3mm_P0.5mm_LayoutBorder3x5y, Package_LGA:LGA-16_3x3mm_P0.5mm_LayoutBorder3x5y, F.Cu at (246.0, 108.5)
- added REF**: JST_PH_B4B-PH-K_1x04_P2.00mm_Vertical, Connector_JST:JST_PH_B4B-PH-K_1x04_P2.00mm_Vertical, F.Cu at (239.5, 95.0)
- added REF**: C_0603_1608Metric, Capacitor_SMD:C_0603_1608Metric, F.Cu at (220.2, 97.2)
- added REF**: R_0603_1608Metric, Resistor_SMD:R_0603_1608Metric, F.Cu at (192.0, 134.0)
- added REF**: C_0603_1608Metric, Capacitor_SMD:C_0603_1608Metric, F.Cu at (194.8, 110.2)
- added REF**: PinHeader_2x03_P2.54mm_Vertical, Connector_PinHeader_2.54mm:PinHeader_2x03_P2.54mm_Vertical, F.Cu at (187.2, 145.8)
- added REF**: USB_Micro-B_Amphenol_10118193_Horizontal, GiraffeTech-Connector:USB_Micro-B_Amphenol_10118193_Horizontal, F.Cu at (248.2, 122.5)
- added REF**: R_0603_1608Metric, Resistor_SMD:R_0603_1608Metric, F.Cu at (217.5, 135.2)
- added REF**: SW_SPST_B3S-1000, Button_Switch_SMD:SW_SPST_B3S-1000, F.Cu at (228.8, 122.5)
- added REF**: SW_SPST_B3S-1000, Button_Switch_SMD:SW_SPST_B3S-1000, F.Cu at (184.8, 104.0)
- added REF**: C_0603_1608Metric, Capacitor_SMD:C_0603_1608Metric, F.Cu at (235.2, 97.2)
- added REF**: JST_PH_B4B-PH-K_1x04_P2.00mm_Vertical, Connector_JST:JST_PH_B4B-PH-K_1x04_P2.00mm_Vertical, F.Cu at (224.5, 95.0)
- added REF**: C_0603_1608Metric, Capacitor_SMD:C_0603_1608Metric, F.Cu at (199.5, 137.5)
- added REF**: R_0603_1608Metric, Resistor_SMD:R_0603_1608Metric, F.Cu at (222.0, 135.2)
- added REF**: MountingHole_3.5mm, MountingHole:MountingHole_3.5mm, F.Cu at (245.8, 96.5)
- added REF**: DINKLE_EK500V-2P, GiraffeTech-Connector:DINKLE_EK500V-2P, F.Cu at (219.8, 147.5)
- added REF**: TQFP-64_10x10mm_P0.5mm, Package_QFP:TQFP-64_10x10mm_P0.5mm, F.Cu at (210.0, 122.5)
- added REF**: C_0603_1608Metric, Capacitor_SMD:C_0603_1608Metric, F.Cu at (197.8, 110.2)
- added REF**: C_0603_1608Metric, Capacitor_SMD:C_0603_1608Metric, F.Cu at (212.8, 94.2)
- added REF**: Dinkle_ED350V_2Pins_Pitch3.5mm, GiraffeTech-Connector:TerminalBlock_Dinkle_ED350V_1x02_P3.50mm_Horizontal, F.Cu at (181.5, 149.0)
- added REF**: C_0603_1608Metric, Capacitor_SMD:C_0603_1608Metric, F.Cu at (245.8, 141.5)
- added REF**: BarrelJack_Horizontal, Connector_BarrelJack:BarrelJack_Horizontal, F.Cu at (229.8, 138.5)
- added REF**: Sensirion_SHT3x, GiraffeTech-Sensiroin:Sensirion_SHT3x, F.Cu at (246.0, 104.2)
- added REF**: LED_0603_1608Metric, LED_SMD:LED_0603_1608Metric, F.Cu at (238.2, 139.2)
- added REF**: C_0603_1608Metric, Capacitor_SMD:C_0603_1608Metric, F.Cu at (242.8, 142.2)
- added REF**: C_0603_1608Metric, Capacitor_SMD:C_0603_1608Metric, F.Cu at (245.8, 138.2)
- added REF**: JST_PH_B4B-PH-K_1x04_P2.00mm_Vertical, Connector_JST:JST_PH_B4B-PH-K_1x04_P2.00mm_Vertical, F.Cu at (232.0, 95.0)
- added REF**: C_0603_1608Metric, Capacitor_SMD:C_0603_1608Metric, F.Cu at (194.5, 138.0)
- added REF**: JST_PH_B4B-PH-K_1x04_P2.00mm_Vertical, Connector_JST:JST_PH_B4B-PH-K_1x04_P2.00mm_Vertical, F.Cu at (209.5, 95.0)
- added REF**: C_0603_1608Metric, Capacitor_SMD:C_0603_1608Metric, F.Cu at (227.8, 97.2)
- added REF**: C_0603_1608Metric, Capacitor_SMD:C_0603_1608Metric, F.Cu at (227.8, 94.2)
- added REF**: C_0603_1608Metric, Capacitor_SMD:C_0603_1608Metric, F.Cu at (198.0, 137.5)
- added REF**: JST_PH_B4B-PH-K_1x04_P2.00mm_Vertical, Connector_JST:JST_PH_B4B-PH-K_1x04_P2.00mm_Vertical, F.Cu at (217.0, 95.0)
- added REF**: R_0603_1608Metric, Resistor_SMD:R_0603_1608Metric, F.Cu at (193.5, 134.0)
- added REF**: LED_0603_1608Metric, LED_SMD:LED_0603_1608Metric, F.Cu at (247.0, 133.0)
- added REF**: SOT-23-5, Package_TO_SOT_SMD:SOT-23-5, F.Cu at (242.8, 139.2)
- added REF**: C_0603_1608Metric, Capacitor_SMD:C_0603_1608Metric, F.Cu at (207.0, 137.5)
- added REF**: DINKLE_EK500V-2P, GiraffeTech-Connector:DINKLE_EK500V-2P, F.Cu at (209.0, 147.5)
- added REF**: PinHeader_1x03_P2.54mm_Vertical, Connector_PinHeader_2.54mm:PinHeader_1x03_P2.54mm_Vertical, F.Cu at (171.5, 103.8)
- added REF**: MountingHole_3.5mm, MountingHole:MountingHole_3.5mm, F.Cu at (173.8, 96.5)
- added REF**: SOT-23-6, Package_TO_SOT_SMD:SOT-23-6, F.Cu at (217.5, 138.0)
- added REF**: C_0603_1608Metric, Capacitor_SMD:C_0603_1608Metric, F.Cu at (212.8, 97.2)
- added REF**: Symbol_Barrel_Polarity, Symbol:Symbol_Barrel_Polarity, F.Cu at (248.2, 139.0)
- added REF**: ESP32-WROOM-32_ButtLess, GiraffeTech-NodeMCU:ESP32-WROOM-32_ButtLess, F.Cu at (185.8, 122.5)
- added REF**: SW_SPST_B3S-1000, Button_Switch_SMD:SW_SPST_B3S-1000, F.Cu at (279.8, 175.2)
- added REF**: SW_SPST_B3S-1000, Button_Switch_SMD:SW_SPST_B3S-1000, F.Cu at (279.8, 167.5)
- added REF**: C_0603_1608Metric, Capacitor_SMD:C_0603_1608Metric, F.Cu at (340.8, 210.8)
- added REF**: C_0603_1608Metric, Capacitor_SMD:C_0603_1608Metric, F.Cu at (294.5, 206.8)
- added REF**: C_0603_1608Metric, Capacitor_SMD:C_0603_1608Metric, F.Cu at (293.0, 206.8)
- added REF**: Symbol_Barrel_Polarity, Symbol:Symbol_Barrel_Polarity, F.Cu at (343.2, 208.2)
- added REF**: C_0603_1608Metric, Capacitor_SMD:C_0603_1608Metric, F.Cu at (315.2, 165.5)
- added REF**: GTK_TFMS08TK-PP-02, GiraffeTech-Connector:GTK_TFMS08TK-PP-02, F.Cu at (299.0, 168.8)
- added REF**: C_0603_1608Metric, Capacitor_SMD:C_0603_1608Metric, F.Cu at (330.2, 165.5)
- added REF**: C_0603_1608Metric, Capacitor_SMD:C_0603_1608Metric, F.Cu at (220.2, 94.2)
- added REF**: QFN-16-1EP_3x3mm_Pitch0.5mm, GiraffeTech-Maxim:QFN-16-1EP_3x3mm_Pitch0.5mm, F.Cu at (298.2, 206.8)
- added REF**: MagneticBuzzer_CUI_CMT-8504-100-SMT, Buzzer_Beeper:MagneticBuzzer_CUI_CMT-8504-100-SMT, F.Cu at (270.0, 206.8)
- added REF**: DINKLE_EK500V-2P, GiraffeTech-Connector:DINKLE_EK500V-2P, F.Cu at (293.5, 216.8)
- added REF**: C_0603_1608Metric, Capacitor_SMD:C_0603_1608Metric, F.Cu at (288.0, 207.2)
- added REF**: Dinkle_ED350V_2Pins_Pitch3.5mm, GiraffeTech-Connector:TerminalBlock_Dinkle_ED350V_1x02_P3.50mm_Horizontal, F.Cu at (333.2, 218.2)
- added REF**: C_0603_1608Metric, Capacitor_SMD:C_0603_1608Metric, F.Cu at (303.5, 206.8)
- added REF**: QFN-16-1EP_3x3mm_Pitch0.5mm, GiraffeTech-Maxim:QFN-16-1EP_3x3mm_Pitch0.5mm, F.Cu at (278.5, 208.5)
- added REF**: MountingHole_3.5mm, MountingHole:MountingHole_3.5mm, F.Cu at (268.8, 215.8)
- added REF**: MountingHole_3.5mm, MountingHole:MountingHole_3.5mm, F.Cu at (340.8, 215.8)
- added REF**: SOT-23-6, Package_TO_SOT_SMD:SOT-23-6, F.Cu at (317.0, 207.2)
- added REF**: GTK_TFMS08TK-PP-02, GiraffeTech-Connector:GTK_TFMS08TK-PP-02, F.Cu at (204.0, 97.5)
- added REF**: PinHeader_2x05_P1.27mm_Vertical, Connector_PinHeader_1.27mm:PinHeader_2x05_P1.27mm_Vertical, F.Cu at (279.9, 204.8)
- added REF**: LGA-16_3x3mm_P0.5mm_LayoutBorder3x5y, Package_LGA:LGA-16_3x3mm_P0.5mm_LayoutBorder3x5y, F.Cu at (341.0, 177.8)
- added REF**: JST_PH_B4B-PH-K_1x04_P2.00mm_Vertical, Connector_JST:JST_PH_B4B-PH-K_1x04_P2.00mm_Vertical, F.Cu at (334.5, 166.2)
- added REF**: C_0603_1608Metric, Capacitor_SMD:C_0603_1608Metric, F.Cu at (315.2, 168.5)
- added REF**: R_0603_1608Metric, Resistor_SMD:R_0603_1608Metric, F.Cu at (287.0, 200.2)
- added REF**: C_0603_1608Metric, Capacitor_SMD:C_0603_1608Metric, F.Cu at (289.8, 181.0)
- added REF**: PinHeader_2x03_P2.54mm_Vertical, Connector_PinHeader_2.54mm:PinHeader_2x03_P2.54mm_Vertical, F.Cu at (282.5, 214.5)
- added REF**: USB_Micro-B_Amphenol_10118193_Horizontal, GiraffeTech-Connector:USB_Micro-B_Amphenol_10118193_Horizontal, F.Cu at (343.2, 191.8)
- added REF**: R_0603_1608Metric, Resistor_SMD:R_0603_1608Metric, F.Cu at (312.5, 204.5)
- added REF**: SW_SPST_B3S-1000, Button_Switch_SMD:SW_SPST_B3S-1000, F.Cu at (323.8, 191.8)
- added REF**: C_0603_1608Metric, Capacitor_SMD:C_0603_1608Metric, F.Cu at (235.2, 94.2)
- added REF**: C_0603_1608Metric, Capacitor_SMD:C_0603_1608Metric, F.Cu at (330.2, 168.5)
- added REF**: JST_PH_B4B-PH-K_1x04_P2.00mm_Vertical, Connector_JST:JST_PH_B4B-PH-K_1x04_P2.00mm_Vertical, F.Cu at (319.5, 166.2)
- added REF**: R_0603_1608Metric, Resistor_SMD:R_0603_1608Metric, F.Cu at (317.0, 204.5)
- added REF**: MountingHole_3.5mm, MountingHole:MountingHole_3.5mm, F.Cu at (340.8, 167.8)
- added REF**: DINKLE_EK500V-2P, GiraffeTech-Connector:DINKLE_EK500V-2P, F.Cu at (314.8, 216.8)
- added REF**: TQFP-64_10x10mm_P0.5mm, Package_QFP:TQFP-64_10x10mm_P0.5mm, F.Cu at (301.8, 191.8)
- added REF**: C_0603_1608Metric, Capacitor_SMD:C_0603_1608Metric, F.Cu at (292.8, 181.0)
- added REF**: C_0603_1608Metric, Capacitor_SMD:C_0603_1608Metric, F.Cu at (307.8, 165.5)
- added REF**: Dinkle_ED350V_2Pins_Pitch3.5mm, GiraffeTech-Connector:TerminalBlock_Dinkle_ED350V_1x02_P3.50mm_Horizontal, F.Cu at (276.5, 216.2)
- added REF**: BarrelJack_Horizontal, Connector_BarrelJack:BarrelJack_Horizontal, F.Cu at (324.8, 207.8)
Other:
- board size 86 x 131.5 mm -> 175 x 198.8 mm
- board text added: "80 x 60 mm"
- board text added: "86 x 60 mm"
- board text added: "RGB"
- board text added: "WS2812"

Commit message: update
Parts:
- moved REF** 27.3 mm to (225.2, 125.0)
- moved REF** 3.50 mm to (232.2, 122.5)
- turned REF** to 270 degrees

Commit message: update
Parts:
- removed the REF** at (246.0, 108.5)
- removed the REF** at (185.8, 122.5)
- added REF**: QFN-24-1EP_4x4mm_P0.5mm_EP2.7x2.6mm, Package_DFN_QFN:QFN-24-1EP_4x4mm_P0.5mm_EP2.7x2.6mm, F.Cu at (245.1, 108.5)
- added REF**: ESP32-WROOM-32_WifiNinaPin, GiraffeTech-NodeMCU:ESP32-WROOM-32_WifiNinaPin, F.Cu at (185.8, 122.5)
- moved REF** 1.25 mm to (246.0, 103.0)

Commit message: update
Parts:
- removed the REF** at (333.2, 208.5)
- removed the REF** at (337.8, 211.5)
- removed the REF** at (340.8, 207.5)
- removed the REF** at (327.0, 166.2)
- removed the REF** at (289.5, 207.2)
- removed the REF** at (304.5, 166.2)
- removed the REF** at (322.8, 168.5)
- removed the REF** at (322.8, 165.5)
- removed the REF** at (312.0, 166.2)
- removed the REF** at (288.5, 200.2)
- removed the REF** at (342.0, 202.2)
- removed the REF** at (302.0, 206.8)
- removed the REF** at (307.8, 168.5)
- removed the REF** at (312.5, 207.2)
- removed the REF** at (280.8, 191.8)
- removed the REF** at (268.8, 167.8)
- removed the REF** at (304.0, 216.8)
- removed the REF** at (279.8, 175.2)
- removed the REF** at (279.8, 167.5)
- removed the REF** at (340.8, 210.8)
- removed the REF** at (294.5, 206.8)
- removed the REF** at (293.0, 206.8)
- removed the REF** at (315.2, 165.5)
- removed the REF** at (330.2, 165.5)
- removed the REF** at (298.2, 206.8)
- removed the REF** at (293.5, 216.8)
- removed the REF** at (288.0, 207.2)
- removed the REF** at (333.2, 218.2)
- removed the REF** at (303.5, 206.8)
- removed the REF** at (278.5, 208.5)
- removed the REF** at (268.8, 215.8)
- removed the REF** at (340.8, 215.8)
- removed the REF** at (317.0, 207.2)
- removed the REF** at (341.0, 177.8)
- removed the REF** at (334.5, 166.2)
- removed the REF** at (315.2, 168.5)
- removed the REF** at (287.0, 200.2)
- removed the REF** at (289.8, 181.0)
- removed the REF** at (312.5, 204.5)
- removed the REF** at (323.8, 191.8)
- removed the REF** at (330.2, 168.5)
- removed the REF** at (319.5, 166.2)
- removed the REF** at (317.0, 204.5)
- removed the REF** at (340.8, 167.8)
- removed the REF** at (314.8, 216.8)
- removed the REF** at (292.8, 181.0)
- removed the REF** at (307.8, 165.5)
- removed the REF** at (276.5, 216.2)
- added REF**: SW_SPDT_CK-JS102011JCQN, GiraffeTech-Electromechanical:SW_SPDT_CK-JS102011JCQN, F.Cu at (240.0, 203.2)
- added REF**: C_0603_1608Metric, Capacitor_SMD:C_0603_1608Metric, F.Cu at (208.5, 207.8)
- added REF**: C_0603_1608Metric, Capacitor_SMD:C_0603_1608Metric, F.Cu at (220.2, 164.5)
- added REF**: SOT-23-6, Package_TO_SOT_SMD:SOT-23-6, F.Cu at (222.0, 208.2)
- added REF**: C_0603_1608Metric, Capacitor_SMD:C_0603_1608Metric, F.Cu at (242.8, 212.5)
- added REF**: R_0603_1608Metric, Resistor_SMD:R_0603_1608Metric, F.Cu at (192.0, 204.2)
- added REF**: QFN-16-1EP_3x3mm_Pitch0.5mm, GiraffeTech-Maxim:QFN-16-1EP_3x3mm_Pitch0.5mm, F.Cu at (203.2, 207.8)
- added REF**: R_0603_1608Metric, Resistor_SMD:R_0603_1608Metric, F.Cu at (217.5, 205.5)
- added REF**: DINKLE_EK500V-2P, GiraffeTech-Connector:DINKLE_EK500V-2P, F.Cu at (209.0, 217.8)
- added REF**: R_0603_1608Metric, Resistor_SMD:R_0603_1608Metric, F.Cu at (222.0, 205.5)
- added REF**: SOT-23-6, Package_TO_SOT_SMD:SOT-23-6, F.Cu at (217.5, 208.2)
- added REF**: MountingHole_3.5mm, MountingHole:MountingHole_3.5mm, F.Cu at (173.8, 166.8)
- added REF**: C_0603_1608Metric, Capacitor_SMD:C_0603_1608Metric, F.Cu at (199.5, 207.8)
- added REF**: JST_PH_B4B-PH-K_1x04_P2.00mm_Vertical, Connector_JST:JST_PH_B4B-PH-K_1x04_P2.00mm_Vertical, F.Cu at (217.0, 165.2)
- added REF**: LED_0603_1608Metric, LED_SMD:LED_0603_1608Metric, F.Cu at (247.0, 203.2)
- added REF**: C_0603_1608Metric, Capacitor_SMD:C_0603_1608Metric, F.Cu at (235.2, 167.5)
- added REF**: C_0603_1608Metric, Capacitor_SMD:C_0603_1608Metric, F.Cu at (235.2, 164.5)
- added REF**: C_0603_1608Metric, Capacitor_SMD:C_0603_1608Metric, F.Cu at (220.2, 167.5)
- added REF**: MountingHole_3.5mm, MountingHole:MountingHole_3.5mm, F.Cu at (245.8, 166.8)
- added REF**: C_0603_1608Metric, Capacitor_SMD:C_0603_1608Metric, F.Cu at (194.5, 208.2)
- added REF**: JST_PH_B4B-PH-K_1x04_P2.00mm_Vertical, Connector_JST:JST_PH_B4B-PH-K_1x04_P2.00mm_Vertical, F.Cu at (209.5, 165.2)
- added REF**: MountingHole_3.5mm, MountingHole:MountingHole_3.5mm, F.Cu at (245.8, 218.8)
- added REF**: C_0603_1608Metric, Capacitor_SMD:C_0603_1608Metric, F.Cu at (193.0, 208.2)
- added REF**: SW_SPST_B3S-1000, Button_Switch_SMD:SW_SPST_B3S-1000, F.Cu at (184.8, 174.2)
- added REF**: LED_0603_1608Metric, LED_SMD:LED_0603_1608Metric, F.Cu at (238.2, 209.5)
- added REF**: C_0603_1608Metric, Capacitor_SMD:C_0603_1608Metric, F.Cu at (198.0, 207.8)
- added REF**: C_0603_1608Metric, Capacitor_SMD:C_0603_1608Metric, F.Cu at (212.8, 164.5)
- added REF**: C_0603_1608Metric, Capacitor_SMD:C_0603_1608Metric, F.Cu at (212.8, 167.5)
- added REF**: Dinkle_ED350V_2Pins_Pitch3.5mm, GiraffeTech-Connector:TerminalBlock_Dinkle_ED350V_1x02_P3.50mm_Horizontal, F.Cu at (181.5, 219.2)
- added REF**: C_0603_1608Metric, Capacitor_SMD:C_0603_1608Metric, F.Cu at (227.8, 164.5)
- added REF**: JST_PH_B4B-PH-K_1x04_P2.00mm_Vertical, Connector_JST:JST_PH_B4B-PH-K_1x04_P2.00mm_Vertical, F.Cu at (239.5, 165.2)
- added REF**: C_0603_1608Metric, Capacitor_SMD:C_0603_1608Metric, F.Cu at (245.8, 208.5)
- added REF**: SW_SPST_B3S-1000, Button_Switch_SMD:SW_SPST_B3S-1000, F.Cu at (232.2, 192.8)
- added REF**: DINKLE_EK500V-2P, GiraffeTech-Connector:DINKLE_EK500V-2P, F.Cu at (198.5, 217.8)
- added REF**: C_0603_1608Metric, Capacitor_SMD:C_0603_1608Metric, F.Cu at (194.8, 180.5)
- added REF**: DINKLE_EK500V-2P, GiraffeTech-Connector:DINKLE_EK500V-2P, F.Cu at (219.8, 217.8)
- added REF**: R_0603_1608Metric, Resistor_SMD:R_0603_1608Metric, F.Cu at (193.5, 204.2)
- added REF**: C_0603_1608Metric, Capacitor_SMD:C_0603_1608Metric, F.Cu at (207.0, 207.8)
- added REF**: C_0603_1608Metric, Capacitor_SMD:C_0603_1608Metric, F.Cu at (197.8, 180.5)
- added REF**: JST_PH_B4B-PH-K_1x04_P2.00mm_Vertical, Connector_JST:JST_PH_B4B-PH-K_1x04_P2.00mm_Vertical, F.Cu at (224.5, 165.2)
- added REF**: QFN-24-1EP_4x4mm_P0.5mm_EP2.7x2.6mm, Package_DFN_QFN:QFN-24-1EP_4x4mm_P0.5mm_EP2.7x2.6mm, F.Cu at (245.1, 178.8)
- added REF**: ESP32-WROOM-32_WifiNinaPin, GiraffeTech-NodeMCU:ESP32-WROOM-32_WifiNinaPin, F.Cu at (185.8, 192.8)
- added REF**: MountingHole_3.5mm, MountingHole:MountingHole_3.5mm, F.Cu at (173.8, 218.8)
- added REF**: Dinkle_ED350V_2Pins_Pitch3.5mm, GiraffeTech-Connector:TerminalBlock_Dinkle_ED350V_1x02_P3.50mm_Horizontal, F.Cu at (238.2, 219.2)
- added REF**: C_0603_1608Metric, Capacitor_SMD:C_0603_1608Metric, F.Cu at (227.8, 167.5)
- added REF**: SW_SPST_B3S-1000, Button_Switch_SMD:SW_SPST_B3S-1000, F.Cu at (184.8, 166.5)
- added REF**: JST_PH_B4B-PH-K_1x04_P2.00mm_Vertical, Connector_JST:JST_PH_B4B-PH-K_1x04_P2.00mm_Vertical, F.Cu at (232.0, 165.2)
- added REF**: QFN-16-1EP_3x3mm_Pitch0.5mm, GiraffeTech-Maxim:QFN-16-1EP_3x3mm_Pitch0.5mm, F.Cu at (182.8, 210.2)
- added REF**: C_0603_1608Metric, Capacitor_SMD:C_0603_1608Metric, F.Cu at (245.8, 211.8)
- moved G*** 115.0 mm to (198.2, 192.8)
- moved MS2 96.5 mm to (248.2, 181.3)
- moved REF** 95.3 mm to (174.8, 208.2)
- moved REF** 95.3 mm to (187.2, 216.0)
- moved REF** 95.0 mm to (171.5, 174.0)
- moved REF** 95.0 mm to (204.0, 167.8)
- moved REF** 95.0 mm to (248.2, 209.2)
- moved REF** 95.0 mm to (248.2, 192.8)
- moved REF** 95.0 mm to (242.8, 209.5)
- moved REF** 95.0 mm to (229.8, 208.8)
- moved REF** 95.0 mm to (246.0, 173.2)
- moved REF** 91.8 mm to (210.0, 192.8), turned to 270 degrees
- moved REF** 55.5 mm to (225.2, 195.2), turned to 180 degrees
Other:
- board size 175 x 198.8 mm -> 175 x 201.8 mm
