File: MP_SamBaseBoard_V1_DraftDesign/MP_SamBaseBoard_V1.kicad_pcb (KiCad board)
At the start: 2 copper layers, 175 x 201.8 mm, 256 parts

Commit message: update
Parts:
- removed the REF** at (222.0, 208.2)
- removed the REF** at (222.0, 205.5)
- removed the REF** at (242.8, 209.5)
Changed lines of the file:
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@@
     (tracks 0)
     (zones 0)
-    (modules 256)
+    (modules 253)
     (nets 1)
   )
@@
     )
   )
-  (module Package_TO_SOT_SMD:SOT-23-6 (layer F.Cu)
-    (at 222 208.25 180)
-    (descr "6-pin SOT-23 package")
-    (tags SOT-23-6)
-    (attr smd)
-    (fp_text reference REF** (at 0 -2.9) (layer F.SilkS) hide
-      (effects (font (size 1 1) (thickness 0.15)))
-    )
-    (fp_text value SOT-23-6 (at 0 2.9) (layer F.Fab)
-      (effects (font (size 1 1) (thickness 0.15)))
-    )
-    (fp_text user %R (at 0 0 90) (layer F.Fab)
-      (effects (font (size 0.5 0.5) (thickness 0.075)))
-    )
-    (fp_line (start -0.9 1.61) (end 0.9 1.61) (layer F.SilkS) (width 0.12))
-    (fp_line (start 0.9 -1.61) (end -1.55 -1.61) (layer F.SilkS) (width 0.12))
-    (fp_line (start 1.9 -1.8) (end -1.9 -1.8) (layer F.CrtYd) (width 0.05))
-    (fp_line (start 1.9 1.8) (end 1.9 -1.8) (layer F.CrtYd) (width 0.05))
-    (fp_line (start -1.9 1.8) (end 1.9 1.8) (layer F.CrtYd) (width 0.05))
-    (fp_line (start -1.9 -1.8) (end -1.9 1.8) (layer F.CrtYd) (width 0.05))
-    (fp_line (start -0.9 -0.9) (end -0.25 -1.55) (layer F.Fab) (width 0.1))
-    (fp_line (start 0.9 -1.55) (end -0.25 -1.55) (layer F.Fab) (width 0.1))
-    (fp_line (start -0.9 -0.9) (end -0.9 1.55) (layer F.Fab) (width 0.1))
-    (fp_line (start 0.9 1.55) (end -0.9 1.55) (layer F.Fab) (width 0.1))
-    (fp_line (start 0.9 -1.55) (end 0.9 1.55) (layer F.Fab) (width 0.1))
-    (pad 1 smd rect (at -1.1 -0.95 180) (size 1.06 0.65) (layers F.Cu F.Paste F.Mask))
-    (pad 2 smd rect (at -1.1 0 180) (size 1.06 0.65) (layers F.Cu F.Paste F.Mask))
-    (pad 3 smd rect (at -1.1 0.95 180) (size 1.06 0.65) (layers F.Cu F.Paste F.Mask))
-    (pad 4 smd rect (at 1.1 0.95 180) (size 1.06 0.65) (layers F.Cu F.Paste F.Mask))
-    (pad 6 smd rect (at 1.1 -0.95 180) (size 1.06 0.65) (layers F.Cu F.Paste F.Mask))
-    (pad 5 smd rect (at 1.1 0 180) (size 1.06 0.65) (layers F.Cu F.Paste F.Mask))
-    (model ${KISYS3DMOD}/Package_TO_SOT_SMD.3dshapes/SOT-23-6.wrl
-      (at (xyz 0 0 0))
-      (scale (xyz 1 1 1))
-      (rotate (xyz 0 0 0))
-    )
-  )
   (module Capacitor_SMD:C_0603_1608Metric (layer F.Cu)
     (at 242.75 212.5)
@@
     (fp_circle (center 0 0.075) (end 0 0.25) (layer F.SilkS) (width 0.5))
     (fp_arc (start 0 0.075) (end 0.75 0.75) (angle 270) (layer F.SilkS) (width 0.15))
-  )
-  (module Resistor_SMD:R_0603_1608Metric (layer F.Cu)
-    (at 222 205.5 180)
-    (descr "Resistor SMD 0603 (1608 Metric), square (rectangular) end terminal, IPC_7351 nominal, (Body size source: http://www.tortai-tech.com/upload/download/2011102023233369053.pdf), generated with kicad-footprint-generator")
-    (tags resistor)
-    (attr smd)
-    (fp_text reference REF** (at 0 -1.43) (layer F.SilkS) hide
-      (effects (font (size 1 1) (thickness 0.15)))
-    )
-    (fp_text value R_0603_1608Metric (at 0 1.43) (layer F.Fab)
-      (effects (font (size 1 1) (thickness 0.15)))
-    )
-    (fp_line (start -0.8 0.4) (end -0.8 -0.4) (layer F.Fab) (width 0.1))
-    (fp_line (start -0.8 -0.4) (end 0.8 -0.4) (layer F.Fab) (width 0.1))
-    (fp_line (start 0.8 -0.4) (end 0.8 0.4) (layer F.Fab) (width 0.1))
-    (fp_line (start 0.8 0.4) (end -0.8 0.4) (layer F.Fab) (width 0.1))
-    (fp_line (start -0.162779 -0.51) (end 0.162779 -0.51) (layer F.SilkS) (width 0.12))
-    (fp_line (start -0.162779 0.51) (end 0.162779 0.51) (layer F.SilkS) (width 0.12))
-    (fp_line (start -1.48 0.73) (end -1.48 -0.73) (layer F.CrtYd) (width 0.05))
-    (fp_line (start -1.48 -0.73) (end 1.48 -0.73) (layer F.CrtYd) (width 0.05))
-    (fp_line (start 1.48 -0.73) (end 1.48 0.73) (layer F.CrtYd) (width 0.05))
-    (fp_line (start 1.48 0.73) (end -1.48 0.73) (layer F.CrtYd) (width 0.05))
-    (fp_text user %R (at 0 0) (layer F.Fab)
-      (effects (font (size 0.4 0.4) (thickness 0.06)))
-    )
-    (pad 1 smd roundrect (at -0.7875 0 180) (size 0.875 0.95) (layers F.Cu F.Paste F.Mask) (roundrect_rratio 0.25))
-    (pad 2 smd roundrect (at 0.7875 0 180) (size 0.875 0.95) (layers F.Cu F.Paste F.Mask) (roundrect_rratio 0.25))
-    (model ${KISYS3DMOD}/Resistor_SMD.3dshapes/R_0603_1608Metric.wrl
-      (at (xyz 0 0 0))
-      (scale (xyz 1 1 1))
-      (rotate (xyz 0 0 0))
-    )
   )
   (module Package_TO_SOT_SMD:SOT-23-6 (layer F.Cu)
@@
       (at (xyz 0 0 0))
       (scale (xyz 1 1 1))
-      (rotate (xyz 0 0 0))
-    )
-  )
-  (module Package_TO_SOT_SMD:SOT-23-5 (layer F.Cu)
-    (at 242.75 209.5 270)
-    (descr "5-pin SOT23 package")
-    (tags SOT-23-5)
-    (attr smd)
-    (fp_text reference REF** (at 0 -2.9 90) (layer F.SilkS) hide
-      (effects (font (size 1 1) (thickness 0.15)))
-    )
-    (fp_text value SOT-23-5 (at 0 2.9 90) (layer F.Fab)
-      (effects (font (size 1 1) (thickness 0.15)))
-    )
-    (fp_text user %R (at 0 0) (layer F.Fab)
-      (effects (font (size 0.5 0.5) (thickness 0.075)))
-    )
-    (fp_line (start -0.9 1.61) (end 0.9 1.61) (layer F.SilkS) (width 0.12))
-    (fp_line (start 0.9 -1.61) (end -1.55 -1.61) (layer F.SilkS) (width 0.12))
-    (fp_line (start -1.9 -1.8) (end 1.9 -1.8) (layer F.CrtYd) (width 0.05))
-    (fp_line (start 1.9 -1.8) (end 1.9 1.8) (layer F.CrtYd) (width 0.05))
-    (fp_line (start 1.9 1.8) (end -1.9 1.8) (layer F.CrtYd) (width 0.05))
-    (fp_line (start -1.9 1.8) (end -1.9 -1.8) (layer F.CrtYd) (width 0.05))
-    (fp_line (start -0.9 -0.9) (end -0.25 -1.55) (layer F.Fab) (width 0.1))
-    (fp_line (start 0.9 -1.55) (end -0.25 -1.55) (layer F.Fab) (width 0.1))
-    (fp_line (start -0.9 -0.9) (end -0.9 1.55) (layer F.Fab) (width 0.1))
-    (fp_line (start 0.9 1.55) (end -0.9 1.55) (layer F.Fab) (width 0.1))
-    (fp_line (start 0.9 -1.55) (end 0.9 1.55) (layer F.Fab) (width 0.1))
-    (pad 1 smd rect (at -1.1 -0.95 270) (size 1.06 0.65) (layers F.Cu F.Paste F.Mask))
-    (pad 2 smd rect (at -1.1 0 270) (size 1.06 0.65) (layers F.Cu F.Paste F.Mask))
-    (pad 3 smd rect (at -1.1 0.95 270) (size 1.06 0.65) (layers F.Cu F.Paste F.Mask))
-    (pad 4 smd rect (at 1.1 0.95 270) (size 1.06 0.65) (layers F.Cu F.Paste F.Mask))
-    (pad 5 smd rect (at 1.1 -0.95 270) (size 1.06 0.65) (layers F.Cu F.Paste F.Mask))
-    (model ${KISYS3DMOD}/Package_TO_SOT_SMD.3dshapes/SOT-23-5.wrl
-      (at (xyz 0 0 0))
-      (scale (xyz 1 1 1))

Commit message: Schematic done, update pcb
Parts:
- removed the G*** at (288.4, 51.0)
- removed the MS2 at (248.2, 181.3)
- removed the MS2 at (335.6, 39.6)
- removed the REF** at (171.5, 174.0)
- removed the REF** at (204.0, 167.8)
- removed the REF** at (331.5, 60.2)
- removed the REF** at (341.0, 40.8)
- removed the REF** at (322.6, 54.8)
- removed the REF** at (354.0, 61.0)
- removed the REF** at (309.8, 26.0)
- removed the REF** at (267.8, 29.8)
- removed the REF** at (306.0, 76.0)
- removed the REF** at (269.2, 64.2)
- removed the REF** at (269.2, 62.8)
- removed the REF** at (278.9, 64.1)
- removed the REF** at (270.2, 72.5)
- removed the REF** at (324.8, 67.0)
- removed the REF** at (295.2, 72.5)
- removed the REF** at (262.2, 68.8)
- removed the REF** at (333.2, 67.8)
- removed the REF** at (341.8, 32.5)
- removed the REF** at (325.5, 35.5)
- removed the REF** at (315.2, 36.0)
- removed the REF** at (333.2, 77.5)
- removed the REF** at (337.8, 70.8)
- removed the REF** at (340.8, 70.0)
- removed the REF** at (328.8, 38.2)
- removed the REF** at (262.8, 77.0)
- removed the REF** at (276.5, 72.5)
- removed the REF** at (272.5, 26.2)
- removed the REF** at (328.8, 35.5)
- removed the REF** at (340.8, 77.0)
- removed the REF** at (301.2, 28.0)
- removed the REF** at (331.2, 26.0)
- removed the REF** at (292.2, 33.2)
- removed the REF** at (282.2, 26.2)
- removed the REF** at (272.5, 35.5)
- removed the REF** at (277.5, 29.8)
- removed the REF** at (340.8, 25.0)
- removed the REF** at (320.5, 26.0)
- removed the REF** at (301.8, 51.0)
- removed the REF** at (262.2, 64.0)
- removed the REF** at (262.8, 25.0)
- removed the REF** at (282.2, 35.5)
- removed the REF** at (333.2, 38.2)
- removed the REF** at (301.5, 72.5)
- removed the REF** at (217.0, 165.2)
- removed the REF** at (343.2, 67.5)
- removed the REF** at (260.8, 33.0)
- removed the REF** at (274.8, 51.0)
- removed the REF** at (287.5, 32.2)
- removed the REF** at (337.8, 67.8)
- removed the REF** at (343.2, 51.0)
- removed the REF** at (324.0, 35.5)
- removed the REF** at (311.5, 36.0)
- removed the REF** at (310.0, 36.0)
- removed the REF** at (289.0, 72.5)
- removed the REF** at (333.2, 35.5)
- removed the REF** at (282.8, 72.5)
- removed the REF** at (291.0, 24.5)
- removed the REF** at (340.8, 66.8)
- removed the REF** at (319.0, 36.0)
- removed the REF** at (320.5, 36.0)
- removed the REF** at (246.0, 173.2)
- removed the REF** at (225.2, 195.2)
- removed the REF** at (209.5, 165.2)
- removed the REF** at (184.8, 174.2)
- removed the REF** at (174.8, 208.2)
- removed the REF** at (239.5, 165.2)
- removed the REF** at (232.2, 192.8)
- removed the REF** at (224.5, 165.2)
- removed the REF** at (245.1, 178.8)
- removed the REF** at (210.0, 192.8)
- removed the REF** at (185.8, 192.8)
- removed the REF** at (184.8, 166.5)
- removed the REF** at (232.0, 165.2)
- added BZ1: Buzzer, Buzzer_Beeper:MagneticBuzzer_Kobitone_254-EMB84Q-RO, F.Cu at (174.8, 208.2)
- added C1: 0.1uF, Capacitor_SMD:C_0603_1608Metric, F.Cu at (104.0, 209.8)
- added C10: 4.7uF, Capacitor_SMD:C_0603_1608Metric, F.Cu at (129.5, 183.7)
- added C11: 10uF, Capacitor_Tantalum_SMD:CP_EIA-3216-12_Kemet-S, F.Cu at (55.0, 221.6)
- added C12: 0.1uF, Capacitor_SMD:C_0603_1608Metric, F.Cu at (106.9, 203.7)
- added C13: 0.1uF, Capacitor_SMD:C_0603_1608Metric, F.Cu at (85.0, 223.4)
- added C14: 10uF, Capacitor_Tantalum_SMD:CP_EIA-3216-12_Kemet-S, F.Cu at (49.3, 221.6)
- added C15: 1uF, Capacitor_SMD:C_0603_1608Metric, F.Cu at (138.5, 174.1)
- added C16: 1uF, Capacitor_SMD:C_0603_1608Metric, F.Cu at (137.8, 179.1)
- added C17: 10uF, Capacitor_Tantalum_SMD:CP_EIA-3216-12_Kemet-S, F.Cu at (37.9, 221.6)
- added C18: 10uF, Capacitor_Tantalum_SMD:CP_EIA-3216-12_Kemet-S, F.Cu at (43.6, 221.6)
- added C19: 0.1uF, Capacitor_SMD:C_0603_1608Metric, F.Cu at (116.1, 205.7)
- added C2: 1uF, Capacitor_SMD:C_0603_1608Metric, F.Cu at (111.3, 200.6)
- added C20: 0.1uF 16V, Capacitor_SMD:C_0603_1608Metric, F.Cu at (119.3, 203.1)
- added C21: 0.1uF, Capacitor_SMD:C_0603_1608Metric, F.Cu at (138.3, 184.1)
- added C22: 0.1uF, Capacitor_SMD:C_0603_1608Metric, F.Cu at (112.1, 210.7)
- added C23: 10uF 16V, Capacitor_Tantalum_SMD:CP_EIA-3216-12_Kemet-S, F.Cu at (106.1, 178.0)
- added C24: 0.1uF 16V, Capacitor_SMD:C_0603_1608Metric, F.Cu at (141.8, 181.6)
- added C25: 0.1uF 16V, Capacitor_SMD:C_0603_1608Metric, F.Cu at (125.2, 197.9)
- added C26: 10uF, Capacitor_Tantalum_SMD:CP_EIA-3216-12_Kemet-S, F.Cu at (60.7, 221.6)
- added C27: 2.2uF 6.3V, Capacitor_SMD:C_0603_1608Metric, F.Cu at (104.9, 217.5)
- added C28: 0.1uF, Capacitor_SMD:C_0603_1608Metric, F.Cu at (116.1, 208.2)
- added C29: 0.1uF, Capacitor_SMD:C_0603_1608Metric, F.Cu at (134.2, 189.4)
- added C3: 0.1uF, Capacitor_SMD:C_0603_1608Metric, F.Cu at (121.0, 192.9)
- added C30: 2.2nF, Capacitor_SMD:C_0603_1608Metric, F.Cu at (126.2, 186.5)
- added C31: 1uF, Capacitor_SMD:C_0603_1608Metric, F.Cu at (115.3, 200.6)
- added C32: 4.7uF, Capacitor_SMD:C_0603_1608Metric, F.Cu at (104.0, 212.4)
- added C33: 4.7uF, Capacitor_SMD:C_0603_1608Metric, F.Cu at (108.1, 208.8)
- added C34: 0.1uF, Capacitor_SMD:C_0603_1608Metric, F.Cu at (96.9, 220.5)
- added C35: 0.1uF, Capacitor_SMD:C_0603_1608Metric, F.Cu at (108.1, 206.3)
- added C36: 0.1uF, Capacitor_SMD:C_0603_1608Metric, F.Cu at (117.2, 198.1)
- added C37: 0.1uF, Capacitor_SMD:C_0603_1608Metric, F.Cu at (125.0, 190.4)
- added C38: 1uF, Capacitor_SMD:C_0603_1608Metric, F.Cu at (133.8, 181.9)
- added C39: 1uF, Capacitor_SMD:C_0603_1608Metric, F.Cu at (138.5, 176.6)
- added C4: 1uF, Capacitor_SMD:C_0603_1608Metric, F.Cu at (89.1, 223.4)
- added C40: 1uF, Capacitor_SMD:C_0603_1608Metric, F.Cu at (111.3, 203.1)
- added C41: 1uF, Capacitor_SMD:C_0603_1608Metric, F.Cu at (99.0, 215.7)
- added C5: 0.1uF, Capacitor_SMD:C_0603_1608Metric, F.Cu at (113.2, 198.1)
- added C6: 1uF, Capacitor_SMD:C_0603_1608Metric, F.Cu at (117.2, 195.5)
- added C7: 22nF, Capacitor_SMD:C_0603_1608Metric, F.Cu at (100.0, 212.4)
- added C8: 22nF, Capacitor_SMD:C_0603_1608Metric, F.Cu at (121.0, 190.4)
- added C9: 4.7uF, Capacitor_SMD:C_0603_1608Metric, F.Cu at (133.8, 179.4)
- added D1: LED, LED_SMD:LED_0603_1608Metric, F.Cu at (113.2, 195.6)
- added D2: LED, LED_SMD:LED_0603_1608Metric, F.Cu at (100.0, 207.3)
- added D3: LED, LED_SMD:LED_0603_1608Metric, F.Cu at (100.0, 209.9)
- added D4: LED, LED_SMD:LED_0603_1608Metric, F.Cu at (92.9, 220.5)
- added D5: LED, LED_SMD:LED_0603_1608Metric, F.Cu at (104.1, 207.3)
- added D6: WS2812B, GiraffeTech-LED:WS2812B_MINI, F.Cu at (89.4, 215.0)
- added D7: WS2812B, GiraffeTech-LED:WS2812B_MINI, F.Cu at (140.7, 165.8)
- added J1: MOTOR-A_CONN, GiraffeTech-Connector:DINKLE_EK500V-2P, F.Cu at (99.2, 200.6)
- added J10: P1_CONN, Connector_JST:JST_PH_B4B-PH-K_1x04_P2.00mm_Vertical, F.Cu at (224.5, 165.2)
- added J11: I2C_CONN, Connector_JST:JST_PH_B4B-PH-K_1x04_P2.00mm_Vertical, F.Cu at (232.0, 165.2)
- added J12: I2C_CONN, Connector_JST:JST_PH_B4B-PH-K_1x04_P2.00mm_Vertical, F.Cu at (239.5, 165.2)
- added J13: SAM_SWD, Connector_PinHeader_1.27mm:PinHeader_2x05_P1.27mm_Vertical, F.Cu at (224.0, 190.2)
- added J14: WS2812_EXT, Connector_PinHeader_2.54mm:PinHeader_1x03_P2.54mm_Vertical, F.Cu at (171.8, 174.0)
- added J15: PWR_JACK, Connector_BarrelJack:BarrelJack_Horizontal, F.Cu at (79.1, 192.9)
- added J2: MOTOR-B_CONN, GiraffeTech-Connector:DINKLE_EK500V-2P, F.Cu at (82.2, 207.2)
- added J3: Adafruit_Feather_CONN, GiraffeTech-Connector:Adafruit-Feather_WoMountPoint, F.Cu at (248.2, 181.2)
- added J4: uSD_Card, GiraffeTech-Connector:GTK_TFMS08TK-PP-02, F.Cu at (204.0, 167.8)
- added J5: Conn_01x02, GiraffeTech-Connector:DINKLE_EK500V-2P, F.Cu at (70.2, 212.1)
- added J6: Conn_01x02, GiraffeTech-Connector:DINKLE_EK500V-2P, F.Cu at (107.1, 186.3)
- added J7: SERVO_CONN, Connector_PinHeader_2.54mm:PinHeader_2x03_P2.54mm_Vertical, F.Cu at (115.1, 180.7)
- added J8: P3_CONN, Connector_JST:JST_PH_B4B-PH-K_1x04_P2.00mm_Vertical, F.Cu at (209.5, 165.2)
- added J9: P2_CONN, Connector_JST:JST_PH_B4B-PH-K_1x04_P2.00mm_Vertical, F.Cu at (217.0, 165.2)
- added L1: 10uH, Inductor_SMD:L_0805_2012Metric, F.Cu at (76.7, 222.5)
- added L2: 0.47uH, GiraffeTech-Inductor:L_0806_2016Metric, F.Cu at (81.0, 222.6)
- added L3: 1uH, GiraffeTech-Inductor:L_1616_2020Metric, F.Cu at (123.7, 181.8)
- added MK1: Knowles_SPW2430HR5H-B, GiraffeTech-Knowles:SPW2430HR5H-B, F.Cu at (134.5, 174.0)
- added Q1: DMP3098L, Package_TO_SOT_SMD:SOT-23, F.Cu at (107.1, 200.2)
- added R1: 10K, Resistor_SMD:R_0603_1608Metric, F.Cu at (130.2, 186.2)
- added R10: 10K, Resistor_SMD:R_0603_1608Metric, F.Cu at (93.1, 223.1)
- added R11: 10K, Resistor_SMD:R_0603_1608Metric, F.Cu at (100.9, 218.2)
- added R12: 10K, Resistor_SMD:R_0603_1608Metric, F.Cu at (112.1, 208.2)
- added R13: 10K, Resistor_SMD:R_0603_1608Metric, F.Cu at (125.2, 195.4)
- added R14: 10K, Resistor_SMD:R_0603_1608Metric, F.Cu at (134.2, 184.4)
- added R15: 10K, Resistor_SMD:R_0603_1608Metric, F.Cu at (141.8, 179.1)
- added R16: 1K, Resistor_SMD:R_0603_1608Metric, F.Cu at (97.1, 223.0)
- added R17: 10K, Resistor_SMD:R_0603_1608Metric, F.Cu at (119.3, 200.6)
- added R18: 1K, Resistor_SMD:R_0603_1608Metric, F.Cu at (129.0, 191.2)
- added R19: 2K, Resistor_SMD:R_0603_1608Metric, F.Cu at (134.2, 186.9)
- added R2: 1M, Resistor_SMD:R_0603_1608Metric, F.Cu at (121.2, 195.4)
- added R20: 1K, Resistor_SMD:R_0603_1608Metric, F.Cu at (115.3, 203.1)
- added R21: 10K, Resistor_SMD:R_0603_1608Metric, F.Cu at (108.0, 213.8)
- added R22: 10K, Resistor_SMD:R_0603_1608Metric, F.Cu at (129.2, 193.7)
- added R23: 10K, Resistor_SMD:R_0603_1608Metric, F.Cu at (101.1, 223.2)
- added R24: RG, Resistor_SMD:R_0603_1608Metric, F.Cu at (138.3, 186.6)
- added R25: 10K, Resistor_SMD:R_0603_1608Metric, F.Cu at (112.0, 213.2)
- added R26: 10K, Resistor_SMD:R_0603_1608Metric, F.Cu at (129.2, 196.3)
- added R27: 10K, Resistor_SMD:R_0603_1608Metric, F.Cu at (120.1, 205.7)
- added R28: 10K, Resistor_SMD:R_0603_1608Metric, F.Cu at (123.3, 202.9)
- added R29: 820K, Resistor_SMD:R_0603_1608Metric, F.Cu at (105.1, 220.0)
- added R3: 10K, Resistor_SMD:R_0603_1608Metric, F.Cu at (125.0, 192.9)
- added R30: 1K, Resistor_SMD:R_0603_1608Metric, F.Cu at (101.1, 220.7)
- added R31: 1K, Resistor_SMD:R_0603_1608Metric, F.Cu at (108.0, 211.3)
- added R32: RB, Resistor_SMD:R_0603_1608Metric, F.Cu at (181.0, 204.8)
- added R4: 10K, Resistor_SMD:R_0603_1608Metric, F.Cu at (103.0, 214.9)
- added R5: 10K, Resistor_SMD:R_0603_1608Metric, F.Cu at (123.3, 200.4)
- added R6: 619K, Resistor_SMD:R_0603_1608Metric, F.Cu at (112.1, 205.7)
- added R7: 100K, Resistor_SMD:R_0603_1608Metric, F.Cu at (130.2, 188.7)
- added R8: 100K, Resistor_SMD:R_0603_1608Metric, F.Cu at (137.8, 181.6)
- added R9: 10K, Resistor_SMD:R_0603_1608Metric, F.Cu at (121.2, 197.9)
- added SW1: RESET, Button_Switch_SMD:SW_SPST_B3S-1000, F.Cu at (232.2, 192.8)
- added SW2: 3v3_PWR_SW, GiraffeTech-Electromechanical:SW_SPDT_CK-JS102011JCQN, F.Cu at (69.6, 220.1)
- added SW3: SW1, Button_Switch_SMD:SW_SPST_B3S-1000, F.Cu at (184.8, 174.2)
- added SW4: SW2, Button_Switch_SMD:SW_SPST_B3S-1000, F.Cu at (184.8, 166.5)
- added U1: ESP32-WROOM-32, GiraffeTech-NodeMCU:ESP32-WROOM-32_WifiNinaPin, F.Cu at (185.8, 192.8)
- added U10: MPU-6050, Sensor_Motion:InvenSense_QFN-24_4x4mm_P0.5mm, F.Cu at (129.4, 175.0)
- added U11: IRFHM9331PbF, GiraffeTech-IR:PQFN_3x3mm, F.Cu at (129.7, 180.3)
- added U12: BD5291FVE-GTR, Package_TO_SOT_SMD:SOT-353_SC-70-5, F.Cu at (122.1, 187.2)
- added U2: ATSAMD51J19A-A, Package_QFP:TQFP-64_10x10mm_P0.5mm, F.Cu at (210.2, 192.8)
- added U3: 74LVC1G125, Package_TO_SOT_SMD:SOT-23-5, F.Cu at (140.6, 170.5)
- added U4: TPS62135, GiraffeTech-Texas:VQFN-HR-11, F.Cu at (88.9, 219.8)
- added U5: TPS62086, GiraffeTech-Texas:Texas_VSON7, F.Cu at (110.8, 178.3)
- added U6: MAX98357AETE, Package_DFN_QFN:TQFN-16-1EP_3x3mm_P0.5mm_EP1.23x1.23mm, F.Cu at (84.3, 190.1)
- added U7: DRV8833RTY, Package_DFN_QFN:Texas_S-PWQFN-N16_EP2.1x2.1mm_ThermalVias, F.Cu at (108.0, 194.8)
- added U8: HDC1080, Package_SON:Texas_PWSON-N6, F.Cu at (94.5, 216.8)
- added U9: MCP73871-1CC, Package_DFN_QFN:QFN-20-1EP_4x4mm_P0.5mm_EP2.5x2.5mm, F.Cu at (115.9, 191.2)
- added Y1: Crystal, Crystal:Crystal_SMD_2012-2Pin_2.0x1.2mm, F.Cu at (142.3, 174.3)
Other:
- board size 175 x 201.8 mm -> 175 x 130.2 mm
- board text added: "80 x 60 mm [Candidate]"
- board text removed: "D1 UART"
- board text removed: "D2 A1"
- board text removed: "D3 A2"
- board text removed: "D4 A3"

Commit message: update
Parts:
- removed the REF** at (209.0, 217.8)
- removed the REF** at (220.2, 164.5)
- removed the REF** at (242.8, 212.5)
- removed the REF** at (192.0, 204.2)
- removed the REF** at (203.2, 207.8)
- removed the REF** at (217.5, 205.5)
- removed the REF** at (217.5, 208.2)
- removed the REF** at (248.2, 192.8)
- removed the REF** at (199.5, 207.8)
- removed the REF** at (235.2, 164.5)
- removed the REF** at (247.0, 203.2)
- removed the REF** at (235.2, 167.5)
- removed the REF** at (220.2, 167.5)
- removed the REF** at (194.5, 208.2)
- removed the REF** at (193.0, 208.2)
- removed the REF** at (238.2, 209.5)
- removed the REF** at (212.8, 164.5)
- removed the REF** at (212.8, 167.5)
- removed the REF** at (198.0, 207.8)
- removed the REF** at (181.5, 219.2)
- removed the REF** at (227.8, 164.5)
- removed the REF** at (245.8, 208.5)
- removed the REF** at (187.2, 216.0)
- removed the REF** at (198.5, 217.8)
- removed the REF** at (194.8, 180.5)
- removed the REF** at (219.8, 217.8)
- removed the REF** at (193.5, 204.2)
- removed the REF** at (207.0, 207.8)
- removed the REF** at (197.8, 180.5)
- removed the REF** at (229.8, 208.8)
- removed the REF** at (238.2, 219.2)
- removed the REF** at (227.8, 167.5)
- removed the REF** at (182.8, 210.2)
- removed the REF** at (245.8, 211.8)
- removed the REF** at (240.0, 203.2)
- removed the REF** at (208.5, 207.8)
- added D8: PWR_LED, LED_SMD:LED_0603_1608Metric, F.Cu at (247.0, 203.2)
- added J16: USB_B_Micro, GiraffeTech-Connector:USB_Micro-B_Amphenol_10118193_Horizontal, F.Cu at (248.2, 192.8)
- added J17: BATT_CONN, GiraffeTech-Connector:TerminalBlock_Dinkle_ED350V_1x02_P3.50mm_Horizontal, F.Cu at (238.2, 219.2)
- added R33: R_USB, Resistor_SMD:R_0603_1608Metric, F.Cu at (241.8, 191.5)
- added R34: R_USB, Resistor_SMD:R_0603_1608Metric, F.Cu at (241.8, 194.0)
- added R35: 330, Resistor_SMD:R_0603_1608Metric, F.Cu at (246.0, 237.0)
- J5: footprint GiraffeTech-Connector:DINKLE_EK500V-2P -> GiraffeTech-Connector:TerminalBlock_Dinkle_ED350V_1x02_P3.50mm_Horizontal
- moved C17 251.5 mm to (288.2, 245.8)
- moved C14 239.1 mm to (288.0, 235.8)
- moved C18 222.0 mm to (264.5, 243.8)
- moved C11 210.1 mm to (264.2, 240.0)
- moved L2 203.4 mm to (284.1, 233.0)
- moved R16 189.7 mm to (282.0, 180.5)
- moved R11 188.9 mm to (288.2, 242.5)
- moved SW2 188.9 mm to (258.2, 211.5)
- moved U5 184.8 mm to (287.8, 231.5)
- moved D2 179.8 mm to (278.3, 184.2)
- moved R21 179.0 mm to (287.0, 209.8)
- moved C26 177.9 mm to (238.5, 217.0)
- moved D3 176.4 mm to (274.5, 184.2)
- moved R12 176.1 mm to (287.0, 188.2)
- moved U4 176.0 mm to (264.2, 234.5)
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Connections:
- R5 pad 1: USB_PWR_SEL -> USB_ID
- U3 pad 1: USB_PWR_SEL -> USB_ID
- U3 pad 2: USB_PWR_SEL -> USB_ID
Routing:
- added copper zone on B.Cu, net GND
- added copper zone on F.Cu, net GND
