File: MP_AvrBaseBoard_v4/MakerPlayground_Baseboard.kicad_pcb (KiCad board)
At the start: 2 copper layers, 69.5 x 60.6 mm, 68 parts, among them J10 112504RT/RH, J11 112504RT/RH, J13 112504RT/RH, J14 112504RT/RH, J2 USB_B_Micro, J3 AVR-ISP-6, J4 112504RT/RH, J5 112504RT/RH, J6 112504RT/RH, J7 112504RT/RH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

Commit message: Fix the GREATEST ERROR on I2C & GND PTH overlap.
Routing:
- net GND: vias 92 -> 90
Changed lines of the file:
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@@
     (thickness 1.6)
     (drawings 336)
-    (tracks 819)
+    (tracks 817)
     (zones 0)
     (modules 68)
@@
   (via (at 123.75 114) (size 0.6) (drill 0.3) (layers F.Cu B.Cu) (net 1))
   (via (at 129 86.5) (size 0.6) (drill 0.3) (layers F.Cu B.Cu) (net 1))
-  (via (at 156.5 109.75) (size 0.6) (drill 0.3) (layers F.Cu B.Cu) (net 1))
-  (via (at 157.25 108.5) (size 0.6) (drill 0.3) (layers F.Cu B.Cu) (net 1))
   (via (at 123.75 116.25) (size 0.6) (drill 0.3) (layers F.Cu B.Cu) (net 1))
   (via (at 123.75 122.75) (size 0.6) (drill 0.3) (layers F.Cu B.Cu) (net 1))

Commit message: v4 upgraded, Improved 5V track location, ground pouring and some via holes position.
Routing:
- net SDA0: track 55.4 -> 64.7 mm
- net A5: track 28.5 -> 20.5 mm
- net +5V: track 319.9 -> 326.6 mm, vias 5 -> 6
- net GND: track 27.6 -> 32.2 mm, vias 90 -> 93
- net ESP_TX: track 51.8 -> 56.1 mm
- net A4: track 25.5 -> 22.2 mm
- net ESP_RX: track 22.2 -> 25.2 mm
- net SCL0: track 62.0 -> 59.6 mm
- net Net-(F1-Pad2): track 5.45 -> 3.69 mm
- net +3V3: track 62.8 -> 64.5 mm
- net SCK: track 10.4 -> 11.5 mm, vias 0 -> 1
- net RST: track 66.6 -> 67.5 mm
